Commit message: Add alicia v5_5 urdf

File: AliciaD/v5_5/gripper100mm/urdf/alicia_duo_with_gripper.urdf (robot description, URDF)
Before this commit: robot alicia_duo_with_gripper, 9 links, 8 joints
Links:
- link Link1: geometry collision mesh filename=package://lingdong_URDF_4.0/meshes/Link1.STL; visual mesh filename=package://lingdong_URDF_4.0/meshes/Link1.STL
- link Link2: geometry collision mesh filename=package://lingdong_URDF_4.0/meshes/Link2.STL; visual mesh filename=package://lingdong_URDF_4.0/meshes/Link2.STL
- link Link3: mass 0.0845575643881721 -> 0.0845575643881719; geometry collision mesh filename=package://lingdong_URDF_4.0/meshes/Link3.STL; visual mesh filename=package://lingdong_URDF_4.0/meshes/Link3.STL
- link Link4: mass 0.0653695985152062 -> 0.0653695983290511; geometry collision mesh filename=package://lingdong_URDF_4.0/meshes/Link4.STL; visual mesh filename=package://lingdong_URDF_4.0/meshes/Link4.STL
- link Link5: mass 0.0507639016939595 -> 0.0507639016939435; geometry collision mesh filename=package://lingdong_URDF_4.0/meshes/Link5.STL; visual mesh filename=package://lingdong_URDF_4.0/meshes/Link5.STL
- link Link6: geometry collision mesh filename=package://lingdong_URDF_4.0/meshes/Link6.STL; visual mesh filename=package://lingdong_URDF_4.0/meshes/Link6.STL
- link Link7: geometry collision mesh filename=package://lingdong_URDF_4.0/meshes/Link7.STL; visual mesh filename=package://lingdong_URDF_4.0/meshes/Link7.STL
- link Link8: mass 0.0256461121677874 -> 0.0256461121677875; geometry collision mesh filename=package://lingdong_URDF_4.0/meshes/Link8.STL; visual mesh filename=package://lingdong_URDF_4.0/meshes/Link8.STL
- link base_link: mass 0.733961424639881 -> 0.73396142463988; geometry collision mesh filename=package://lingdong_URDF_4.0/meshes/base_link.STL; visual mesh filename=package://lingdong_URDF_4.0/meshes/base_link.STL
