Commit message: Refactor the repo

File: urdf/Alicia-D_v5_4/alicia_d_with_gripper.urdf (robot description, URDF)
Before this commit: robot alicia_D_v5_5, 11 links, 10 joints
Links:
- link Grasp_base: geometry collision mesh filename=../../meshes/Alicia-D_v5_4/Grasp_base.STL; visual mesh filename=../../meshes/Alicia-D_v5_4/Grasp_base.STL
- link Link1: geometry collision mesh filename=../../meshes/Alicia-D_v5_4/Link1.STL; visual mesh filename=../../meshes/Alicia-D_v5_4/Link1.STL
- link Link2: geometry collision mesh filename=../../meshes/Alicia-D_v5_4/Link2.STL; visual mesh filename=../../meshes/Alicia-D_v5_4/Link2.STL
- link Link3: geometry collision mesh filename=../../meshes/Alicia-D_v5_4/Link3.STL; visual mesh filename=../../meshes/Alicia-D_v5_4/Link3.STL
- link Link4: geometry collision mesh filename=../../meshes/Alicia-D_v5_4/Link4.STL; visual mesh filename=../../meshes/Alicia-D_v5_4/Link4.STL
- link Link5: geometry collision mesh filename=../../meshes/Alicia-D_v5_4/Link5.STL; visual mesh filename=../../meshes/Alicia-D_v5_4/Link5.STL
- link Link6: geometry collision mesh filename=../../meshes/Alicia-D_v5_4/Link6.STL; visual mesh filename=../../meshes/Alicia-D_v5_4/Link6.STL
- link Link7: geometry collision mesh filename=../../meshes/Alicia-D_v5_4/Link7.STL; visual mesh filename=../../meshes/Alicia-D_v5_4/Link7.STL
- link Link8: geometry collision mesh filename=../../meshes/Alicia-D_v5_4/Link8.STL; visual mesh filename=../../meshes/Alicia-D_v5_4/Link8.STL
- link base_link: geometry collision mesh filename=../../meshes/Alicia-D_v5_4/base_link.STL; visual mesh filename=../../meshes/Alicia-D_v5_4/base_link.STL

File: urdf/Alicia-D_v5_5/alicia_d_gripper_100mm.urdf (robot description, URDF)
Before this commit: robot alicia_duo_with_gripper, 9 links, 8 joints
Links:
- link Link1: geometry collision mesh filename=../../meshes/Alicia-D_v5_5/gripper100mm/Link1.STL; visual mesh filename=../../meshes/Alicia-D_v5_5/gripper100mm/Link1.STL
- link Link2: geometry collision mesh filename=../../meshes/Alicia-D_v5_5/gripper100mm/Link2.STL; visual mesh filename=../../meshes/Alicia-D_v5_5/gripper100mm/Link2.STL
- link Link3: geometry collision mesh filename=../../meshes/Alicia-D_v5_5/gripper100mm/Link3.STL; visual mesh filename=../../meshes/Alicia-D_v5_5/gripper100mm/Link3.STL
- link Link4: geometry collision mesh filename=../../meshes/Alicia-D_v5_5/gripper100mm/Link4.STL; visual mesh filename=../../meshes/Alicia-D_v5_5/gripper100mm/Link4.STL
- link Link5: geometry collision mesh filename=../../meshes/Alicia-D_v5_5/gripper100mm/Link5.STL; visual mesh filename=../../meshes/Alicia-D_v5_5/gripper100mm/Link5.STL
- link Link6: geometry collision mesh filename=../../meshes/Alicia-D_v5_5/gripper100mm/Link6.STL; visual mesh filename=../../meshes/Alicia-D_v5_5/gripper100mm/Link6.STL
- link Link7: geometry collision mesh filename=../../meshes/Alicia-D_v5_5/gripper100mm/Link7.STL; visual mesh filename=../../meshes/Alicia-D_v5_5/gripper100mm/Link7.STL
- link Link8: geometry collision mesh filename=../../meshes/Alicia-D_v5_5/gripper100mm/Link8.STL; visual mesh filename=../../meshes/Alicia-D_v5_5/gripper100mm/Link8.STL
- link base_link: geometry collision mesh filename=../../meshes/Alicia-D_v5_5/gripper100mm/base_link.STL; visual mesh filename=../../meshes/Alicia-D_v5_5/gripper100mm/base_link.STL
Joints:
- joint left_finger: axis 0 0 -1 -> 0 0 1; limit lower=0 upper=-0.05 effort=5 velocity=12 -> lower=-0.05 upper=0 effort=5 velocity=12
- joint right_finger: axis 0 0 1 -> 0 0 -1; limit lower=0.05 upper=0 effort=5 velocity=12 -> lower=0 upper=0.05 effort=5 velocity=12

File: urdf/Alicia-D_v5_5/alicia_d_gripper_50mm.urdf (robot description, URDF)
Before this commit: robot alicia_duo_with_gripper, 9 links, 8 joints
Links:
- link Link1: geometry collision mesh filename=../../meshes/Alicia-D_v5_5/gripper50mm/Link1.STL; visual mesh filename=../../meshes/Alicia-D_v5_5/gripper50mm/Link1.STL
- link Link2: geometry collision mesh filename=../../meshes/Alicia-D_v5_5/gripper50mm/Link2.STL; visual mesh filename=../../meshes/Alicia-D_v5_5/gripper50mm/Link2.STL
- link Link3: geometry collision mesh filename=../../meshes/Alicia-D_v5_5/gripper50mm/Link3.STL; visual mesh filename=../../meshes/Alicia-D_v5_5/gripper50mm/Link3.STL
- link Link4: geometry collision mesh filename=../../meshes/Alicia-D_v5_5/gripper50mm/Link4.STL; visual mesh filename=../../meshes/Alicia-D_v5_5/gripper50mm/Link4.STL
- link Link5: geometry collision mesh filename=../../meshes/Alicia-D_v5_5/gripper50mm/Link5.STL; visual mesh filename=../../meshes/Alicia-D_v5_5/gripper50mm/Link5.STL
- link Link6: geometry collision mesh filename=../../meshes/Alicia-D_v5_5/gripper50mm/Link6.STL; visual mesh filename=../../meshes/Alicia-D_v5_5/gripper50mm/Link6.STL
- link Link7: geometry collision mesh filename=../../meshes/Alicia-D_v5_5/gripper50mm/Link7.STL; visual mesh filename=../../meshes/Alicia-D_v5_5/gripper50mm/Link7.STL
- link Link8: geometry collision mesh filename=../../meshes/Alicia-D_v5_5/gripper50mm/Link8.STL; visual mesh filename=../../meshes/Alicia-D_v5_5/gripper50mm/Link8.STL
- link base_link: geometry collision mesh filename=../../meshes/Alicia-D_v5_5/gripper50mm/base_link.STL; visual mesh filename=../../meshes/Alicia-D_v5_5/gripper50mm/base_link.STL
Joints:
- joint left_finger: axis 0 0 -1 -> 0 0 1; limit lower=0 upper=-0.05 effort=5 velocity=12 -> lower=-0.025 upper=0 effort=5 velocity=10
- joint right_finger: axis 0 0 1 -> 0 0 -1; limit lower=0.05 upper=0 effort=5 velocity=12 -> lower=0 upper=0.025 effort=5 velocity=10

File: urdf/Bessica-D_v1_0/Bessica-D_Covered.urdf (robot description, URDF)
Before this commit: robot BessicaDCodver, 22 links, 21 joints
Links:
- link base_link: geometry collision mesh filename=../../meshes/Bessica-D_v1_0/withCover/base_link.STL; visual mesh filename=../../meshes/Bessica-D_v1_0/withCover/base_link.STL
- link left_arm_base_link: geometry collision mesh filename=../../meshes/Bessica-D_v1_0/withCover/left_arm_base_link.STL; visual mesh filename=../../meshes/Bessica-D_v1_0/withCover/left_arm_base_link.STL
- link left_arm_gripper_left_finger: geometry collision mesh filename=../../meshes/Bessica-D_v1_0/withCover/left_arm_gripper_left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; visual mesh filename=../../meshes/Bessica-D_v1_0/withCover/left_arm_gripper_left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
- link left_arm_gripper_right_finger: geometry collision mesh filename=../../meshes/Bessica-D_v1_0/withCover/left_arm_gripper_righ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; visual mesh filename=../../meshes/Bessica-D_v1_0/withCover/left_arm_gripper_righ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
- link left_arm_link1: geometry collision mesh filename=../../meshes/Bessica-D_v1_0/withCover/left_arm_link1.STL; visual mesh filename=../../meshes/Bessica-D_v1_0/withCover/left_arm_link1.STL
- link left_arm_link2: geometry collision mesh filename=../../meshes/Bessica-D_v1_0/withCover/left_arm_link2.STL; visual mesh filename=../../meshes/Bessica-D_v1_0/withCover/left_arm_link2.STL
- link left_arm_link3: geometry collision mesh filename=../../meshes/Bessica-D_v1_0/withCover/left_arm_link3.STL; visual mesh filename=../../meshes/Bessica-D_v1_0/withCover/left_arm_link3.STL
- link left_arm_link4: geometry collision mesh filename=../../meshes/Bessica-D_v1_0/withCover/left_arm_link4.STL; visual mesh filename=../../meshes/Bessica-D_v1_0/withCover/left_arm_link4.STL
- link left_arm_link5: geometry collision mesh filename=../../meshes/Bessica-D_v1_0/withCover/left_arm_link5.STL; visual mesh filename=../../meshes/Bessica-D_v1_0/withCover/left_arm_link5.STL
- link left_arm_link6: geometry collision mesh filename=../../meshes/Bessica-D_v1_0/withCover/left_arm_link6.STL; visual mesh filename=../../meshes/Bessica-D_v1_0/withCover/left_arm_link6.STL
- link left_arm_link7: geometry collision mesh filename=../../meshes/Bessica-D_v1_0/withCover/left_arm_link7.STL; visual mesh filename=../../meshes/Bessica-D_v1_0/withCover/left_arm_link7.STL
- link right_arm_base_link: geometry collision mesh filename=../../meshes/Bessica-D_v1_0/withCover/right_arm_base_link.S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; visual mesh filename=../../meshes/Bessica-D_v1_0/withCover/right_arm_base_link.S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
- link right_arm_gripper_left_finger: geometry collision mesh filename=../../meshes/Bessica-D_v1_0/withCover/right_arm_gripper_lef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; visual mesh filename=../../meshes/Bessica-D_v1_0/withCover/right_arm_gripper_lef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
- link right_arm_gripper_right_finger: geometry collision mesh filename=../../meshes/Bessica-D_v1_0/withCover/right_arm_gripper_rig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; visual mesh filename=../../meshes/Bessica-D_v1_0/withCover/right_arm_gripper_rig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
- link right_arm_link1: geometry collision mesh filename=../../meshes/Bessica-D_v1_0/withCover/right_arm_link1.STL; visual mesh filename=../../meshes/Bessica-D_v1_0/withCover/right_arm_link1.STL
- link right_arm_link2: geometry collision mesh filename=../../meshes/Bessica-D_v1_0/withCover/right_arm_link2.STL; visual mesh filename=../../meshes/Bessica-D_v1_0/withCover/right_arm_link2.STL
- link right_arm_link3: geometry collision mesh filename=../../meshes/Bessica-D_v1_0/withCover/right_arm_link3.STL; visual mesh filename=../../meshes/Bessica-D_v1_0/withCover/right_arm_link3.STL
- link right_arm_link4: geometry collision mesh filename=../../meshes/Bessica-D_v1_0/withCover/right_arm_link4.STL; visual mesh filename=../../meshes/Bessica-D_v1_0/withCover/right_arm_link4.STL
- link right_arm_link5: geometry collision mesh filename=../../meshes/Bessica-D_v1_0/withCover/right_arm_link5.STL; visual mesh filename=../../meshes/Bessica-D_v1_0/withCover/right_arm_link5.STL
- link right_arm_link6: geometry collision mesh filename=../../meshes/Bessica-D_v1_0/withCover/right_arm_link6.STL; visual mesh filename=../../meshes/Bessica-D_v1_0/withCover/right_arm_link6.STL
- link right_arm_link7: geometry collision mesh filename=../../meshes/Bessica-D_v1_0/withCover/right_arm_link7.STL; visual mesh filename=../../meshes/Bessica-D_v1_0/withCover/right_arm_link7.STL
