Commit message: Modify Bessica urdf

File: urdf/Bessica-D_v1_0/bessica_D_skeleton.urdf (robot description, URDF)
Before this commit: robot bessica_d_v2_1, 23 links, 22 joints
Links:
- link base_link: geometry collision mesh filename=../../meshes/Bessica-D_v1_0/SkeletonOnly/base_link.STL; visual mesh filename=../../meshes/Bessica-D_v1_0/SkeletonOnly/base_link.STL
- link left_arm_base_link: geometry collision mesh filename=../../meshes/Bessica-D_v1_0/SkeletonOnly/left_arm_base_link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; visual mesh filename=../../meshes/Bessica-D_v1_0/SkeletonOnly/left_arm_base_link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
- link left_arm_gripper_base: geometry collision mesh filename=../../meshes/Bessica-D_v1_0/SkeletonOnly/left_arm_gripper_b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; visual mesh filename=../../meshes/Bessica-D_v1_0/SkeletonOnly/left_arm_gripper_b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
- link left_arm_gripper_left_finger: geometry collision mesh filename=../../meshes/Bessica-D_v1_0/SkeletonOnly/left_arm_gripper_l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; visual mesh filename=../../meshes/Bessica-D_v1_0/SkeletonOnly/left_arm_gripper_l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
- link left_arm_gripper_right_finger: geometry collision mesh filename=../../meshes/Bessica-D_v1_0/SkeletonOnly/left_arm_gripper_r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; visual mesh filename=../../meshes/Bessica-D_v1_0/SkeletonOnly/left_arm_gripper_r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
- link left_arm_link1: geometry collision mesh filename=../../meshes/Bessica-D_v1_0/SkeletonOnly/left_arm_link1.STL; visual mesh filename=../../meshes/Bessica-D_v1_0/SkeletonOnly/left_arm_link1.STL
- link left_arm_link2: geometry collision mesh filename=../../meshes/Bessica-D_v1_0/SkeletonOnly/left_arm_link2.STL; visual mesh filename=../../meshes/Bessica-D_v1_0/SkeletonOnly/left_arm_link2.STL
- link left_arm_link3: geometry collision mesh filename=../../meshes/Bessica-D_v1_0/SkeletonOnly/left_arm_link3.STL; visual mesh filename=../../meshes/Bessica-D_v1_0/SkeletonOnly/left_arm_link3.STL
- link left_arm_link4: geometry collision mesh filename=../../meshes/Bessica-D_v1_0/SkeletonOnly/left_arm_link4.STL; visual mesh filename=../../meshes/Bessica-D_v1_0/SkeletonOnly/left_arm_link4.STL
- link left_arm_link5: geometry collision mesh filename=../../meshes/Bessica-D_v1_0/SkeletonOnly/left_arm_link5.STL; visual mesh filename=../../meshes/Bessica-D_v1_0/SkeletonOnly/left_arm_link5.STL
- link left_arm_link6: geometry collision mesh filename=../../meshes/Bessica-D_v1_0/SkeletonOnly/left_arm_link6.STL; visual mesh filename=../../meshes/Bessica-D_v1_0/SkeletonOnly/left_arm_link6.STL
- link left_arm_link7: geometry collision mesh filename=../../meshes/Bessica-D_v1_0/SkeletonOnly/left_arm_link7.STL; visual mesh filename=../../meshes/Bessica-D_v1_0/SkeletonOnly/left_arm_link7.STL
- link right_arm_base_link: geometry collision mesh filename=../../meshes/Bessica-D_v1_0/SkeletonOnly/right_arm_base_lin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; visual mesh filename=../../meshes/Bessica-D_v1_0/SkeletonOnly/right_arm_base_lin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
- link right_arm_gripper_base: geometry collision mesh filename=../../meshes/Bessica-D_v1_0/SkeletonOnly/right_arm_gripper_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; visual mesh filename=../../meshes/Bessica-D_v1_0/SkeletonOnly/right_arm_gripper_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
- link right_arm_gripper_left_finger: geometry collision mesh filename=../../meshes/Bessica-D_v1_0/SkeletonOnly/right_arm_gripper_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; visual mesh filename=../../meshes/Bessica-D_v1_0/SkeletonOnly/right_arm_gripper_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
- link right_arm_gripper_right_finger: geometry collision mesh filename=../../meshes/Bessica-D_v1_0/SkeletonOnly/right_arm_gripper_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; visual mesh filename=../../meshes/Bessica-D_v1_0/SkeletonOnly/right_arm_gripper_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
- link right_arm_link1: geometry collision mesh filename=../../meshes/Bessica-D_v1_0/SkeletonOnly/right_arm_link1.STL; visual mesh filename=../../meshes/Bessica-D_v1_0/SkeletonOnly/right_arm_link1.STL
- link right_arm_link2: geometry collision mesh filename=../../meshes/Bessica-D_v1_0/SkeletonOnly/right_arm_link2.STL; visual mesh filename=../../meshes/Bessica-D_v1_0/SkeletonOnly/right_arm_link2.STL
- link right_arm_link3: geometry collision mesh filename=../../meshes/Bessica-D_v1_0/SkeletonOnly/right_arm_link3.STL; visual mesh filename=../../meshes/Bessica-D_v1_0/SkeletonOnly/right_arm_link3.STL
- link right_arm_link4: geometry collision mesh filename=../../meshes/Bessica-D_v1_0/SkeletonOnly/right_arm_link4.STL; visual mesh filename=../../meshes/Bessica-D_v1_0/SkeletonOnly/right_arm_link4.STL
- link right_arm_link5: geometry collision mesh filename=../../meshes/Bessica-D_v1_0/SkeletonOnly/right_arm_link5.STL; visual mesh filename=../../meshes/Bessica-D_v1_0/SkeletonOnly/right_arm_link5.STL
- link right_arm_link6: geometry collision mesh filename=../../meshes/Bessica-D_v1_0/SkeletonOnly/right_arm_link6.STL; visual mesh filename=../../meshes/Bessica-D_v1_0/SkeletonOnly/right_arm_link6.STL
- link right_arm_link7: geometry collision mesh filename=../../meshes/Bessica-D_v1_0/SkeletonOnly/right_arm_link7.STL; visual mesh filename=../../meshes/Bessica-D_v1_0/SkeletonOnly/right_arm_link7.STL
