Commit message: Rename the folder and add tool0

File: robot_descriptions/urdf/Alicia_D_v5_4/alicia_d_with_gripper.urdf (robot description, URDF)
Before this commit: robot alicia_D_v5_4_gripper_50mm, 11 links, 10 joints
Links:
- link Grasp_base: geometry collision mesh filename=../../meshes/Alicia_D_v5_4/Grasp_base.STL; visual mesh filename=../../meshes/Alicia_D_v5_4/Grasp_base.STL
- link Link1: geometry collision mesh filename=../../meshes/Alicia_D_v5_4/Link1.STL; visual mesh filename=../../meshes/Alicia_D_v5_4/Link1.STL
- link Link2: geometry collision mesh filename=../../meshes/Alicia_D_v5_4/Link2.STL; visual mesh filename=../../meshes/Alicia_D_v5_4/Link2.STL
- link Link3: geometry collision mesh filename=../../meshes/Alicia_D_v5_4/Link3.STL; visual mesh filename=../../meshes/Alicia_D_v5_4/Link3.STL
- link Link4: geometry collision mesh filename=../../meshes/Alicia_D_v5_4/Link4.STL; visual mesh filename=../../meshes/Alicia_D_v5_4/Link4.STL
- link Link5: geometry collision mesh filename=../../meshes/Alicia_D_v5_4/Link5.STL; visual mesh filename=../../meshes/Alicia_D_v5_4/Link5.STL
- link Link6: geometry collision mesh filename=../../meshes/Alicia_D_v5_4/Link6.STL; visual mesh filename=../../meshes/Alicia_D_v5_4/Link6.STL
- link Link7: geometry collision mesh filename=../../meshes/Alicia_D_v5_4/Link7.STL; visual mesh filename=../../meshes/Alicia_D_v5_4/Link7.STL
- link Link8: geometry collision mesh filename=../../meshes/Alicia_D_v5_4/Link8.STL; visual mesh filename=../../meshes/Alicia_D_v5_4/Link8.STL
- link base_link: geometry collision mesh filename=../../meshes/Alicia_D_v5_4/base_link.STL; visual mesh filename=../../meshes/Alicia_D_v5_4/base_link.STL

File: robot_descriptions/urdf/Alicia_D_v5_5/alicia_d_gripper_100mm.urdf (robot description, URDF)
Before this commit: robot alicia_d_with_gripper, 9 links, 8 joints
Links:
- added link tool0; visual sphere radius=0.005
- link Link1: mass 0.195233452997327 -> 0.195233452997315; geometry collision mesh filename=../../meshes/Alicia_D_v5_5/gripper100mm/Link1.STL; visual mesh filename=../../meshes/Alicia_D_v5_5/gripper100mm/Link1.STL
- link Link2: mass 0.207033693061786 -> 0.207033693061785; geometry collision mesh filename=../../meshes/Alicia_D_v5_5/gripper100mm/Link2.STL; visual mesh filename=../../meshes/Alicia_D_v5_5/gripper100mm/Link2.STL
- link Link3: mass 0.0845575636182319 -> 0.0845575643881719; geometry collision mesh filename=../../meshes/Alicia_D_v5_5/gripper100mm/Link3.STL; visual mesh filename=../../meshes/Alicia_D_v5_5/gripper100mm/Link3.STL
- link Link4: mass 0.0653695953286769 -> 0.0653695983290511; geometry collision mesh filename=../../meshes/Alicia_D_v5_5/gripper100mm/Link4.STL; visual mesh filename=../../meshes/Alicia_D_v5_5/gripper100mm/Link4.STL
- link Link5: mass 0.0507639016939355 -> 0.0507639016939435; geometry collision mesh filename=../../meshes/Alicia_D_v5_5/gripper100mm/Link5.STL; visual mesh filename=../../meshes/Alicia_D_v5_5/gripper100mm/Link5.STL
- link Link6: mass 0.130364883326573 -> 0.123298967748658; geometry collision mesh filename=../../meshes/Alicia_D_v5_5/gripper100mm/Link6.STL; visual mesh filename=../../meshes/Alicia_D_v5_5/gripper100mm/Link6.STL
- link Link7: geometry collision mesh filename=../../meshes/Alicia_D_v5_5/gripper100mm/Link7.STL; visual mesh filename=../../meshes/Alicia_D_v5_5/gripper100mm/Link7.STL
- link Link8: mass 0.0256461121677874 -> 0.0256461121677875; geometry collision mesh filename=../../meshes/Alicia_D_v5_5/gripper100mm/Link8.STL; visual mesh filename=../../meshes/Alicia_D_v5_5/gripper100mm/Link8.STL
- link base_link: geometry collision mesh filename=../../meshes/Alicia_D_v5_5/gripper100mm/base_link.STL; visual mesh filename=../../meshes/Alicia_D_v5_5/gripper100mm/base_link.STL
Joints:
- added joint Grasp2tool: type fixed, parent Link6, child tool0, origin xyz=-0.0002 -0.0003 0.13118 rpy=0 0 0, axis 0 0 0
- joint Joint6: origin xyz=-0.00385 -0.0575 0.001 rpy=1.5708 0 0 -> xyz=-0.00384999999999946 -0.0574999999999999 0.00100000000000069 rpy=1.5707963267949 0 0
- joint left_finger: limit lower=-0.025 upper=0 effort=5 velocity=10 -> lower=-0.05 upper=0 effort=5 velocity=12; origin xyz=0.0002 -0.025469 0.13098 rpy=1.5708 0 0 -> xyz=-0.0002 -0.036537 0.13098 rpy=1.5708 0 0
- joint right_finger: limit lower=0 upper=0.025 effort=5 velocity=10 -> lower=0 upper=0.05 effort=5 velocity=12; origin xyz=0.0002 0.025469 0.13098 rpy=-1.5708 0 0 -> xyz=-0.0002 0.036518 0.13098 rpy=-1.5708 0 0

File: robot_descriptions/urdf/Alicia_D_v5_5/alicia_d_gripper_50mm.urdf (robot description, URDF)
Before this commit: robot alicia_d_with_gripper, 9 links, 8 joints
Links:
- added link tool0; visual sphere radius=0.005
- link Link1: mass 0.195233452997315 -> 0.195233452997327; geometry collision mesh filename=../../meshes/Alicia_D_v5_5/gripper50mm/Link1.STL; visual mesh filename=../../meshes/Alicia_D_v5_5/gripper50mm/Link1.STL
- link Link2: mass 0.207033693061785 -> 0.207033693061786; geometry collision mesh filename=../../meshes/Alicia_D_v5_5/gripper50mm/Link2.STL; visual mesh filename=../../meshes/Alicia_D_v5_5/gripper50mm/Link2.STL
- link Link3: mass 0.0845575643881719 -> 0.0845575636182319; geometry collision mesh filename=../../meshes/Alicia_D_v5_5/gripper50mm/Link3.STL; visual mesh filename=../../meshes/Alicia_D_v5_5/gripper50mm/Link3.STL
- link Link4: mass 0.0653695983290511 -> 0.0653695953286769; geometry collision mesh filename=../../meshes/Alicia_D_v5_5/gripper50mm/Link4.STL; visual mesh filename=../../meshes/Alicia_D_v5_5/gripper50mm/Link4.STL
- link Link5: mass 0.0507639016939435 -> 0.0507639016939355; geometry collision mesh filename=../../meshes/Alicia_D_v5_5/gripper50mm/Link5.STL; visual mesh filename=../../meshes/Alicia_D_v5_5/gripper50mm/Link5.STL
- link Link6: mass 0.123298967748658 -> 0.130364883326573; geometry collision mesh filename=../../meshes/Alicia_D_v5_5/gripper50mm/Link6.STL; visual mesh filename=../../meshes/Alicia_D_v5_5/gripper50mm/Link6.STL
- link Link7: geometry collision mesh filename=../../meshes/Alicia_D_v5_5/gripper50mm/Link7.STL; visual mesh filename=../../meshes/Alicia_D_v5_5/gripper50mm/Link7.STL
- link Link8: mass 0.0256461121677875 -> 0.0256461121677874; geometry collision mesh filename=../../meshes/Alicia_D_v5_5/gripper50mm/Link8.STL; visual mesh filename=../../meshes/Alicia_D_v5_5/gripper50mm/Link8.STL
- link base_link: geometry collision mesh filename=../../meshes/Alicia_D_v5_5/gripper50mm/base_link.STL; visual mesh filename=../../meshes/Alicia_D_v5_5/gripper50mm/base_link.STL
Joints:
- added joint Grasp2tool: type fixed, parent Link6, child tool0, origin xyz=-0.0002 -0.0003 0.13118 rpy=0 0 0, axis 0 0 0
- joint Joint6: origin xyz=-0.00384999999999946 -0.0574999999999999 0.00100000000000069 rpy=1.5707963267949 0 0 -> xyz=-0.00385 -0.0575 0.001 rpy=1.5708 0 0
- joint left_finger: limit lower=-0.05 upper=0 effort=5 velocity=12 -> lower=-0.025 upper=0 effort=5 velocity=10; origin xyz=-0.0002 -0.036537 0.13098 rpy=1.5708 0 0 -> xyz=0.0002 -0.025469 0.13098 rpy=1.5708 0 0
- joint right_finger: limit lower=0 upper=0.05 effort=5 velocity=12 -> lower=0 upper=0.025 effort=5 velocity=10; origin xyz=-0.0002 0.036518 0.13098 rpy=-1.5708 0 0 -> xyz=0.0002 0.025469 0.13098 rpy=-1.5708 0 0

File: robot_descriptions/urdf/Bessica_D_v1_0/Bessica-D_Covered.urdf (robot description, URDF)
Before this commit: robot Bessica-D_Covered, 22 links, 21 joints
Links:
- link base_link: geometry collision mesh filename=../../meshes/Bessica_D_v1_0/withCover/base_link.STL; visual mesh filename=../../meshes/Bessica_D_v1_0/withCover/base_link.STL
- link left_arm_base_link: geometry collision mesh filename=../../meshes/Bessica_D_v1_0/withCover/left_arm_base_link.STL; visual mesh filename=../../meshes/Bessica_D_v1_0/withCover/left_arm_base_link.STL
- link left_arm_gripper_left_finger: geometry collision mesh filename=../../meshes/Bessica_D_v1_0/withCover/left_arm_gripper_left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; visual mesh filename=../../meshes/Bessica_D_v1_0/withCover/left_arm_gripper_left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
- link left_arm_gripper_right_finger: geometry collision mesh filename=../../meshes/Bessica_D_v1_0/withCover/left_arm_gripper_righ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; visual mesh filename=../../meshes/Bessica_D_v1_0/withCover/left_arm_gripper_righ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
- link left_arm_link1: geometry collision mesh filename=../../meshes/Bessica_D_v1_0/withCover/left_arm_link1.STL; visual mesh filename=../../meshes/Bessica_D_v1_0/withCover/left_arm_link1.STL
- link left_arm_link2: geometry collision mesh filename=../../meshes/Bessica_D_v1_0/withCover/left_arm_link2.STL; visual mesh filename=../../meshes/Bessica_D_v1_0/withCover/left_arm_link2.STL
- link left_arm_link3: geometry collision mesh filename=../../meshes/Bessica_D_v1_0/withCover/left_arm_link3.STL; visual mesh filename=../../meshes/Bessica_D_v1_0/withCover/left_arm_link3.STL
- link left_arm_link4: geometry collision mesh filename=../../meshes/Bessica_D_v1_0/withCover/left_arm_link4.STL; visual mesh filename=../../meshes/Bessica_D_v1_0/withCover/left_arm_link4.STL
- link left_arm_link5: geometry collision mesh filename=../../meshes/Bessica_D_v1_0/withCover/left_arm_link5.STL; visual mesh filename=../../meshes/Bessica_D_v1_0/withCover/left_arm_link5.STL
- link left_arm_link6: geometry collision mesh filename=../../meshes/Bessica_D_v1_0/withCover/left_arm_link6.STL; visual mesh filename=../../meshes/Bessica_D_v1_0/withCover/left_arm_link6.STL
- link left_arm_link7: geometry collision mesh filename=../../meshes/Bessica_D_v1_0/withCover/left_arm_link7.STL; visual mesh filename=../../meshes/Bessica_D_v1_0/withCover/left_arm_link7.STL
- link right_arm_base_link: geometry collision mesh filename=../../meshes/Bessica_D_v1_0/withCover/right_arm_base_link.S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; visual mesh filename=../../meshes/Bessica_D_v1_0/withCover/right_arm_base_link.S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
- link right_arm_gripper_left_finger: geometry collision mesh filename=../../meshes/Bessica_D_v1_0/withCover/right_arm_gripper_lef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; visual mesh filename=../../meshes/Bessica_D_v1_0/withCover/right_arm_gripper_lef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
- link right_arm_gripper_right_finger: geometry collision mesh filename=../../meshes/Bessica_D_v1_0/withCover/right_arm_gripper_rig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; visual mesh filename=../../meshes/Bessica_D_v1_0/withCover/right_arm_gripper_rig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
- link right_arm_link1: geometry collision mesh filename=../../meshes/Bessica_D_v1_0/withCover/right_arm_link1.STL; visual mesh filename=../../meshes/Bessica_D_v1_0/withCover/right_arm_link1.STL
- link right_arm_link2: geometry collision mesh filename=../../meshes/Bessica_D_v1_0/withCover/right_arm_link2.STL; visual mesh filename=../../meshes/Bessica_D_v1_0/withCover/right_arm_link2.STL
- link right_arm_link3: geometry collision mesh filename=../../meshes/Bessica_D_v1_0/withCover/right_arm_link3.STL; visual mesh filename=../../meshes/Bessica_D_v1_0/withCover/right_arm_link3.STL
- link right_arm_link4: geometry collision mesh filename=../../meshes/Bessica_D_v1_0/withCover/right_arm_link4.STL; visual mesh filename=../../meshes/Bessica_D_v1_0/withCover/right_arm_link4.STL
- link right_arm_link5: geometry collision mesh filename=../../meshes/Bessica_D_v1_0/withCover/right_arm_link5.STL; visual mesh filename=../../meshes/Bessica_D_v1_0/withCover/right_arm_link5.STL
- link right_arm_link6: geometry collision mesh filename=../../meshes/Bessica_D_v1_0/withCover/right_arm_link6.STL; visual mesh filename=../../meshes/Bessica_D_v1_0/withCover/right_arm_link6.STL
- link right_arm_link7: geometry collision mesh filename=../../meshes/Bessica_D_v1_0/withCover/right_arm_link7.STL; visual mesh filename=../../meshes/Bessica_D_v1_0/withCover/right_arm_link7.STL

File: robot_descriptions/urdf/Bessica_D_v1_0/bessica_D_skeleton.urdf (robot description, URDF)
Before this commit: robot bessica_d_v2_1, 23 links, 22 joints
Links:
- link base_link: geometry collision mesh filename=../../meshes/Bessica_D_v1_0/SkeletonOnly/base_link.STL; visual mesh filename=../../meshes/Bessica_D_v1_0/SkeletonOnly/base_link.STL
- link left_arm_base_link: geometry collision mesh filename=../../meshes/Bessica_D_v1_0/SkeletonOnly/left_arm_base_link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; visual mesh filename=../../meshes/Bessica_D_v1_0/SkeletonOnly/left_arm_base_link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
- link left_arm_gripper_base: geometry collision mesh filename=../../meshes/Bessica_D_v1_0/SkeletonOnly/left_arm_gripper_b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; visual mesh filename=../../meshes/Bessica_D_v1_0/SkeletonOnly/left_arm_gripper_b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
- link left_arm_gripper_left_finger: geometry collision mesh filename=../../meshes/Bessica_D_v1_0/SkeletonOnly/left_arm_gripper_l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; visual mesh filename=../../meshes/Bessica_D_v1_0/SkeletonOnly/left_arm_gripper_l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
- link left_arm_gripper_right_finger: geometry collision mesh filename=../../meshes/Bessica_D_v1_0/SkeletonOnly/left_arm_gripper_r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; visual mesh filename=../../meshes/Bessica_D_v1_0/SkeletonOnly/left_arm_gripper_r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
- link left_arm_link1: geometry collision mesh filename=../../meshes/Bessica_D_v1_0/SkeletonOnly/left_arm_link1.STL; visual mesh filename=../../meshes/Bessica_D_v1_0/SkeletonOnly/left_arm_link1.STL
- link left_arm_link2: geometry collision mesh filename=../../meshes/Bessica_D_v1_0/SkeletonOnly/left_arm_link2.STL; visual mesh filename=../../meshes/Bessica_D_v1_0/SkeletonOnly/left_arm_link2.STL
- link left_arm_link3: geometry collision mesh filename=../../meshes/Bessica_D_v1_0/SkeletonOnly/left_arm_link3.STL; visual mesh filename=../../meshes/Bessica_D_v1_0/SkeletonOnly/left_arm_link3.STL
- link left_arm_link4: geometry collision mesh filename=../../meshes/Bessica_D_v1_0/SkeletonOnly/left_arm_link4.STL; visual mesh filename=../../meshes/Bessica_D_v1_0/SkeletonOnly/left_arm_link4.STL
- link left_arm_link5: geometry collision mesh filename=../../meshes/Bessica_D_v1_0/SkeletonOnly/left_arm_link5.STL; visual mesh filename=../../meshes/Bessica_D_v1_0/SkeletonOnly/left_arm_link5.STL
- link left_arm_link6: geometry collision mesh filename=../../meshes/Bessica_D_v1_0/SkeletonOnly/left_arm_link6.STL; visual mesh filename=../../meshes/Bessica_D_v1_0/SkeletonOnly/left_arm_link6.STL
- link left_arm_link7: geometry collision mesh filename=../../meshes/Bessica_D_v1_0/SkeletonOnly/left_arm_link7.STL; visual mesh filename=../../meshes/Bessica_D_v1_0/SkeletonOnly/left_arm_link7.STL
- link right_arm_base_link: geometry collision mesh filename=../../meshes/Bessica_D_v1_0/SkeletonOnly/right_arm_base_lin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; visual mesh filename=../../meshes/Bessica_D_v1_0/SkeletonOnly/right_arm_base_lin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
- link right_arm_gripper_base: geometry collision mesh filename=../../meshes/Bessica_D_v1_0/SkeletonOnly/right_arm_gripper_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; visual mesh filename=../../meshes/Bessica_D_v1_0/SkeletonOnly/right_arm_gripper_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
- link right_arm_gripper_left_finger: geometry collision mesh filename=../../meshes/Bessica_D_v1_0/SkeletonOnly/right_arm_gripper_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; visual mesh filename=../../meshes/Bessica_D_v1_0/SkeletonOnly/right_arm_gripper_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
- link right_arm_gripper_right_finger: geometry collision mesh filename=../../meshes/Bessica_D_v1_0/SkeletonOnly/right_arm_gripper_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; visual mesh filename=../../meshes/Bessica_D_v1_0/SkeletonOnly/right_arm_gripper_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
- link right_arm_link1: geometry collision mesh filename=../../meshes/Bessica_D_v1_0/SkeletonOnly/right_arm_link1.STL; visual mesh filename=../../meshes/Bessica_D_v1_0/SkeletonOnly/right_arm_link1.STL
- link right_arm_link2: geometry collision mesh filename=../../meshes/Bessica_D_v1_0/SkeletonOnly/right_arm_link2.STL; visual mesh filename=../../meshes/Bessica_D_v1_0/SkeletonOnly/right_arm_link2.STL
- link right_arm_link3: geometry collision mesh filename=../../meshes/Bessica_D_v1_0/SkeletonOnly/right_arm_link3.STL; visual mesh filename=../../meshes/Bessica_D_v1_0/SkeletonOnly/right_arm_link3.STL
- link right_arm_link4: geometry collision mesh filename=../../meshes/Bessica_D_v1_0/SkeletonOnly/right_arm_link4.STL; visual mesh filename=../../meshes/Bessica_D_v1_0/SkeletonOnly/right_arm_link4.STL
- link right_arm_link5: geometry collision mesh filename=../../meshes/Bessica_D_v1_0/SkeletonOnly/right_arm_link5.STL; visual mesh filename=../../meshes/Bessica_D_v1_0/SkeletonOnly/right_arm_link5.STL
- link right_arm_link6: geometry collision mesh filename=../../meshes/Bessica_D_v1_0/SkeletonOnly/right_arm_link6.STL; visual mesh filename=../../meshes/Bessica_D_v1_0/SkeletonOnly/right_arm_link6.STL
- link right_arm_link7: geometry collision mesh filename=../../meshes/Bessica_D_v1_0/SkeletonOnly/right_arm_link7.STL; visual mesh filename=../../meshes/Bessica_D_v1_0/SkeletonOnly/right_arm_link7.STL
