Commit message: Correct the rotation direction

File: robot_descriptions/urdf/Alicia_D_v5_5/Alicia_D_gripper_100mm.urdf (robot description, URDF)
Before this commit: robot alicia_d_with_gripper, 10 links, 9 joints
Joints:
- joint Joint1: axis 0 0 -1 -> 0 0 1
- joint Joint2: axis 0 0 1 -> 0 0 -1
- joint Joint3: axis 0 0 1 -> 0 0 -1
- joint Joint4: axis 0 0 -1 -> 0 0 1
- joint Joint5: axis 0 0 1 -> 0 0 -1

File: robot_descriptions/urdf/Alicia_D_v5_5/Alicia_D_gripper_50mm.urdf (robot description, URDF)
Before this commit: robot alicia_d_with_gripper, 10 links, 9 joints
Joints:
- joint Joint1: axis 0 0 -1 -> 0 0 1
- joint Joint2: axis 0 0 1 -> 0 0 -1
- joint Joint3: axis 0 0 1 -> 0 0 -1
- joint Joint4: axis 0 0 -1 -> 0 0 1
- joint Joint5: axis 0 0 1 -> 0 0 -1

Commit message: Rotate the robot orientation

File: robot_descriptions/urdf/Alicia_D_v5_5/Alicia_D_gripper_100mm.urdf (robot description, URDF)
Before this commit: robot Alicia_D_gripper_100mm, 10 links, 9 joints
Links:
- added link world, mass 0.001
Joints:
- added joint virtual_joint: type revolute, parent world, child base_link, origin xyz=0 0 0 rpy=0 0 3.14, axis 0 0 1, limit lower=-3.14159 upper=3.14159 effort=0 velocity=0

File: robot_descriptions/urdf/Alicia_D_v5_5/Alicia_D_gripper_50mm.urdf (robot description, URDF)
Before this commit: robot Alicia_D_gripper_50mm, 10 links, 9 joints
Links:
- added link world, mass 0.001
Joints:
- added joint virtual_joint: type revolute, parent world, child base_link, origin xyz=0 0 0 rpy=0 0 3.14, axis 0 0 1, limit lower=-3.14159 upper=3.14159 effort=0 velocity=0
