Commit message: Standarlize the file names

File: robot_descriptions/urdf/Alicia_D_v5_5/Alicia_D_v5_5_gripper_100mm.urdf (robot description, URDF)
Before this commit: robot alicia_D_v5_4_gripper_50mm, 11 links, 10 joints
Links:
- link Grasp_base: geometry collision mesh filename=../../meshes/Alicia_D_v5_5/Grasp_base.STL; visual mesh filename=../../meshes/Alicia_D_v5_5/Grasp_base.STL
- link Link1: geometry collision mesh filename=../../meshes/Alicia_D_v5_5/Link1.STL; visual mesh filename=../../meshes/Alicia_D_v5_5/Link1.STL
- link Link2: geometry collision mesh filename=../../meshes/Alicia_D_v5_5/Link2.STL; visual mesh filename=../../meshes/Alicia_D_v5_5/Link2.STL
- link Link3: geometry collision mesh filename=../../meshes/Alicia_D_v5_5/Link3.STL; visual mesh filename=../../meshes/Alicia_D_v5_5/Link3.STL
- link Link4: geometry collision mesh filename=../../meshes/Alicia_D_v5_5/Link4.STL; visual mesh filename=../../meshes/Alicia_D_v5_5/Link4.STL
- link Link5: geometry collision mesh filename=../../meshes/Alicia_D_v5_5/Link5.STL; visual mesh filename=../../meshes/Alicia_D_v5_5/Link5.STL
- link Link6: geometry collision mesh filename=../../meshes/Alicia_D_v5_5/Link6.STL; visual mesh filename=../../meshes/Alicia_D_v5_5/Link6.STL
- link Link7: geometry collision mesh filename=../../meshes/Alicia_D_v5_5/Link7.STL; visual mesh filename=../../meshes/Alicia_D_v5_5/Link7.STL
- link Link8: geometry collision mesh filename=../../meshes/Alicia_D_v5_5/Link8.STL; visual mesh filename=../../meshes/Alicia_D_v5_5/Link8.STL
- link base_link: geometry collision mesh filename=../../meshes/Alicia_D_v5_5/base_link.STL; visual mesh filename=../../meshes/Alicia_D_v5_5/base_link.STL

File: robot_descriptions/urdf/Alicia_D_v5_6/Alicia_D_v5_6_gripper_100mm.urdf (robot description, URDF)
Before this commit: robot Alicia_D_gripper_100mm, 11 links, 10 joints
Links:
- link Link1: geometry collision mesh filename=../../meshes/Alicia_D_v5_6/gripper100mm/Link1.STL; visual mesh filename=../../meshes/Alicia_D_v5_6/gripper100mm/Link1.STL
- link Link2: geometry collision mesh filename=../../meshes/Alicia_D_v5_6/gripper100mm/Link2.STL; visual mesh filename=../../meshes/Alicia_D_v5_6/gripper100mm/Link2.STL
- link Link3: geometry collision mesh filename=../../meshes/Alicia_D_v5_6/gripper100mm/Link3.STL; visual mesh filename=../../meshes/Alicia_D_v5_6/gripper100mm/Link3.STL
- link Link4: geometry collision mesh filename=../../meshes/Alicia_D_v5_6/gripper100mm/Link4.STL; visual mesh filename=../../meshes/Alicia_D_v5_6/gripper100mm/Link4.STL
- link Link5: geometry collision mesh filename=../../meshes/Alicia_D_v5_6/gripper100mm/Link5.STL; visual mesh filename=../../meshes/Alicia_D_v5_6/gripper100mm/Link5.STL
- link Link6: geometry collision mesh filename=../../meshes/Alicia_D_v5_6/gripper100mm/Link6.STL; visual mesh filename=../../meshes/Alicia_D_v5_6/gripper100mm/Link6.STL
- link Link7: geometry collision mesh filename=../../meshes/Alicia_D_v5_6/gripper100mm/Link7.STL; visual mesh filename=../../meshes/Alicia_D_v5_6/gripper100mm/Link7.STL
- link Link8: geometry collision mesh filename=../../meshes/Alicia_D_v5_6/gripper100mm/Link8.STL; visual mesh filename=../../meshes/Alicia_D_v5_6/gripper100mm/Link8.STL
- link base_link: geometry collision mesh filename=../../meshes/Alicia_D_v5_6/gripper100mm/base_link.STL; visual mesh filename=../../meshes/Alicia_D_v5_6/gripper100mm/base_link.STL

File: robot_descriptions/urdf/Alicia_D_v5_6/Alicia_D_v5_6_gripper_50mm.urdf (robot description, URDF)
Before this commit: robot Alicia_D_v5_5_gripper_50mm, 11 links, 10 joints
Links:
- link Link1: geometry collision mesh filename=../../meshes/Alicia_D_v5_6/gripper50mm/Link1.STL; visual mesh filename=../../meshes/Alicia_D_v5_6/gripper50mm/Link1.STL
- link Link2: geometry collision mesh filename=../../meshes/Alicia_D_v5_6/gripper50mm/Link2.STL; visual mesh filename=../../meshes/Alicia_D_v5_6/gripper50mm/Link2.STL
- link Link3: geometry collision mesh filename=../../meshes/Alicia_D_v5_6/gripper50mm/Link3.STL; visual mesh filename=../../meshes/Alicia_D_v5_6/gripper50mm/Link3.STL
- link Link4: geometry collision mesh filename=../../meshes/Alicia_D_v5_6/gripper50mm/Link4.STL; visual mesh filename=../../meshes/Alicia_D_v5_6/gripper50mm/Link4.STL
- link Link5: geometry collision mesh filename=../../meshes/Alicia_D_v5_6/gripper50mm/Link5.STL; visual mesh filename=../../meshes/Alicia_D_v5_6/gripper50mm/Link5.STL
- link Link6: geometry collision mesh filename=../../meshes/Alicia_D_v5_6/gripper50mm/Link6.STL; visual mesh filename=../../meshes/Alicia_D_v5_6/gripper50mm/Link6.STL
- link Link7: geometry collision mesh filename=../../meshes/Alicia_D_v5_6/gripper50mm/Link7.STL; visual mesh filename=../../meshes/Alicia_D_v5_6/gripper50mm/Link7.STL
- link Link8: geometry collision mesh filename=../../meshes/Alicia_D_v5_6/gripper50mm/Link8.STL; visual mesh filename=../../meshes/Alicia_D_v5_6/gripper50mm/Link8.STL
- link base_link: geometry collision mesh filename=../../meshes/Alicia_D_v5_6/gripper50mm/base_link.STL; visual mesh filename=../../meshes/Alicia_D_v5_6/gripper50mm/base_link.STL
