Commit message: Update the robot rotation

File: robot_descriptions/urdf/Alicia_D_v5_6/Alicia_D_gripper_100mm.urdf (robot description, URDF)
Before this commit: robot Alicia_D_v5_6_gripper_100mm, 11 links, 10 joints
Links:
- link world: mass 0.001 -> None
Joints:
- removed joint virtual_joint
- added joint world_to_base_joint: type fixed, parent world, child base_link, origin xyz=0 0 0 rpy=0 0 3.14

File: robot_descriptions/urdf/Alicia_D_v5_6/Alicia_D_gripper_50mm.urdf (robot description, URDF)
Before this commit: robot Alicia_D_v5_6_gripper_50mm, 11 links, 10 joints
Links:
- link world: mass 0.001 -> None
Joints:
- removed joint virtual_joint
- added joint world_to_base_joint: type fixed, parent world, child base_link, origin xyz=0 0 0 rpy=0 0 3.14

Commit message: Update Alicia-M v1.0

File: robot_descriptions/urdf/Alicia_D_v5_6/Alicia_D_gripper_100mm.urdf (robot description, URDF)
Before this commit: robot Alicia_D_v5_6_gripper_100mm, 11 links, 10 joints
Links:
- link Link1: geometry collision mesh filename=../../meshes/Alicia_D_v5_6/gripper_100mm/Link1.STL; visual mesh filename=../../meshes/Alicia_D_v5_6/gripper_100mm/Link1.STL
- link Link2: geometry collision mesh filename=../../meshes/Alicia_D_v5_6/gripper_100mm/Link2.STL; visual mesh filename=../../meshes/Alicia_D_v5_6/gripper_100mm/Link2.STL
- link Link3: geometry collision mesh filename=../../meshes/Alicia_D_v5_6/gripper_100mm/Link3.STL; visual mesh filename=../../meshes/Alicia_D_v5_6/gripper_100mm/Link3.STL
- link Link4: geometry collision mesh filename=../../meshes/Alicia_D_v5_6/gripper_100mm/Link4.STL; visual mesh filename=../../meshes/Alicia_D_v5_6/gripper_100mm/Link4.STL
- link Link5: geometry collision mesh filename=../../meshes/Alicia_D_v5_6/gripper_100mm/Link5.STL; visual mesh filename=../../meshes/Alicia_D_v5_6/gripper_100mm/Link5.STL
- link Link6: geometry collision mesh filename=../../meshes/Alicia_D_v5_6/gripper_100mm/Link6.STL; visual mesh filename=../../meshes/Alicia_D_v5_6/gripper_100mm/Link6.STL
- link Link7: geometry collision mesh filename=../../meshes/Alicia_D_v5_6/gripper_100mm/Link7.STL; visual mesh filename=../../meshes/Alicia_D_v5_6/gripper_100mm/Link7.STL
- link Link8: geometry collision mesh filename=../../meshes/Alicia_D_v5_6/gripper_100mm/Link8.STL; visual mesh filename=../../meshes/Alicia_D_v5_6/gripper_100mm/Link8.STL
- link base_link: geometry collision mesh filename=../../meshes/Alicia_D_v5_6/gripper_100mm/base_link.STL; visual mesh filename=../../meshes/Alicia_D_v5_6/gripper_100mm/base_link.STL

File: robot_descriptions/urdf/Alicia_D_v5_6/Alicia_D_gripper_50mm.urdf (robot description, URDF)
Before this commit: robot Alicia_D_v5_6_gripper_50mm, 11 links, 10 joints
Links:
- link Link1: geometry collision mesh filename=../../meshes/Alicia_D_v5_6/gripper_50mm/Link1.STL; visual mesh filename=../../meshes/Alicia_D_v5_6/gripper_50mm/Link1.STL
- link Link2: geometry collision mesh filename=../../meshes/Alicia_D_v5_6/gripper_50mm/Link2.STL; visual mesh filename=../../meshes/Alicia_D_v5_6/gripper_50mm/Link2.STL
- link Link3: geometry collision mesh filename=../../meshes/Alicia_D_v5_6/gripper_50mm/Link3.STL; visual mesh filename=../../meshes/Alicia_D_v5_6/gripper_50mm/Link3.STL
- link Link4: geometry collision mesh filename=../../meshes/Alicia_D_v5_6/gripper_50mm/Link4.STL; visual mesh filename=../../meshes/Alicia_D_v5_6/gripper_50mm/Link4.STL
- link Link5: geometry collision mesh filename=../../meshes/Alicia_D_v5_6/gripper_50mm/Link5.STL; visual mesh filename=../../meshes/Alicia_D_v5_6/gripper_50mm/Link5.STL
- link Link6: geometry collision mesh filename=../../meshes/Alicia_D_v5_6/gripper_50mm/Link6.STL; visual mesh filename=../../meshes/Alicia_D_v5_6/gripper_50mm/Link6.STL
- link Link7: geometry collision mesh filename=../../meshes/Alicia_D_v5_6/gripper_50mm/Link7.STL; visual mesh filename=../../meshes/Alicia_D_v5_6/gripper_50mm/Link7.STL
- link Link8: geometry collision mesh filename=../../meshes/Alicia_D_v5_6/gripper_50mm/Link8.STL; visual mesh filename=../../meshes/Alicia_D_v5_6/gripper_50mm/Link8.STL
- link base_link: geometry collision mesh filename=../../meshes/Alicia_D_v5_6/gripper_50mm/base_link.STL; visual mesh filename=../../meshes/Alicia_D_v5_6/gripper_50mm/base_link.STL

File: robot_descriptions/urdf/Alicia_M_v1_0/Alicia_M_gripper_100mm.urdf (robot description, URDF)
Before this commit: robot Alicia_M_v1_0, 10 links, 9 joints
Links:
- link base_link: geometry collision mesh filename=../../meshes/Alicia_M_v1_0/gripper_100mm/base_link.STL; visual mesh filename=../../meshes/Alicia_M_v1_0/gripper_100mm/base_link.STL
- link grasp_link: geometry collision mesh filename=../../meshes/Alicia_M_v1_0/gripper_100mm/grasp_link.STL; visual mesh filename=../../meshes/Alicia_M_v1_0/gripper_100mm/grasp_link.STL
- link link1: geometry collision mesh filename=../../meshes/Alicia_M_v1_0/gripper_100mm/link1.STL; visual mesh filename=../../meshes/Alicia_M_v1_0/gripper_100mm/link1.STL
- link link2: geometry collision mesh filename=../../meshes/Alicia_M_v1_0/gripper_100mm/link2.STL; visual mesh filename=../../meshes/Alicia_M_v1_0/gripper_100mm/link2.STL
- link link3: geometry collision mesh filename=../../meshes/Alicia_M_v1_0/gripper_100mm/link3.STL; visual mesh filename=../../meshes/Alicia_M_v1_0/gripper_100mm/link3.STL
- link link4: geometry collision mesh filename=../../meshes/Alicia_M_v1_0/gripper_100mm/link4.STL; visual mesh filename=../../meshes/Alicia_M_v1_0/gripper_100mm/link4.STL
- link link5: geometry collision mesh filename=../../meshes/Alicia_M_v1_0/gripper_100mm/link5.STL; visual mesh filename=../../meshes/Alicia_M_v1_0/gripper_100mm/link5.STL
- link link6: geometry collision mesh filename=../../meshes/Alicia_M_v1_0/gripper_100mm/link6.STL; visual mesh filename=../../meshes/Alicia_M_v1_0/gripper_100mm/link6.STL
- link link8: geometry collision mesh filename=../../meshes/Alicia_M_v1_0/gripper_100mm/link8.STL; visual mesh filename=../../meshes/Alicia_M_v1_0/gripper_100mm/link8.STL
- link link9: geometry collision mesh filename=../../meshes/Alicia_M_v1_0/gripper_100mm/link9.STL; visual mesh filename=../../meshes/Alicia_M_v1_0/gripper_100mm/link9.STL
