Commit message: Add gripper center link to bessica

File: synriard/urdf/Bessica_D_v1_0/Bessica_D_v1_0_covered.urdf (robot description, URDF)
Before this commit: robot Bessica_D_v1_0_Covered, 22 links, 21 joints
Links:
- added link left_gripper_center, mass 0.001; visual sphere radius=0.005
- added link right_gripper_center, mass 0.001; visual sphere radius=0.005
Joints:
- added joint left_gripper_center_joint: type fixed, parent left_arm_link7, child left_gripper_center, origin xyz=0.14128 0 0.00015 rpy=0 0 0
- added joint right_gripper_center_joint: type fixed, parent right_arm_link7, child right_gripper_center, origin xyz=0.14128 0 0.00015 rpy=0 0 0
