Commit message: Update the bessica urdf

File: synriard/urdf/Bessica_D_v1_0/Bessica_D_v1_0_covered copy.urdf (robot description, URDF)
Before this commit: robot bessica_d, 24 links, 23 joints
Links:
- removed link head
- added link world, mass 0.001
- link base_link: mass 2.26415289791904 -> 2.26415289785668
- link left_arm_base_link: mass 0.760760214288355 -> 0.760760214227773
- link left_arm_gripper_left_finger: mass 0.0256462689646809 -> 0.0256462690106051
- link left_arm_gripper_right_finger: mass 0.0256462690106051 -> 0.0256462690210739
- link left_arm_link1: mass 0.315733947117255 -> 0.315733967014059
- link left_arm_link2: mass 0.0501482304995307 -> 0.0501482304791557
- link left_arm_link3: mass 0.373333387538863 -> 0.373333384305912
- link left_arm_link4: mass 0.0480071391158089 -> 0.0480071391155924
- link left_arm_link5: mass 0.207077276180107 -> 0.207077278840904
- link left_arm_link6: mass 0.0325622574715583 -> 0.0325622574716532
- link left_arm_link7: mass 0.134233364312826 -> 0.13423336431278
- link left_gripper_center: mass None -> 0.001
- link right_arm_base_link: mass 0.760760214237615 -> 0.760760214227773
- link right_arm_gripper_left_finger: mass 0.0256462690507917 -> 0.0256462690106051
- link right_arm_link1: mass 0.3157339691478 -> 0.315733985052084
- link right_arm_link2: mass 0.0501482304791555 -> 0.0501482304791557
- link right_arm_link3: mass 0.368447313337917 -> 0.368447310994795
- link right_arm_link4: mass 0.048007139134458 -> 0.048007139115809
- link right_arm_link5: mass 0.207077281082729 -> 0.207077276965592
- link right_arm_link6: mass 0.0325622574715594 -> 0.032562257471606
- link right_gripper_center: mass None -> 0.001
Joints:
- removed joint head
- removed joint left_gripper_joint
- removed joint right_gripper_joint
- added joint left_gripper_center_joint: type fixed, parent left_arm_link7, child left_gripper_center, origin xyz=0.14128 0 0.00015 rpy=0 0 0
- added joint right_gripper_center_joint: type fixed, parent right_arm_link7, child right_gripper_center, origin xyz=0.14128 0 0.00015 rpy=0 0 0
- added joint virtual_base_joint: type fixed, parent world, child base_link, origin xyz=0 0 0 rpy=1.5707963267949 0 1.5707963267949, axis 0 0 1, limit lower=-3.14159 upper=3.14159 effort=0 velocity=0
- joint left_arm_base_joint: axis 0 0 0 -> 0 0 1; origin xyz=0 -0.100000000333333 1.01500000133333 rpy=1.5707963267949 0 0 -> xyz=0 1.01500000066667 0.1 rpy=0 0 0
- joint left_arm_gripper_joint1: axis 0 0 0 -> 0 0 1; origin xyz=0.141279659620444 -0.0505000000000146 -0.000149999999993239 rpy=-1.57079632679466 0 0 -> xyz=0.14128 0.0505 0.00015 rpy=1.5708 0 0
- joint left_arm_gripper_joint2: axis 0 0 0 -> 0 0 1; limit (none) -> lower=0 upper=-0.05 effort=5 velocity=12; origin xyz=0.141279659620445 0.0504999999999851 -0.000149999999972228 rpy=1.57079632679513 0 0 -> xyz=0.14128 -0.0505 0.00015 rpy=-1.5708 0 0
- joint left_arm_joint1: axis 0 0 1 -> 0 0 -1; origin xyz=0 0 0.1145 rpy=0 0 0 -> xyz=0 0 0.114499999999998 rpy=0 0 0
- joint left_arm_joint2: axis 0 0 -1 -> 0 0 1; origin xyz=0 0 0.04287 rpy=1.57079632679489 0 1.5707963267949 -> xyz=0 0 0.04287 rpy=1.5707963267949 0 -1.5707963267949
- joint left_arm_joint3: axis 0 0 1 -> 0 0 -1; origin xyz=-0.0657500000000001 -9.99999999995171E-05 -0.000400000003120824 rpy=1.5707963267949 0 -1.5707963267949 -> xyz=0.0657500000000003 -9.99999999993784E-05 0.000400000000008027 rpy=-1.57079632679489 0 -1.5707963267949
- joint left_arm_joint4: origin xyz=0.00383999999999432 0 0.20080999933334 rpy=-1.5707963267949 0 0 -> xyz=0.00384000000000162 0 0.200810000000001 rpy=1.5707963267949 0 0
- joint left_arm_joint5: origin xyz=0 -0.0657500006666611 0.000199999999990721 rpy=-1.5707963267949 0 0 -> xyz=0 0.0657500000000002 -0.000199999999991251 rpy=-1.5707963267949 0 0
- joint left_arm_joint6: axis 0 0 -1 -> 0 0 1; origin xyz=0.00379000000002061 5.00000000002069E-05 -0.17879999933334 rpy=1.5707963267949 0 0 -> xyz=0.00378999999999965 -5.00000000000156E-05 0.1788 rpy=1.5707963267949 0 0
- joint left_arm_joint7: axis 0 0 -1 -> 0 0 1; origin xyz=9.99999999615753E-05 -0.0556000006666605 -9.99999999948057E-05 rpy=-1.57079632679513 0 -1.5707963267949 -> xyz=0.000100000000000044 0.0556 9.99999999912035E-05 rpy=-1.5707963267949 0 1.5707963267949
- joint right_arm_base_joint: axis 0 0 0 -> 0 0 1; origin xyz=0 0.0999999996666618 1.01500000066667 rpy=0 0 0 -> xyz=0 1.01500000066667 -0.1 rpy=3.14159265358979 0 0
- joint right_arm_gripper_joint1: axis 0 0 0 -> 0 0 1; origin xyz=0.141279659620446 -0.0505000000000126 -0.000150000000035122 rpy=-1.57079632679466 0 0 -> xyz=0.14128 0.0505 0.00015 rpy=1.5708 0 0
- joint right_arm_gripper_joint2: axis 0 0 0 -> 0 0 1; origin xyz=0.141279659620446 0.050499999999987 -0.00015000000001425 rpy=1.57079632679513 0 0 -> xyz=0.14128 -0.0505 0.00015 rpy=-1.5708 0 0
- joint right_arm_joint1: axis 0 -1 0 -> 0 0 -1; origin xyz=0 0.114500000000005 0 rpy=3.14159265358979 0 0 -> xyz=0 0 0.1145 rpy=3.14159265358979 0 0
- joint right_arm_joint2: axis 0 0 -1 -> 0 0 1; origin xyz=0 -0.0428699999999995 0 rpy=-3.14159264133724 1.57079625690226 0 -> xyz=0 0 -0.0428699999999988 rpy=-1.5707963267949 0 -1.57079639523237
- joint right_arm_joint3: axis 0 0 1 -> 0 0 -1; origin xyz=-0.0639500000000018 -0.000100000000001099 -0.000399999996885698 rpy=1.57079632679464 0 -1.5707963267949 -> xyz=0.0657499999999946 -9.99999999982126E-05 0.000400000000008029 rpy=1.5707963267949 0 -1.5707963267949
- joint right_arm_joint4: axis 0 0 -1 -> 0 0 1; origin xyz=0.00384000000000018 0 0.20261 rpy=-1.57079632679465 0 0 -> xyz=0.0038400000000019 0 -0.200810000000001 rpy=-1.5707963267949 0 0
- joint right_arm_joint5: origin xyz=0 -0.0639500000000002 0.000199999999992483 rpy=-1.57079632679515 0 0 -> xyz=0 0.0657500000000004 -0.000199999999991113 rpy=1.5707963267949 0 0
- joint right_arm_joint6: origin xyz=0.00378999999999963 5.00000000468472E-05 -0.1806 rpy=1.57079632679515 0 0 -> xyz=0.00378999999999963 5.00000000001502E-05 -0.1788 rpy=-1.5707963267949 0 0
- joint right_arm_joint7: origin xyz=0.000100000000024303 -0.0556000006666655 -9.99999999954217E-05 rpy=-1.57079632679513 0 -1.5707963267949 -> xyz=0.000100000000001432 0.0556 9.99999999912379E-05 rpy=-1.5707963267949 0 1.5707963267949
