Commit message: Update the Vertical Alicia-D

File: synriard/urdf/Alicia_D_v5_6/Alicia_D_v5_6_vertical_50mm.urdf (robot description, URDF)
Before this commit: robot Alicia_D_v5_6_gripper_50mm, 10 links, 9 joints
Links:
- link Link1: mass 0.195233453613076 -> 0.195233494789617; geometry collision mesh filename=../../meshes/Alicia_D_v5_6/vertical/Link1.STL; visual mesh filename=../../meshes/Alicia_D_v5_6/vertical/Link1.STL
- link Link2: mass 0.207033693061784 -> 0.20703369319785; geometry collision mesh filename=../../meshes/Alicia_D_v5_6/vertical/Link2.STL; visual mesh filename=../../meshes/Alicia_D_v5_6/vertical/Link2.STL
- link Link3: mass 0.0845575681430809 -> 0.0845575648033612; geometry collision mesh filename=../../meshes/Alicia_D_v5_6/vertical/Link3.STL; visual mesh filename=../../meshes/Alicia_D_v5_6/vertical/Link3.STL
- link Link4: mass 0.0653695951968861 -> 0.0653695784138105; geometry collision mesh filename=../../meshes/Alicia_D_v5_6/vertical/Link4.STL; visual mesh filename=../../meshes/Alicia_D_v5_6/vertical/Link4.STL
- link Link5: mass 0.0507639016868948 -> 0.0507638951828307; geometry collision mesh filename=../../meshes/Alicia_D_v5_6/vertical/Link5.STL; visual mesh filename=../../meshes/Alicia_D_v5_6/vertical/Link5.STL
- link Link6: mass 0.130364883211194 -> 0.130364815702518; geometry collision mesh filename=../../meshes/Alicia_D_v5_6/vertical/Link6.STL; visual mesh filename=../../meshes/Alicia_D_v5_6/vertical/Link6.STL
- link base_link: mass 0.733961424024115 -> 0.733961424518811; geometry collision mesh filename=../../meshes/Alicia_D_v5_6/vertical/base_link.STL; visual mesh filename=../../meshes/Alicia_D_v5_6/vertical/base_link.STL
- link left_gripper: mass 0.025646112167786 -> 0.0256462690131208; geometry collision mesh filename=../../meshes/Alicia_D_v5_6/vertical/left_gripper.STL; visual mesh filename=../../meshes/Alicia_D_v5_6/vertical/left_gripper.STL
- link right_gripper: mass 0.025646112167786 -> 0.0256462690106051; geometry collision mesh filename=../../meshes/Alicia_D_v5_6/vertical/right_gripper.STL; visual mesh filename=../../meshes/Alicia_D_v5_6/vertical/right_gripper.STL
Joints:
- joint Joint1: axis 0 0 1 -> 0 0 -1; origin xyz=0 0 0.1295 rpy=0 0 0 -> xyz=0.1295 0 0 rpy=0 -1.5708 3.14159
- joint Joint2: limit lower=-1.5708 upper=1.5708 effort=5 velocity=12 -> lower=-0.5 upper=3.14159 effort=5 velocity=12; origin xyz=0 0 0.04287 rpy=1.5708 1.5708 0 -> xyz=0 0 0.0428700000000002 rpy=-1.5707963267949 0 0
- joint Joint3: limit lower=-0.78 upper=3.14 effort=5 velocity=12 -> lower=-2.5 upper=0.8 effort=5 velocity=12; origin xyz=-0.22367 0.022492 -5E-05 rpy=0 0 2.3562 -> xyz=-0.223671302741225 0.0224916129580053 -5.00000000000885E-05 rpy=0 0 -1.5707963267949
- joint Joint4: axis 0 0 -1 -> 0 0 1; origin xyz=-0.00211 -0.099 0.0002 rpy=-1.5708 0 -3.1416 -> xyz=-0.00211000000000214 -0.0990000000000028 0.000200000000000403 rpy=-1.5707963267949 0 0
- joint Joint5: origin xyz=0 -0.0005 0.12235 rpy=-1.5708 0 0 -> xyz=0 -0.000499999999999259 -0.12235 rpy=1.5707963267949 0 3.14159265358979
- joint Joint6: axis 0 0 1 -> 0 0 -1; origin xyz=-0.00385 -0.0575 0.001 rpy=-1.5708 0 0 -> xyz=-0.00384999999999948 -0.0574999999999999 0.000999999999999556 rpy=1.57079632679489 0 0
- joint finger: origin xyz=0.0002 0 -0.13098 rpy=0 0 0 -> xyz=0.0002 0 0.13098 rpy=0 0 0
- joint left_finger: origin xyz=0.000199999999998979 0.0254999999999971 -0.130979659620445 rpy=-1.5707963267949 0 -3.14159265358979 -> xyz=0.000199999999998958 -0.0254999999999972 0.130979659620445 rpy=1.5707963267949 0 3.14159265358979
- joint right_finger: origin xyz=0.0002 -0.0255 -0.13098 rpy=1.5708 0 0 -> xyz=0.000200000000001796 0.0255000000000029 0.130979659620445 rpy=-1.5707963267949 0 0

File: synriard/urdf/Bessica_D_v1_1/Bessica_D_v1_1_skeleton.urdf (robot description, URDF)
Before this commit: robot lingyue_urdf_1.0, 24 links, 21 joints
Links:
- removed link left_gripper_center
- removed link right_gripper_center
- added link left_tool0; visual sphere radius=0.005
- added link right_tool0; visual sphere radius=0.005
- link base_link: mass 2.01690048544311 -> 2.97915154863328
- link head: mass 0.142402684646725 -> 0.14240268640264
- link left_arm_base_link: mass 0.708886467816498 -> 0.708886467098045
- link left_arm_gripper_left_finger: mass 0.0256462691012979 -> 0.025646269010605
- link left_arm_gripper_right_finger: mass 0.0256462691014171 -> 0.025646269010605
- link left_arm_link1: mass 0.197841064757444 -> 0.197841071704829
- link left_arm_link2: mass 0.0472690683067017 -> 0.047269050971783
- link left_arm_link3: mass 0.14045156535093 -> 0.140451564579074
- link left_arm_link4: mass 0.0427207248005301 -> 0.0427207248079551
- link left_arm_link5: mass 0.110396950769399 -> 0.110396951419793
- link left_arm_link6: mass 0.0345706786766195 -> 0.0345706786766011
- link left_arm_link7: mass 0.130827779580124 -> 0.130827779886618
- link right_arm_base_link: mass 0.708886467492412 -> 0.708886467477366
- link right_arm_gripper_left_finger: mass 0.025646269101417 -> 0.0256462690507918
- link right_arm_gripper_right_finger: mass 0.0256462691012978 -> 0.0256462690507921
- link right_arm_link1: mass 0.208265932404293 -> 0.208265932443548
- link right_arm_link2: mass 0.0472690683829237 -> 0.0472690682635543
- link right_arm_link3: mass 0.140451565348764 -> 0.140451564761292
- link right_arm_link4: mass 0.0427207248005302 -> 0.0427207248079551
- link right_arm_link5: mass 0.110396949311228 -> 0.110396949965053
- link right_arm_link6: mass 0.0345706786766193 -> 0.0345706786766012
- link right_arm_link7: mass 0.134443483288705 -> 0.134443483448265
Joints:
- joint head: origin xyz=0.0608245014818929 0.00175926213288763 0.700041453535697 rpy=0 0 0 -> xyz=0.0608244989821353 0.00175926213288549 0.700041453535696 rpy=0 0 0
- joint left_arm_gripper_joint: child left_gripper_center -> left_tool0; origin xyz=0.14128 0.0037519 -0.00015 rpy=3.1416 0 0 -> xyz=0.14058 -0.0041524 0.00015 rpy=0 0 0
- joint left_arm_gripper_joint1: origin xyz=0.14128 -0.046748 -0.00015 rpy=-1.5708 0 0 -> xyz=0.14058 0.046348 0.00015 rpy=1.5708 0 0
- joint left_arm_gripper_joint2: origin xyz=0.14128 0.054252 -0.00015 rpy=1.5708 0 0 -> xyz=0.14058 -0.054652 0.00015 rpy=-1.5708 0 0
- joint left_arm_joint1: limit lower=-2.14 upper=2.14 effort=5 velocity=12 -> lower=-2.749 upper=2.749 effort=5 velocity=12; origin xyz=5.00000000009382E-05 0 0.1146 rpy=0 0 0 -> xyz=4.99975002436759E-05 0 0.1146 rpy=3.14159265358979 0 0
- joint left_arm_joint2: axis 0 0 1 -> 0 0 0.999999999999908; limit lower=-2.14 upper=2.14 effort=5 velocity=12 -> lower=-0.1 upper=3.14159 effort=5 velocity=12; origin xyz=0 0 0.04286 rpy=1.5707963267949 0 1.5707963267949 -> xyz=0 0 -0.04286 rpy=1.5707963267949 0 -1.5707963267949
- joint left_arm_joint3: axis 0 0 -1 -> 0 0 -0.999999999999908; limit lower=-2.14 upper=2.14 effort=5 velocity=12 -> lower=-2.79 upper=2.79 effort=5 velocity=12; origin xyz=-0.0645499999999944 0 0.000300000000004297 rpy=1.5707963267949 0 -1.5707963267949 -> xyz=-0.0645499982324007 0 -0.000299995732645275 rpy=0 -1.5707963267949 0
- joint left_arm_joint4: axis 0 0 -1 -> 0 0 1; limit lower=-2.14 upper=2.14 effort=5 velocity=12 -> lower=-0.5236 upper=2.95 effort=5 velocity=12; origin xyz=-1.89941608861599E-05 -5.00000000028533E-05 0.181600000000001 rpy=-1.5707963267949 0 0 -> xyz=-1.89941608896571E-05 -4.99999999989398E-05 0.1816 rpy=1.57079632191723 -1.57079611188729 0
- joint left_arm_joint5: axis 0 0 1 -> 0 0 -1; limit lower=-2.14 upper=2.14 effort=5 velocity=12 -> lower=-2.79 upper=2.79 effort=5 velocity=12; origin xyz=0 -0.0487999999999995 -9.99999999999612E-05 rpy=-1.5707963267949 0 0 -> xyz=0 -0.0488000000000013 9.99999999971857E-05 rpy=1.5707963267949 1.5707963267949 0
- joint left_arm_joint6: limit lower=-2.14 upper=2.14 effort=5 velocity=12 -> lower=-1.675 upper=1.675 effort=5 velocity=12; origin xyz=0.00288999999999712 0.00207606801469368 -0.10801 rpy=1.5707963267949 0 0 -> xyz=0.00289000000000006 -0.00207606624709478 0.108009995732641 rpy=-1.5707963267949 0 0
- joint left_arm_joint7: limit lower=-2.14 upper=2.14 effort=5 velocity=12 -> lower=-1.448 upper=1.448 effort=5 velocity=12; origin xyz=-0.00150000000000011 -0.0556100008049838 0.00375194992308486 rpy=-1.5707963267949 0 -1.5707963267949 -> xyz=-0.00149999999999997 -0.0563100878103864 0.00415239451449378 rpy=1.5707963267949 0 -1.5707963267949
- joint right_arm_gripper_joint: child right_gripper_center -> right_tool0; origin xyz=0.14128 0 -0.00015 rpy=-3.1416 0 0 -> xyz=0.14128 0 0.00015 rpy=0 0 0
- joint right_arm_gripper_joint1: axis 0 0.054375 -0.99852 -> 0 0 -1; origin xyz=0.14128 0.0505 -0.00015 rpy=1.5708 0 0 -> xyz=0.14128 -0.0505 0.00015 rpy=-1.5708 0 0
- joint right_arm_gripper_joint2: axis 0 -0.054375 0.99852 -> 0 0 1; origin xyz=0.14128 -0.0505 -0.00015 rpy=-1.5708 0 0 -> xyz=0.14128 0.0505 0.00015 rpy=1.5708 0 0
- joint right_arm_joint1: axis 0 1 0 -> 0 -1 0; limit lower=-2.14 upper=2.14 effort=5 velocity=12 -> lower=-2.749 upper=2.749 effort=5 velocity=12; origin xyz=-5.00000000009382E-05 0.1146 0 rpy=3.14159265358979 0 0 -> xyz=-4.9995E-05 -0.1146 0 rpy=0 0 0
- joint right_arm_joint2: axis 0 0 -1 -> 0 0 1; limit lower=-2.14 upper=2.14 effort=5 velocity=12 -> lower=-0.1 upper=3.1416 effort=5 velocity=12; origin xyz=0 -0.0428600000000001 0 rpy=3.14159265358979 1.5707963267949 0 -> xyz=0 -0.04286 0 rpy=0 1.5708 0
- joint right_arm_joint3: axis 0 0 -1 -> 0 0 1; limit lower=-2.14 upper=2.14 effort=5 velocity=12 -> lower=-2.79 upper=2.79 effort=5 velocity=12; origin xyz=-0.0645499999999983 0 0.00030000000000413 rpy=1.5707963267949 0 -1.5707963267949 -> xyz=-0.06455 0 -0.0003 rpy=3.1416 1.5708 0
- joint right_arm_joint4: limit lower=-2.14 upper=2.14 effort=5 velocity=12 -> lower=-0.5236 upper=2.95 effort=5 velocity=12; origin xyz=-1.89941608920163E-05 -5.00000000027701E-05 0.181600000000001 rpy=-1.5707963267949 0 0 -> xyz=-1.8989E-05 -4.9997E-05 0.1816 rpy=1.5708 1.5708 0
- joint right_arm_joint5: limit lower=-2.14 upper=2.14 effort=5 velocity=12 -> lower=-2.79 upper=2.79 effort=5 velocity=12; origin xyz=0 -0.0487999999999997 -0.000100000000000044 rpy=-1.5707963267949 0 0 -> xyz=0 0.0487999946213909 0.000100002721817094 rpy=1.5707963267948 -1.5707963267949 3.14159265358979
- joint right_arm_joint6: axis 0 0 1 -> 0 0 -1; limit lower=-2.14 upper=2.14 effort=5 velocity=12 -> lower=-1.675 upper=1.675 effort=5 velocity=12; origin xyz=0.00288999999999712 0.00207606801469368 -0.10801 rpy=1.5707963267949 0 0 -> xyz=0.00289 -0.0020761 0.10801 rpy=-1.5708 0 0
- joint right_arm_joint7: axis 0 0 -1 -> 0 0 1; limit lower=-2.14 upper=2.14 effort=5 velocity=12 -> lower=-1.448 upper=1.448 effort=5 velocity=12; origin xyz=-0.00149999999999995 -0.05561 0 rpy=-1.57079632065809 0 -1.5707963267949 -> xyz=-0.0015 -0.05561 0 rpy=1.5708 0 -1.5708
