Commit message: Update the joint limitation

File: synriard/urdf/Alicia_D_v5_6/Alicia_D_v5_6_gripper_50mm.urdf (robot description, URDF)
Before this commit: robot Alicia_D_v5_6_gripper_50mm, 10 links, 9 joints
Joints:
- joint Joint2: limit lower=-1.5708 upper=1.5708 effort=5 velocity=12 -> lower=-2 upper=2 effort=5 velocity=12
- joint Joint3: limit lower=-0.78 upper=3.14 effort=5 velocity=12 -> lower=-0.5 upper=3.14159 effort=5 velocity=12
- joint Joint6: limit lower=-3.14 upper=3.14 effort=5 velocity=12 -> lower=-3.14159 upper=3.14159 effort=5 velocity=12

File: synriard/urdf/Alicia_D_v5_6/Alicia_D_v5_6_leader.urdf (robot description, URDF)
Before this commit: robot Alicia_D_v5_6_leader, 7 links, 6 joints
Joints:
- joint joint1: limit lower=-2.8 upper=2.8 effort=5 velocity=10 -> lower=-2.749 upper=2.749 effort=5 velocity=10
- joint joint3: limit lower=-0.79 upper=1.57 effort=5 velocity=10 -> lower=-0.6 upper=2.2 effort=5 velocity=10
- joint joint4: limit lower=-2.8 upper=2.8 effort=5 velocity=10 -> lower=-2.79 upper=2.79 effort=5 velocity=10
- joint joint5: limit lower=-1.75 upper=1.75 effort=5 velocity=10 -> lower=-1.57 upper=1.57 effort=5 velocity=10
- joint joint6: limit lower=-3.14 upper=3.14 effort=5 velocity=10 -> lower=-3.14159 upper=3.14159 effort=5 velocity=10

File: synriard/urdf/Alicia_D_v5_6/Alicia_D_v5_6_vertical_50mm.urdf (robot description, URDF)
Before this commit: robot Alicia_D_v5_6_vertical_50mm, 10 links, 9 joints
Joints:
- joint Joint6: limit lower=-3.14 upper=3.14 effort=5 velocity=12 -> lower=-3.14159 upper=3.14159 effort=5 velocity=12
