Commit message: Refactor all models follow {name}_{version}_{variant} naming convention

File: synriard/urdf/Alicia_D_v5_6/Alicia_D_v5_6_gripper_100mm.urdf (robot description, URDF)
Before this commit: robot Alicia_D_v5_6_gripper_50mm, 11 links, 10 joints
Links:
- link Link1: mass 0.195233452997327 -> 0.195233452997315; geometry collision mesh filename=../../meshes/Alicia_D_v5_6/gripper_100mm/Link1.STL; visual mesh filename=../../meshes/Alicia_D_v5_6/gripper_100mm/Link1.STL
- link Link2: mass 0.207033693061786 -> 0.207033693061785; geometry collision mesh filename=../../meshes/Alicia_D_v5_6/gripper_100mm/Link2.STL; visual mesh filename=../../meshes/Alicia_D_v5_6/gripper_100mm/Link2.STL
- link Link3: mass 0.0845575636182319 -> 0.0845575643881719; geometry collision mesh filename=../../meshes/Alicia_D_v5_6/gripper_100mm/Link3.STL; visual mesh filename=../../meshes/Alicia_D_v5_6/gripper_100mm/Link3.STL
- link Link4: mass 0.0653695953286769 -> 0.0653695983290511; geometry collision mesh filename=../../meshes/Alicia_D_v5_6/gripper_100mm/Link4.STL; visual mesh filename=../../meshes/Alicia_D_v5_6/gripper_100mm/Link4.STL
- link Link5: mass 0.0507639016939355 -> 0.0507639016939435; geometry collision mesh filename=../../meshes/Alicia_D_v5_6/gripper_100mm/Link5.STL; visual mesh filename=../../meshes/Alicia_D_v5_6/gripper_100mm/Link5.STL
- link Link6: mass 0.130364883326573 -> 0.123298967748658; geometry collision mesh filename=../../meshes/Alicia_D_v5_6/gripper_100mm/Link6.STL; visual mesh filename=../../meshes/Alicia_D_v5_6/gripper_100mm/Link6.STL
- link Link7: geometry collision mesh filename=../../meshes/Alicia_D_v5_6/gripper_100mm/Link7.STL; visual mesh filename=../../meshes/Alicia_D_v5_6/gripper_100mm/Link7.STL
- link Link8: mass 0.0256461121677874 -> 0.0256461121677875; geometry collision mesh filename=../../meshes/Alicia_D_v5_6/gripper_100mm/Link8.STL; visual mesh filename=../../meshes/Alicia_D_v5_6/gripper_100mm/Link8.STL
- link base_link: geometry collision mesh filename=../../meshes/Alicia_D_v5_6/gripper_100mm/base_link.STL; visual mesh filename=../../meshes/Alicia_D_v5_6/gripper_100mm/base_link.STL
Joints:
- joint Joint6: origin xyz=-0.00385 -0.0575 0.001 rpy=1.5708 0 0 -> xyz=-0.00384999999999946 -0.0574999999999999 0.00100000000000069 rpy=1.5707963267949 0 0
- joint left_finger: limit lower=-0.025 upper=0 effort=5 velocity=10 -> lower=-0.05 upper=0 effort=5 velocity=12; origin xyz=0.0002 -0.025469 0.13098 rpy=1.5708 0 0 -> xyz=-0.0002 -0.036537 0.13098 rpy=1.5708 0 0
- joint right_finger: limit lower=0 upper=0.025 effort=5 velocity=10 -> lower=0 upper=0.05 effort=5 velocity=12; origin xyz=0.0002 0.025469 0.13098 rpy=-1.5708 0 0 -> xyz=-0.0002 0.036518 0.13098 rpy=-1.5708 0 0

File: synriard/urdf/Alicia_D_v5_6/Alicia_D_v5_6_gripper_50mm.urdf (robot description, URDF)
Before this commit: robot Alicia_D_v5_6_gripper_100mm, 11 links, 10 joints
Links:
- link Link1: mass 0.195233452997315 -> 0.195233452997327; geometry collision mesh filename=../../meshes/Alicia_D_v5_6/gripper_50mm/Link1.STL; visual mesh filename=../../meshes/Alicia_D_v5_6/gripper_50mm/Link1.STL
- link Link2: mass 0.207033693061785 -> 0.207033693061786; geometry collision mesh filename=../../meshes/Alicia_D_v5_6/gripper_50mm/Link2.STL; visual mesh filename=../../meshes/Alicia_D_v5_6/gripper_50mm/Link2.STL
- link Link3: mass 0.0845575643881719 -> 0.0845575636182319; geometry collision mesh filename=../../meshes/Alicia_D_v5_6/gripper_50mm/Link3.STL; visual mesh filename=../../meshes/Alicia_D_v5_6/gripper_50mm/Link3.STL
- link Link4: mass 0.0653695983290511 -> 0.0653695953286769; geometry collision mesh filename=../../meshes/Alicia_D_v5_6/gripper_50mm/Link4.STL; visual mesh filename=../../meshes/Alicia_D_v5_6/gripper_50mm/Link4.STL
- link Link5: mass 0.0507639016939435 -> 0.0507639016939355; geometry collision mesh filename=../../meshes/Alicia_D_v5_6/gripper_50mm/Link5.STL; visual mesh filename=../../meshes/Alicia_D_v5_6/gripper_50mm/Link5.STL
- link Link6: mass 0.123298967748658 -> 0.130364883326573; geometry collision mesh filename=../../meshes/Alicia_D_v5_6/gripper_50mm/Link6.STL; visual mesh filename=../../meshes/Alicia_D_v5_6/gripper_50mm/Link6.STL
- link Link7: geometry collision mesh filename=../../meshes/Alicia_D_v5_6/gripper_50mm/Link7.STL; visual mesh filename=../../meshes/Alicia_D_v5_6/gripper_50mm/Link7.STL
- link Link8: mass 0.0256461121677875 -> 0.0256461121677874; geometry collision mesh filename=../../meshes/Alicia_D_v5_6/gripper_50mm/Link8.STL; visual mesh filename=../../meshes/Alicia_D_v5_6/gripper_50mm/Link8.STL
- link base_link: geometry collision mesh filename=../../meshes/Alicia_D_v5_6/gripper_50mm/base_link.STL; visual mesh filename=../../meshes/Alicia_D_v5_6/gripper_50mm/base_link.STL
Joints:
- joint Joint6: origin xyz=-0.00384999999999946 -0.0574999999999999 0.00100000000000069 rpy=1.5707963267949 0 0 -> xyz=-0.00385 -0.0575 0.001 rpy=1.5708 0 0
- joint left_finger: limit lower=-0.05 upper=0 effort=5 velocity=12 -> lower=-0.025 upper=0 effort=5 velocity=10; origin xyz=-0.0002 -0.036537 0.13098 rpy=1.5708 0 0 -> xyz=0.0002 -0.025469 0.13098 rpy=1.5708 0 0
- joint right_finger: limit lower=0 upper=0.05 effort=5 velocity=12 -> lower=0 upper=0.025 effort=5 velocity=10; origin xyz=-0.0002 0.036518 0.13098 rpy=-1.5708 0 0 -> xyz=0.0002 0.025469 0.13098 rpy=-1.5708 0 0

Commit message: Update Alicia-D V5.6 with gripper range fix

File: synriard/urdf/Alicia_D_v5_6/Alicia_D_v5_6_gripper_100mm.urdf (robot description, URDF)
Before this commit: robot Alicia_D_v5_6_gripper_100mm, 11 links, 10 joints
Links:
- removed link Link7
- removed link Link8
- removed link tool0
- removed link world
- added link gripper_center; visual sphere radius=0.005
- added link left_gripper, mass 0.025646111367227; collision mesh filename=../../meshes/Alicia_D_v5_6/gripper_100mm/left_gripper.STL; visual mesh filename=../../meshes/Alicia_D_v5_6/gripper_100mm/left_gripper.STL
- added link right_gripper, mass 0.0256461131643355; collision mesh filename=../../meshes/Alicia_D_v5_6/gripper_100mm/right_gripper.STL; visual mesh filename=../../meshes/Alicia_D_v5_6/gripper_100mm/right_gripper.STL
- link Link1: mass 0.195233452997315 -> 0.195233452997321
- link Link2: mass 0.207033693061785 -> 0.20703368934203
- link Link3: mass 0.0845575643881719 -> 0.0845575626224312
- link Link4: mass 0.0653695983290511 -> 0.0653695946193964
- link Link5: mass 0.0507639016939435 -> 0.0507639007674356
- link Link6: mass 0.123298967748658 -> 0.123436287808883
- link base_link: mass 0.73396142463988 -> 0.733961424639881
Joints:
- removed joint Grasp2tool
- removed joint left_finger
- removed joint right_finger
- removed joint world_to_base_joint
- added joint LGripper: type prismatic, parent Link6, child left_gripper, origin xyz=-0.000200000000001033 -0.050497849845622 0.130979659620446 rpy=1.5707963267949 0 0, axis 0 0 -1, limit lower=0 upper=0.05 effort=5 velocity=12
- added joint RGripper: type prismatic, parent Link6, child right_gripper, origin xyz=-0.0002 0.050502 0.13098 rpy=-1.5708 0 0, axis 0 0 1, limit lower=-0.05 upper=0 effort=5 velocity=12
- added joint finger: type fixed, parent Link6, child gripper_center, origin xyz=-0.0002 0 0.13048 rpy=0 0 0, axis 0 0 0
- joint Joint1: axis 0 0 1 -> -0.0397713509246861 0 -0.999208806829496; limit lower=-2.16 upper=2.16 effort=5 velocity=12 -> lower=-2.7925 upper=2.7525 effort=5 velocity=12; origin xyz=0 0 0.1295 rpy=0 0 0 -> xyz=0 0 0.1295 rpy=0 -0.0397818431857344 0
- joint Joint2: axis 0 0 -1 -> 0 0 1; limit lower=-1.57 upper=1.57 effort=5 velocity=12 -> lower=-2 upper=2 effort=5 velocity=12; origin xyz=0 0 0.0428699999999999 rpy=1.5707963267949 -1.5707963267949 0 -> xyz=0.00170499781414124 0 0.0428360815487805 rpy=1.5707963267949 -1.5707963267949 0
- joint Joint3: axis 0 0 -1 -> 0 0 1; limit lower=-0.5 upper=2.35619 effort=5 velocity=12 -> lower=-2.8 upper=0.38 effort=5 velocity=12; origin xyz=0.223671302741224 0.0225916129580062 -5.00000000004269E-05 rpy=0 0 -2.35619455367747 -> xyz=0.223671302741224 0.0226916129580064 -4.99999999962493E-05 rpy=0 0 -2.35619449019234
- joint Joint4: axis 0 0 1 -> 0 0 -1; origin xyz=0.00211000000000205 -0.0990000000000029 -0.000199999999999935 rpy=1.5707963267949 0 -3.14159265358979 -> xyz=0.00211000000000178 -0.0990000000000033 -0.0002000000000025 rpy=1.5707963267949 0 0
- joint Joint5: axis 0 0 -1 -> 0 0 1; limit lower=-1.57 upper=1.57 effort=5 velocity=12 -> lower=-1.5 upper=1.5 effort=5 velocity=12; origin xyz=0 -0.000500000000000358 -0.12235 rpy=1.5707963267949 0 3.14159265358979 -> xyz=0 -0.000500000000001193 0.12235 rpy=1.5707963267949 0 0
- joint Joint6: origin xyz=-0.00384999999999946 -0.0574999999999999 0.00100000000000069 rpy=1.5707963267949 0 0 -> xyz=-0.00384999999999935 0.0574999999999998 -0.00100000000000219 rpy=-1.5707963267949 0 0

File: synriard/urdf/Alicia_D_v5_6/Alicia_D_v5_6_gripper_50mm.urdf (robot description, URDF)
Before this commit: robot Alicia_D_v5_6_gripper_50mm, 11 links, 10 joints
Links:
- removed link Link7
- removed link Link8
- removed link tool0
- removed link world
- added link gripper_center; visual sphere radius=0.005
- added link left_gripper, mass 0.0256461113672271; collision mesh filename=../../meshes/Alicia_D_v5_6/gripper_50mm/left_gripper.STL; visual mesh filename=../../meshes/Alicia_D_v5_6/gripper_50mm/left_gripper.STL
- added link right_gripper, mass 0.0256461131643356; collision mesh filename=../../meshes/Alicia_D_v5_6/gripper_50mm/right_gripper.STL; visual mesh filename=../../meshes/Alicia_D_v5_6/gripper_50mm/right_gripper.STL
- link Link1: mass 0.195233452997327 -> 0.195233452997321
- link Link2: mass 0.207033693061786 -> 0.207033689183231
- link Link3: mass 0.0845575636182319 -> 0.084557560592733
- link Link4: mass 0.0653695953286769 -> 0.0653695946194211
- link Link5: mass 0.0507639016939355 -> 0.0507639007674435
- link Link6: mass 0.130364883326573 -> 0.130364885866405
- link base_link: mass 0.73396142463988 -> 0.733961424639881
Joints:
- removed joint Grasp2tool
- removed joint left_finger
- removed joint right_finger
- removed joint world_to_base_joint
- added joint LGripper: type prismatic, parent Link6, child left_gripper, origin xyz=0.0002 -0.0255 0.13098 rpy=1.5708 0 0, axis 0 0 -1, limit lower=0 upper=0.025 effort=5 velocity=12
- added joint RGripper: type prismatic, parent Link6, child right_gripper, origin xyz=0.0002 0.0255 0.13098 rpy=-1.5708 0 0, axis 0 0 1, limit lower=-0.025 upper=0 effort=5 velocity=12
- added joint finger: type fixed, parent Link6, child gripper_center, origin xyz=0.0002 0 0.13098 rpy=0 0 0, axis 0 0 0
- joint Joint1: axis 0 0 1 -> -0.0397713509246861 0 -0.999208806829496; limit lower=-2.16 upper=2.16 effort=5 velocity=12 -> lower=-2.7925 upper=2.7525 effort=5 velocity=12; origin xyz=0 0 0.1295 rpy=0 0 0 -> xyz=0 0 0.1295 rpy=0 -0.0397818431857344 0
- joint Joint2: axis 0 0 -1 -> 0 0 1; limit lower=-1.57 upper=1.57 effort=5 velocity=12 -> lower=-2 upper=2 effort=5 velocity=12; origin xyz=0 0 0.0428699999999999 rpy=1.5707963267949 -1.5707963267949 0 -> xyz=0.00170499781414124 0 0.0428360815487805 rpy=1.5707963267949 -1.5707963267949 0
- joint Joint3: axis 0 0 -1 -> 0 0 1; limit lower=-0.5 upper=2.35619 effort=5 velocity=12 -> lower=-2.8 upper=0.38 effort=5 velocity=12; origin xyz=0.223671302741224 0.0225916129580062 -5.00000000004269E-05 rpy=0 0 -2.35619455367747 -> xyz=0.223671302741224 0.0226916129580064 -4.99999999962493E-05 rpy=0 0 -2.35619449019234
- joint Joint4: axis 0 0 1 -> 0 0 -1; origin xyz=0.00211000000000205 -0.0990000000000029 -0.000199999999999935 rpy=1.5707963267949 0 -3.14159265358979 -> xyz=0.00211000000000178 -0.0990000000000033 -0.0002000000000025 rpy=1.5707963267949 0 0
- joint Joint5: axis 0 0 -1 -> 0 0 1; limit lower=-1.57 upper=1.57 effort=5 velocity=12 -> lower=-1.5 upper=1.5 effort=5 velocity=12; origin xyz=0 -0.000500000000000358 -0.12235 rpy=1.5707963267949 0 3.14159265358979 -> xyz=0 -0.000500000000001193 0.12235 rpy=1.5707963267949 0 0
- joint Joint6: origin xyz=-0.00385 -0.0575 0.001 rpy=1.5708 0 0 -> xyz=-0.00384999999999935 0.0574999999999998 -0.00100000000000219 rpy=-1.5707963267949 0 0

Commit message: Update the Alicia-D v5.6 version

File: synriard/urdf/Alicia_D_v5_6/Alicia_D_v5_6_gripper_100mm.urdf (robot description, URDF)
Before this commit: robot Alicia_D_v5_6_gripper_100mm, 10 links, 9 joints
Links:
- removed link gripper_center
- added link tool0; visual sphere radius=0.005
- link Link1: mass 0.195233452997321 -> 0.195233495556057
- link Link2: mass 0.20703368934203 -> 0.207033693066089
- link Link3: mass 0.0845575626224312 -> 0.0845575651613574
- link Link4: mass 0.0653695946193964 -> 0.0653695951425785
- link Link5: mass 0.0507639007674356 -> 0.050763902309721
- link Link6: mass 0.123436287808883 -> 0.119820573151617
- link base_link: mass 0.733961424639881 -> 0.733961424954529
- link left_gripper: mass 0.025646111367227 -> 0.0256461121677845
- link right_gripper: mass 0.0256461131643355 -> 0.0256461121677874
Joints:
- removed joint LGripper
- removed joint RGripper
- added joint left_finger: type prismatic, parent Link6, child left_gripper, origin xyz=-0.000200000000001088 -0.050497849845622 0.130979659620446 rpy=1.5707963267949 0 3.14159265358979, axis 0 0 1, limit lower=0 upper=0.05 effort=5 velocity=12
- added joint right_finger: type prismatic, parent Link6, child right_gripper, origin xyz=-0.000199999999998035 0.050502150154378 0.130979659620446 rpy=-1.5707963267949 0 3.14159265358978, axis 0 0 -1, limit lower=-0.05 upper=0 effort=5 velocity=12
- joint Joint1: axis -0.0397713509246861 0 -0.999208806829496 -> 0 0 1; limit lower=-2.7925 upper=2.7525 effort=5 velocity=12 -> lower=-2.749 upper=2.749 effort=5 velocity=12; origin xyz=0 0 0.1295 rpy=0 -0.0397818431857344 0 -> xyz=0 0 0.1295 rpy=0 0 0
- joint Joint2: origin xyz=0.00170499781414124 0 0.0428360815487805 rpy=1.5707963267949 -1.5707963267949 0 -> xyz=0 0 0.04287 rpy=1.5708 1.5708 0
- joint Joint3: limit lower=-2.8 upper=0.38 effort=5 velocity=12 -> lower=-0.5 upper=3.14159 effort=5 velocity=12; origin xyz=0.223671302741224 0.0226916129580064 -4.99999999962493E-05 rpy=0 0 -2.35619449019234 -> xyz=-0.22367 0.022492 -5E-05 rpy=0 0 2.3562
- joint Joint4: axis 0 0 -1 -> 0 0 1; limit lower=-2.7925 upper=2.7925 effort=5 velocity=12 -> lower=-2.79 upper=2.79 effort=5 velocity=12; origin xyz=0.00211000000000178 -0.0990000000000033 -0.0002000000000025 rpy=1.5707963267949 0 0 -> xyz=-0.00211 -0.099 0.0002 rpy=-1.5708 0 0
- joint Joint5: axis 0 0 1 -> 0 0 -1; limit lower=-1.5 upper=1.5 effort=5 velocity=12 -> lower=-1.57 upper=1.57 effort=5 velocity=12; origin xyz=0 -0.000500000000001193 0.12235 rpy=1.5707963267949 0 0 -> xyz=0 -0.0005 -0.12235 rpy=1.5708 0 -3.1416
- joint Joint6: limit lower=-3.14 upper=3.14 effort=5 velocity=12 -> lower=-3.14159 upper=3.14159 effort=5 velocity=12; origin xyz=-0.00384999999999935 0.0574999999999998 -0.00100000000000219 rpy=-1.5707963267949 0 0 -> xyz=-0.00385 -0.0575 0.001 rpy=1.5708 0 0
- joint finger: child gripper_center -> tool0; origin xyz=-0.0002 0 0.13048 rpy=0 0 0 -> xyz=-0.0002 0 0.13098 rpy=0 0 0

Commit message: Merge gripper 50mm and 100mm stl files.

File: synriard/urdf/Alicia_D_v5_6/Alicia_D_v5_6_gripper_100mm.urdf (robot description, URDF)
Before this commit: robot Alicia_D_v5_6_gripper_100mm, 10 links, 9 joints
Links:
- link Link1: geometry collision mesh filename=../../meshes/Alicia_D_v5_6/follower_standard/Link1.STL; visual mesh filename=../../meshes/Alicia_D_v5_6/follower_standard/Link1.STL
- link Link2: geometry collision mesh filename=../../meshes/Alicia_D_v5_6/follower_standard/Link2.STL; visual mesh filename=../../meshes/Alicia_D_v5_6/follower_standard/Link2.STL
- link Link3: geometry collision mesh filename=../../meshes/Alicia_D_v5_6/follower_standard/Link3.STL; visual mesh filename=../../meshes/Alicia_D_v5_6/follower_standard/Link3.STL
- link Link4: geometry collision mesh filename=../../meshes/Alicia_D_v5_6/follower_standard/Link4.STL; visual mesh filename=../../meshes/Alicia_D_v5_6/follower_standard/Link4_100mm.STL
- link Link5: geometry collision mesh filename=../../meshes/Alicia_D_v5_6/follower_standard/Link5.STL; visual mesh filename=../../meshes/Alicia_D_v5_6/follower_standard/Link5.STL
- link Link6: geometry collision mesh filename=../../meshes/Alicia_D_v5_6/follower_standard/Link6.STL; visual mesh filename=../../meshes/Alicia_D_v5_6/follower_standard/Link6_100mm.STL
- link base_link: geometry collision mesh filename=../../meshes/Alicia_D_v5_6/follower_standard/base_link.STL; visual mesh filename=../../meshes/Alicia_D_v5_6/follower_standard/base_link.STL
- link left_gripper: geometry collision mesh filename=../../meshes/Alicia_D_v5_6/follower_standard/left_gripper_1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; visual mesh filename=../../meshes/Alicia_D_v5_6/follower_standard/left_gripper_1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
- link right_gripper: geometry collision mesh filename=../../meshes/Alicia_D_v5_6/follower_standard/right_gripper_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; visual mesh filename=../../meshes/Alicia_D_v5_6/follower_standard/right_gripper_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

File: synriard/urdf/Alicia_D_v5_6/Alicia_D_v5_6_gripper_50mm.urdf (robot description, URDF)
Before this commit: robot Alicia_D_v5_6_gripper_50mm, 10 links, 9 joints
Links:
- link Link1: geometry collision mesh filename=../../meshes/Alicia_D_v5_6/follower_standard/Link1.STL; visual mesh filename=../../meshes/Alicia_D_v5_6/follower_standard/Link1.STL
- link Link2: geometry collision mesh filename=../../meshes/Alicia_D_v5_6/follower_standard/Link2.STL; visual mesh filename=../../meshes/Alicia_D_v5_6/follower_standard/Link2.STL
- link Link3: geometry collision mesh filename=../../meshes/Alicia_D_v5_6/follower_standard/Link3.STL; visual mesh filename=../../meshes/Alicia_D_v5_6/follower_standard/Link3.STL
- link Link4: geometry collision mesh filename=../../meshes/Alicia_D_v5_6/follower_standard/Link4.STL; visual mesh filename=../../meshes/Alicia_D_v5_6/follower_standard/Link4.STL
- link Link5: geometry collision mesh filename=../../meshes/Alicia_D_v5_6/follower_standard/Link5.STL; visual mesh filename=../../meshes/Alicia_D_v5_6/follower_standard/Link5.STL
- link Link6: geometry collision mesh filename=../../meshes/Alicia_D_v5_6/follower_standard/Link6.STL; visual mesh filename=../../meshes/Alicia_D_v5_6/follower_standard/Link6.STL
- link base_link: geometry collision mesh filename=../../meshes/Alicia_D_v5_6/follower_standard/base_link.STL; visual mesh filename=../../meshes/Alicia_D_v5_6/follower_standard/base_link.STL
- link left_gripper: geometry collision mesh filename=../../meshes/Alicia_D_v5_6/follower_standard/left_gripper_5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; visual mesh filename=../../meshes/Alicia_D_v5_6/follower_standard/left_gripper_5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
- link right_gripper: geometry collision mesh filename=../../meshes/Alicia_D_v5_6/follower_standard/right_gripper_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; visual mesh filename=../../meshes/Alicia_D_v5_6/follower_standard/right_gripper_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

Commit message: Update Alicia-D v5.6 & Alicia-M v1.1

File: synriard/urdf/Alicia_D_v5_6/Alicia_D_v5_6_gripper_100mm.urdf (robot description, URDF)
Before this commit: robot Alicia_D_v5_6_gripper_100mm, 10 links, 9 joints
Links:
- link Link4: geometry collision mesh filename=../../meshes/Alicia_D_v5_6/follower_standard/Link4_100mm.STL; visual mesh filename=../../meshes/Alicia_D_v5_6/follower_standard/Link4_100mm.STL
- link Link6: geometry collision mesh filename=../../meshes/Alicia_D_v5_6/follower_standard/Link6_100mm.STL; visual mesh filename=../../meshes/Alicia_D_v5_6/follower_standard/Link6_100mm.STL
