Commit message: Unified mesh names

File: synriard/urdf/Alicia_D_v5_6/Alicia_D_v5_6_gripper_100mm.urdf (robot description, URDF)
Before this commit: robot Alicia_D_v5_6_gripper_100mm, 10 links, 9 joints
Links:
- removed link Link1
- removed link Link2
- removed link Link3
- removed link Link4
- removed link Link5
- removed link Link6
- added link link1, mass 0.195233495556057; collision mesh filename=../../meshes/Alicia_D_v5_6/follower_standard/link1.STL; visual mesh filename=../../meshes/Alicia_D_v5_6/follower_standard/link1.STL
- added link link2, mass 0.207033693066089; collision mesh filename=../../meshes/Alicia_D_v5_6/follower_standard/link2.STL; visual mesh filename=../../meshes/Alicia_D_v5_6/follower_standard/link2.STL
- added link link3, mass 0.0845575651613574; collision mesh filename=../../meshes/Alicia_D_v5_6/follower_standard/link3.STL; visual mesh filename=../../meshes/Alicia_D_v5_6/follower_standard/link3.STL
- added link link4, mass 0.0653695951425785; collision mesh filename=../../meshes/Alicia_D_v5_6/follower_standard/link4_100mm.STL; visual mesh filename=../../meshes/Alicia_D_v5_6/follower_standard/link4_100mm.STL
- added link link5, mass 0.050763902309721; collision mesh filename=../../meshes/Alicia_D_v5_6/follower_standard/link5.STL; visual mesh filename=../../meshes/Alicia_D_v5_6/follower_standard/link5.STL
- added link link6, mass 0.119820573151617; collision mesh filename=../../meshes/Alicia_D_v5_6/follower_standard/link6_100mm.STL; visual mesh filename=../../meshes/Alicia_D_v5_6/follower_standard/link6_100mm.STL
Joints:
- joint Joint1: child Link1 -> link1
- joint Joint2: child Link2 -> link2; parent Link1 -> link1
- joint Joint3: child Link3 -> link3; parent Link2 -> link2
- joint Joint4: child Link4 -> link4; parent Link3 -> link3
- joint Joint5: child Link5 -> link5; parent Link4 -> link4
- joint Joint6: child Link6 -> link6; parent Link5 -> link5
- joint finger: parent Link6 -> link6
- joint left_finger: parent Link6 -> link6
- joint right_finger: parent Link6 -> link6

File: synriard/urdf/Alicia_D_v5_6/Alicia_D_v5_6_gripper_50mm.urdf (robot description, URDF)
Before this commit: robot Alicia_D_v5_6_gripper_50mm, 10 links, 9 joints
Links:
- removed link Link1
- removed link Link2
- removed link Link3
- removed link Link4
- removed link Link5
- removed link Link6
- added link link1, mass 0.195233453613076; collision mesh filename=../../meshes/Alicia_D_v5_6/follower_standard/link1.STL; visual mesh filename=../../meshes/Alicia_D_v5_6/follower_standard/link1.STL
- added link link2, mass 0.207033693061784; collision mesh filename=../../meshes/Alicia_D_v5_6/follower_standard/link2.STL; visual mesh filename=../../meshes/Alicia_D_v5_6/follower_standard/link2.STL
- added link link3, mass 0.0845575681430809; collision mesh filename=../../meshes/Alicia_D_v5_6/follower_standard/link3.STL; visual mesh filename=../../meshes/Alicia_D_v5_6/follower_standard/link3.STL
- added link link4, mass 0.0653695951968861; collision mesh filename=../../meshes/Alicia_D_v5_6/follower_standard/link4.STL; visual mesh filename=../../meshes/Alicia_D_v5_6/follower_standard/link4.STL
- added link link5, mass 0.0507639016868948; collision mesh filename=../../meshes/Alicia_D_v5_6/follower_standard/link5.STL; visual mesh filename=../../meshes/Alicia_D_v5_6/follower_standard/link5.STL
- added link link6, mass 0.130364883211194; collision mesh filename=../../meshes/Alicia_D_v5_6/follower_standard/link6.STL; visual mesh filename=../../meshes/Alicia_D_v5_6/follower_standard/link6.STL
Joints:
- joint Joint1: child Link1 -> link1
- joint Joint2: child Link2 -> link2; parent Link1 -> link1
- joint Joint3: child Link3 -> link3; parent Link2 -> link2
- joint Joint4: child Link4 -> link4; parent Link3 -> link3
- joint Joint5: child Link5 -> link5; parent Link4 -> link4
- joint Joint6: child Link6 -> link6; parent Link5 -> link5
- joint finger: parent Link6 -> link6
- joint left_finger: parent Link6 -> link6
- joint right_finger: parent Link6 -> link6

File: synriard/urdf/Alicia_D_v5_6/Alicia_D_v5_6_vertical_50mm.urdf (robot description, URDF)
Before this commit: robot Alicia_D_v5_6_vertical_50mm, 10 links, 9 joints
Links:
- removed link Link1
- removed link Link2
- removed link Link3
- removed link Link4
- removed link Link5
- removed link Link6
- added link link1, mass 0.195233494789617; collision mesh filename=../../meshes/Alicia_D_v5_6/vertical/link1.STL; visual mesh filename=../../meshes/Alicia_D_v5_6/vertical/link1.STL
- added link link2, mass 0.20703369319785; collision mesh filename=../../meshes/Alicia_D_v5_6/vertical/link2.STL; visual mesh filename=../../meshes/Alicia_D_v5_6/vertical/link2.STL
- added link link3, mass 0.0845575648033612; collision mesh filename=../../meshes/Alicia_D_v5_6/vertical/link3.STL; visual mesh filename=../../meshes/Alicia_D_v5_6/vertical/link3.STL
- added link link4, mass 0.0653695784138105; collision mesh filename=../../meshes/Alicia_D_v5_6/vertical/link4.STL; visual mesh filename=../../meshes/Alicia_D_v5_6/vertical/link4.STL
- added link link5, mass 0.0507638951828307; collision mesh filename=../../meshes/Alicia_D_v5_6/vertical/link5.STL; visual mesh filename=../../meshes/Alicia_D_v5_6/vertical/link5.STL
- added link link6, mass 0.130364815702518; collision mesh filename=../../meshes/Alicia_D_v5_6/vertical/link6.STL; visual mesh filename=../../meshes/Alicia_D_v5_6/vertical/link6.STL
Joints:
- joint Joint1: child Link1 -> link1
- joint Joint2: child Link2 -> link2; parent Link1 -> link1
- joint Joint3: child Link3 -> link3; parent Link2 -> link2
- joint Joint4: child Link4 -> link4; parent Link3 -> link3
- joint Joint5: child Link5 -> link5; parent Link4 -> link4
- joint Joint6: child Link6 -> link6; parent Link5 -> link5
- joint finger: parent Link6 -> link6
- joint left_finger: parent Link6 -> link6
- joint right_finger: parent Link6 -> link6
