Commit message: Add force feedback leader arm

File: synriard/urdf/Alicia_D_v5_6/Alicia_D_v5_6_gripper_100mm.urdf (robot description, URDF)
Before this commit: robot Alicia_D_v5_6_gripper_100mm, 10 links, 9 joints
Links:
- link base_link: geometry collision mesh filename=base_link.STL; visual mesh filename=base_link.STL
- link left_gripper: geometry collision mesh filename=left_gripper_100mm.STL; visual mesh filename=left_gripper_100mm.STL
- link link1: geometry collision mesh filename=link1.STL; visual mesh filename=link1.STL
- link link2: geometry collision mesh filename=link2.STL; visual mesh filename=link2.STL
- link link3: geometry collision mesh filename=link3.STL; visual mesh filename=link3.STL
- link link4: geometry collision mesh filename=link4_100mm.STL; visual mesh filename=link4_100mm.STL
- link link5: geometry collision mesh filename=link5.STL; visual mesh filename=link5.STL
- link link6: geometry collision mesh filename=link6_100mm.STL; visual mesh filename=link6_100mm.STL
- link right_gripper: geometry collision mesh filename=right_gripper_100mm.STL; visual mesh filename=right_gripper_100mm.STL

File: synriard/urdf/Alicia_D_v5_6/Alicia_D_v5_6_gripper_50mm.urdf (robot description, URDF)
Before this commit: robot Alicia_D_v5_6_gripper_50mm, 10 links, 9 joints
Links:
- link base_link: geometry collision mesh filename=base_link.STL; visual mesh filename=base_link.STL
- link left_gripper: geometry collision mesh filename=left_gripper_50mm.STL; visual mesh filename=left_gripper_50mm.STL
- link link1: geometry collision mesh filename=link1.STL; visual mesh filename=link1.STL
- link link2: geometry collision mesh filename=link2.STL; visual mesh filename=link2.STL
- link link3: geometry collision mesh filename=link3.STL; visual mesh filename=link3.STL
- link link4: geometry collision mesh filename=link4.STL; visual mesh filename=link4.STL
- link link5: geometry collision mesh filename=link5.STL; visual mesh filename=link5.STL
- link link6: geometry collision mesh filename=link6.STL; visual mesh filename=link6.STL
- link right_gripper: geometry collision mesh filename=right_gripper_50mm.STL; visual mesh filename=right_gripper_50mm.STL

File: synriard/urdf/Alicia_D_v5_6/Alicia_D_v5_6_vertical_50mm.urdf (robot description, URDF)
Before this commit: robot Alicia_D_v5_6_vertical_50mm, 10 links, 9 joints
Links:
- link base_link: geometry collision mesh filename=base_link.STL; visual mesh filename=base_link.STL
- link left_gripper: geometry collision mesh filename=left_gripper.STL; visual mesh filename=left_gripper.STL
- link link1: geometry collision mesh filename=link1.STL; visual mesh filename=link1.STL
- link link2: geometry collision mesh filename=link2.STL; visual mesh filename=link2.STL
- link link3: geometry collision mesh filename=link3.STL; visual mesh filename=link3.STL
- link link4: geometry collision mesh filename=link4.STL; visual mesh filename=link4.STL
- link link5: geometry collision mesh filename=link5.STL; visual mesh filename=link5.STL
- link link6: geometry collision mesh filename=link6.STL; visual mesh filename=link6.STL
- link right_gripper: geometry collision mesh filename=right_gripper.STL; visual mesh filename=right_gripper.STL

File: synriard/urdf/Alicia_D_v6_1_2/Alicia_D_v6_1_2_leader_ffb.urdf (robot description, URDF)
Before this commit: robot Alicia_D_v5_6_leader_ur, 8 links, 7 joints
Links:
- removed link tool0
- link base_link: mass 0.365261662647833 -> 0.682998590998489
- link link1: mass 0.0240091651576837 -> 0.0457400706155227
- link link2: mass 0.0953620090038457 -> 0.153069147969342
- link link3: mass 0.0959280140923854 -> 0.0756083267095565
- link link4: mass 0.0468353202184797 -> 0.0748379713334714
- link link5: mass 0.047589349042095 -> 0.075608308116058
- link link6: mass 0.148889214888287 -> 0.163310330375371
Joints:
- removed joint tool0_fixed_joint
- joint joint1: limit lower=-3.14159 upper=3.14159 effort=5 velocity=12 -> lower=-2.79 upper=2.79 effort=5 velocity=10; origin xyz=-0.01474 0 0.05085 rpy=0 0 0 -> xyz=0 0 0.0448 rpy=0 0 0
- joint joint2: limit lower=-1.75 upper=1.75 effort=5 velocity=12 -> lower=0 upper=3.14 effort=5 velocity=10; origin xyz=0 -0.0003 0.04286 rpy=1.5708 -1.5708 0 -> xyz=0 -0.0009 0.04841 rpy=1.5708 -0.088115 0
- joint joint3: limit lower=0.6 upper=2.2 effort=5 velocity=12 -> lower=-3.14 upper=0 effort=5 velocity=10; origin xyz=0.18922 0.027473 -0.00041 rpy=0 0 0.7854 -> xyz=-0.18612 0.044304 -0.0003 rpy=0 0 -0.059975
- joint joint4: axis 0 0 -1 -> 0 0 1; limit lower=-3.14159 upper=3.14159 effort=5 velocity=12 -> lower=-2.79 upper=2.79 effort=5 velocity=10; origin xyz=0 0.1601 0.0187 rpy=0 0 0 -> xyz=0.071381 0.0018862 -0.0005 rpy=-1.5708 0 -1.5989
- joint joint5: axis 0 0 -1 -> 0 -0.1141 -0.99347; limit lower=-3.14159 upper=3.14159 effort=5 velocity=12 -> lower=-1.57 upper=1.57 effort=5 velocity=10; origin xyz=0 0.02 0.05115 rpy=-1.5708 0 0 -> xyz=-0.00014 -0.0001 0.11461 rpy=0.29064 -1.5708 1.212
- joint joint6: axis 0 0 -1 -> 0 -0.23368 0.97231; limit lower=-3.14159 upper=3.14159 effort=5 velocity=12 -> lower=-3.14 upper=3.14 effort=5 velocity=10; origin xyz=0 -0.0213 0.05115 rpy=1.5708 0 0 -> xyz=0.0713 0.0039254 -5.2447E-05 rpy=-1.8067 0.11662 -1.5708

File: synriard/urdf/Alicia_M_v1_2/Alicia_M_v1_2_follower.urdf (robot description, URDF)
Before this commit: robot alicia_m_v1_2_follower, 11 links, 10 joints
Links:
- link base_link: mass 1.75527696706568 -> 1.2877
- link grasp_base: mass 0.0142808342625993 -> 0.0425
- link link1: mass 0.237800297288607 -> 0.5406
- link link2: mass 0.579389297908421 -> 0.7456
- link link3: mass 0.523091405901433 -> 0.4848
- link link4: mass 0.558638138215147 -> 0.5496
- link link5: mass 0.345531194942532 -> 0.40889
- link link6: mass 0.651 -> 0.4758
- link link7: mass 0.0243852132391449 -> 0.0260
- link link8: mass 0.0243852132391449 -> 0.0260

File: synriard/urdf/Alicia_M_v1_2/Alicia_M_v1_2_follower_ARX.urdf (robot description, URDF)
Before this commit: robot alicia_m_v1_2_follower_arx, 10 links, 9 joints
Links:
- link base_link: mass 1.30948144128201 -> 1.2877
- link link1: mass 0.243059270540488 -> 0.5406
- link link2: mass 0.37082554681883 -> 0.579389297158098
- link link6: mass 0.460840762126697 -> 0.4188
- link link7: mass 0.0249330594865369 -> 0.0274
- link link8: mass 0.0249330594865369 -> 0.0274

File: synriard/urdf/Alicia_M_v1_2/Alicia_M_v1_2_follower_ARX_PX6D.urdf (robot description, URDF)
Before this commit: robot alicia_m_v1_2_follower_arx_px6d, 10 links, 9 joints
Links:
- link link6: mass 0.504336757553032 -> 0.6038
