Commit message: Add tool0 for leader arm

File: synriard/urdf/Alicia_D_v5_6/Alicia_D_v5_6_leader.urdf (robot description, URDF)
Before this commit: robot Alicia_D_v5_6_leader, 7 links, 6 joints
Links:
- added link tool0; visual sphere radius=0.005
Joints:
- added joint tool0_joint: type fixed, parent link6, child tool0, origin xyz=0 0 0.05 rpy=0 0 0, axis 0 0 0
- joint joint4: axis 0 0 1 -> 0 0 -1
- joint joint6: axis 0 0 1 -> 0 0 -1
