Commit message: Add the arx leader arm urdf and upate arx panixi follower urdf mass

File: synriard/urdf/Alicia_D_v5_6/Alicia_D_v5_6_leader_arx.urdf (robot description, URDF)
Before this commit: robot Alicia_D_v5_6_leader, 8 links, 7 joints
Links:
- added link world
- link base_link: mass 0.368093424916451 -> 0.686438268035788
- link link1: mass 0.0243712954879011 -> 0.045739977477124
- link link2: mass 0.0953620083959412 -> 0.152608321825774
- link link3: mass 0.0548526651976208 -> 0.112441385533658
- link link4: mass 0.0644611791940891 -> 0.0728790310641603
- link link5: mass 0.0510330827595259 -> 0.0497669997048517
- link link6: mass 0.148889229292563 -> 0.16331007308822
Joints:
- added joint world_fixed: type fixed, parent world, child base_link, origin xyz=0 0 0 rpy=1.5708 0 0
- joint joint1: axis 0 1 0 -> 0 0 1; limit lower=-2.749 upper=2.749 effort=5 velocity=10 -> lower=-2.9656 upper=2.9656 effort=5 velocity=10; origin xyz=0 0 0.05085 rpy=1.5707963267949 0 0 -> xyz=0 0.0448 0 rpy=-1.5708 0 0
- joint joint2: limit lower=-1.75 upper=1.75 effort=5 velocity=10 -> lower=-3.14 upper=0 effort=5 velocity=10; origin xyz=0 0.0428599999999999 -0.000300000000000013 rpy=3.14159265358979 0 1.5707963267949 -> xyz=0 -0.0009 0.04841 rpy=1.5708 0 0
- joint joint3: limit lower=-0.6 upper=2.2 effort=5 velocity=10 -> lower=-3.14 upper=0 effort=5 velocity=10; origin xyz=0.1892 0.027452 0.001 rpy=0 0 -2.3562 -> xyz=-0.1893 0.027753 -0.0003 rpy=0 0 0
- joint joint4: axis 0 0 -1 -> 0 0 1; limit lower=-2.79 upper=2.79 effort=5 velocity=10 -> lower=-2.355 upper=0.785 effort=5 velocity=10; origin xyz=-0.00389378030941123 -0.0576000000000002 0.000500000000000021 rpy=1.5707963267949 0 0 -> xyz=0.18791 0.00403 3E-05 rpy=0 0 0
- joint joint5: axis 0 0 -1 -> 0 0 1; origin xyz=0 0 0.12231 rpy=-1.5707963267949 0 0 -> xyz=0.056471 0.021474 -0.00018156 rpy=1.5708 0 0
- joint joint6: axis 0 0 -1 -> 0 0 1; limit lower=-3.14159 upper=3.14159 effort=5 velocity=10 -> lower=-2.9656 upper=2.9656 effort=5 velocity=10; origin xyz=-0.0038938 -0.0575 0.0005 rpy=1.5708 0 0 -> xyz=0.02695 0.00014 0.04691 rpy=-1.5708 0 -1.5708

File: synriard/urdf/Alicia_M_v1_2/Alicia_M_v1_2_follower.urdf (robot description, URDF)
Before this commit: robot alicia_m_v1_2_follower, 11 links, 10 joints
Links:
- link link6: mass 0.46822726567622 -> 0.651

File: synriard/urdf/Alicia_M_v1_2/Alicia_M_v1_2_follower_ARX_PX6D.urdf (robot description, URDF)
Before this commit: robot alicia_m_v1_2_follower_arx_px6d, 10 links, 9 joints
Links:
- link link7: mass 0.0249330594865369 -> 0.0274
- link link8: mass 0.0249330594865369 -> 0.0274
