Commit message: Update the bessica v1-1 urdf

File: synriard/urdf/Bessica_D_v1_1/Bessica_D_v1_1_skeleton.urdf (robot description, URDF)
Before this commit: robot 123, 24 links, 21 joints
Links:
- link base_link: geometry collision mesh filename=/home/ubuntu/Alicia/Synria-Robot-Descriptions/synriard/mesh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 scale=1 1 1; visual mesh filename=/home/ubuntu/Alicia/Synria-Robot-Descriptions/synriard/mesh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 scale=1 1 1
- link head: geometry collision mesh filename=/home/ubuntu/Alicia/Synria-Robot-Descriptions/synriard/mesh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 scale=1 1 1; visual mesh filename=/home/ubuntu/Alicia/Synria-Robot-Descriptions/synriard/mesh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 scale=1 1 1
- link left_arm_base_link: geometry collision mesh filename=/home/ubuntu/Alicia/Synria-Robot-Descriptions/synriard/mesh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 scale=1 1 1; visual mesh filename=/home/ubuntu/Alicia/Synria-Robot-Descriptions/synriard/mesh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 scale=1 1 1
- link left_arm_gripper_left_finger: geometry collision mesh filename=/home/ubuntu/Alicia/Synria-Robot-Descriptions/synriard/mesh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 scale=1 1 1; visual mesh filename=/home/ubuntu/Alicia/Synria-Robot-Descriptions/synriard/mesh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 scale=1 1 1
- link left_arm_gripper_right_finger: geometry collision mesh filename=/home/ubuntu/Alicia/Synria-Robot-Descriptions/synriard/mesh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 scale=1 1 1; visual mesh filename=/home/ubuntu/Alicia/Synria-Robot-Descriptions/synriard/mesh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 scale=1 1 1
- link left_arm_link1: geometry collision mesh filename=/home/ubuntu/Alicia/Synria-Robot-Descriptions/synriard/mesh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 scale=1 1 1; visual mesh filename=/home/ubuntu/Alicia/Synria-Robot-Descriptions/synriard/mesh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 scale=1 1 1
- link left_arm_link2: geometry collision mesh filename=/home/ubuntu/Alicia/Synria-Robot-Descriptions/synriard/mesh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 scale=1 1 1; visual mesh filename=/home/ubuntu/Alicia/Synria-Robot-Descriptions/synriard/mesh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 scale=1 1 1
- link left_arm_link3: geometry collision mesh filename=/home/ubuntu/Alicia/Synria-Robot-Descriptions/synriard/mesh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 scale=1 1 1; visual mesh filename=/home/ubuntu/Alicia/Synria-Robot-Descriptions/synriard/mesh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 scale=1 1 1
- link left_arm_link4: geometry collision mesh filename=/home/ubuntu/Alicia/Synria-Robot-Descriptions/synriard/mesh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 scale=1 1 1; visual mesh filename=/home/ubuntu/Alicia/Synria-Robot-Descriptions/synriard/mesh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 scale=1 1 1
- link left_arm_link5: geometry collision mesh filename=/home/ubuntu/Alicia/Synria-Robot-Descriptions/synriard/mesh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 scale=1 1 1; visual mesh filename=/home/ubuntu/Alicia/Synria-Robot-Descriptions/synriard/mesh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 scale=1 1 1
- link left_arm_link6: geometry collision mesh filename=/home/ubuntu/Alicia/Synria-Robot-Descriptions/synriard/mesh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 scale=1 1 1; visual mesh filename=/home/ubuntu/Alicia/Synria-Robot-Descriptions/synriard/mesh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 scale=1 1 1
- link left_arm_link7: geometry collision mesh filename=/home/ubuntu/Alicia/Synria-Robot-Descriptions/synriard/mesh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 scale=1 1 1; visual mesh filename=/home/ubuntu/Alicia/Synria-Robot-Descriptions/synriard/mesh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 scale=1 1 1
- link right_arm_base_link: geometry collision mesh filename=/home/ubuntu/Alicia/Synria-Robot-Descriptions/synriard/mesh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 scale=1 1 1; visual mesh filename=/home/ubuntu/Alicia/Synria-Robot-Descriptions/synriard/mesh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 scale=1 1 1
- link right_arm_gripper_left_finger: geometry collision mesh filename=/home/ubuntu/Alicia/Synria-Robot-Descriptions/synriard/mesh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 scale=1 1 1; visual mesh filename=/home/ubuntu/Alicia/Synria-Robot-Descriptions/synriard/mesh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 scale=1 1 1
- link right_arm_gripper_right_finger: geometry collision mesh filename=/home/ubuntu/Alicia/Synria-Robot-Descriptions/synriard/mesh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 scale=1 1 1; visual mesh filename=/home/ubuntu/Alicia/Synria-Robot-Descriptions/synriard/mesh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 scale=1 1 1
- link right_arm_link1: geometry collision mesh filename=/home/ubuntu/Alicia/Synria-Robot-Descriptions/synriard/mesh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 scale=1 1 1; visual mesh filename=/home/ubuntu/Alicia/Synria-Robot-Descriptions/synriard/mesh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 scale=1 1 1
- link right_arm_link2: geometry collision mesh filename=/home/ubuntu/Alicia/Synria-Robot-Descriptions/synriard/mesh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 scale=1 1 1; visual mesh filename=/home/ubuntu/Alicia/Synria-Robot-Descriptions/synriard/mesh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 scale=1 1 1
- link right_arm_link3: geometry collision mesh filename=/home/ubuntu/Alicia/Synria-Robot-Descriptions/synriard/mesh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 scale=1 1 1; visual mesh filename=/home/ubuntu/Alicia/Synria-Robot-Descriptions/synriard/mesh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 scale=1 1 1
- link right_arm_link4: geometry collision mesh filename=/home/ubuntu/Alicia/Synria-Robot-Descriptions/synriard/mesh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 scale=1 1 1; visual mesh filename=/home/ubuntu/Alicia/Synria-Robot-Descriptions/synriard/mesh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 scale=1 1 1
- link right_arm_link5: geometry collision mesh filename=/home/ubuntu/Alicia/Synria-Robot-Descriptions/synriard/mesh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 scale=1 1 1; visual mesh filename=/home/ubuntu/Alicia/Synria-Robot-Descriptions/synriard/mesh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 scale=1 1 1
- link right_arm_link6: geometry collision mesh filename=/home/ubuntu/Alicia/Synria-Robot-Descriptions/synriard/mesh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 scale=1 1 1; visual mesh filename=/home/ubuntu/Alicia/Synria-Robot-Descriptions/synriard/mesh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 scale=1 1 1
- link right_arm_link7: geometry collision mesh filename=/home/ubuntu/Alicia/Synria-Robot-Descriptions/synriard/mesh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 scale=1 1 1; visual mesh filename=/home/ubuntu/Alicia/Synria-Robot-Descriptions/synriard/mesh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 scale=1 1 1
Joints:
- added joint left_arm_base_joint: type fixed, parent head, child left_arm_base_link, origin xyz=-0.0608244908152262 0.0882407378671147 -0.185541452202364 rpy=1.5707963267949 0 -3.14159265358979, axis 0 0 0
- added joint right_arm_base_joint: type fixed, parent head, child right_arm_base_link, origin xyz=-0.060825 -0.091759 -0.18554 rpy=3.1416 0 -3.1416, axis 0 0 0

Commit message: Update the bessica urdf

File: synriard/urdf/Bessica_D_v1_1/Bessica_D_v1_1_skeleton.urdf (robot description, URDF)
Before this commit: robot Bessica_D_v1_1_skeleton, 24 links, 23 joints
Links:
- removed link head
- added link head_link, mass 0.14240268640264; collision mesh filename=../../meshes/Bessica_D_v1_1/SkeletonOnly/head.STL scale=1 1 1; visual mesh filename=../../meshes/Bessica_D_v1_1/SkeletonOnly/head.STL scale=1 1 1
- link base_link: geometry collision mesh filename=../../meshes/Bessica_D_v1_1/SkeletonOnly/base_link.STL scale=1 1 1; visual mesh filename=../../meshes/Bessica_D_v1_1/SkeletonOnly/base_link.STL scale=1 1 1
- link left_arm_base_link: geometry collision mesh filename=../../meshes/Bessica_D_v1_1/SkeletonOnly/left_arm_base_link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 scale=1 1 1; visual mesh filename=../../meshes/Bessica_D_v1_1/SkeletonOnly/left_arm_base_link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 scale=1 1 1
- link left_arm_gripper_left_finger: geometry collision mesh filename=../../meshes/Bessica_D_v1_1/SkeletonOnly/left_arm_gripper_l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 scale=1 1 1; visual mesh filename=../../meshes/Bessica_D_v1_1/SkeletonOnly/left_arm_gripper_l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 scale=1 1 1
- link left_arm_gripper_right_finger: geometry collision mesh filename=../../meshes/Bessica_D_v1_1/SkeletonOnly/left_arm_gripper_r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 scale=1 1 1; visual mesh filename=../../meshes/Bessica_D_v1_1/SkeletonOnly/left_arm_gripper_r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 scale=1 1 1
- link left_arm_link1: geometry collision mesh filename=../../meshes/Bessica_D_v1_1/SkeletonOnly/left_arm_link1.STL scale=1 1 1; visual mesh filename=../../meshes/Bessica_D_v1_1/SkeletonOnly/left_arm_link1.STL scale=1 1 1
- link left_arm_link2: geometry collision mesh filename=../../meshes/Bessica_D_v1_1/SkeletonOnly/left_arm_link2.STL scale=1 1 1; visual mesh filename=../../meshes/Bessica_D_v1_1/SkeletonOnly/left_arm_link2.STL scale=1 1 1
- link left_arm_link3: geometry collision mesh filename=../../meshes/Bessica_D_v1_1/SkeletonOnly/left_arm_link3.STL scale=1 1 1; visual mesh filename=../../meshes/Bessica_D_v1_1/SkeletonOnly/left_arm_link3.STL scale=1 1 1
- link left_arm_link4: geometry collision mesh filename=../../meshes/Bessica_D_v1_1/SkeletonOnly/left_arm_link4.STL scale=1 1 1; visual mesh filename=../../meshes/Bessica_D_v1_1/SkeletonOnly/left_arm_link4.STL scale=1 1 1
- link left_arm_link5: geometry collision mesh filename=../../meshes/Bessica_D_v1_1/SkeletonOnly/left_arm_link5.STL scale=1 1 1; visual mesh filename=../../meshes/Bessica_D_v1_1/SkeletonOnly/left_arm_link5.STL scale=1 1 1
- link left_arm_link6: geometry collision mesh filename=../../meshes/Bessica_D_v1_1/SkeletonOnly/left_arm_link6.STL scale=1 1 1; visual mesh filename=../../meshes/Bessica_D_v1_1/SkeletonOnly/left_arm_link6.STL scale=1 1 1
- link left_arm_link7: geometry collision mesh filename=../../meshes/Bessica_D_v1_1/SkeletonOnly/left_arm_link7.STL scale=1 1 1; visual mesh filename=../../meshes/Bessica_D_v1_1/SkeletonOnly/left_arm_link7.STL scale=1 1 1
- link right_arm_base_link: geometry collision mesh filename=../../meshes/Bessica_D_v1_1/SkeletonOnly/right_arm_base_lin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 scale=1 1 1; visual mesh filename=../../meshes/Bessica_D_v1_1/SkeletonOnly/right_arm_base_lin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 scale=1 1 1
- link right_arm_gripper_left_finger: geometry collision mesh filename=../../meshes/Bessica_D_v1_1/SkeletonOnly/right_arm_gripper_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 scale=1 1 1; visual mesh filename=../../meshes/Bessica_D_v1_1/SkeletonOnly/right_arm_gripper_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 scale=1 1 1
- link right_arm_gripper_right_finger: geometry collision mesh filename=../../meshes/Bessica_D_v1_1/SkeletonOnly/right_arm_gripper_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 scale=1 1 1; visual mesh filename=../../meshes/Bessica_D_v1_1/SkeletonOnly/right_arm_gripper_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 scale=1 1 1
- link right_arm_link1: geometry collision mesh filename=../../meshes/Bessica_D_v1_1/SkeletonOnly/right_arm_link1.STL scale=1 1 1; visual mesh filename=../../meshes/Bessica_D_v1_1/SkeletonOnly/right_arm_link1.STL scale=1 1 1
- link right_arm_link2: geometry collision mesh filename=../../meshes/Bessica_D_v1_1/SkeletonOnly/right_arm_link2.STL scale=1 1 1; visual mesh filename=../../meshes/Bessica_D_v1_1/SkeletonOnly/right_arm_link2.STL scale=1 1 1
- link right_arm_link3: geometry collision mesh filename=../../meshes/Bessica_D_v1_1/SkeletonOnly/right_arm_link3.STL scale=1 1 1; visual mesh filename=../../meshes/Bessica_D_v1_1/SkeletonOnly/right_arm_link3.STL scale=1 1 1
- link right_arm_link4: geometry collision mesh filename=../../meshes/Bessica_D_v1_1/SkeletonOnly/right_arm_link4.STL scale=1 1 1; visual mesh filename=../../meshes/Bessica_D_v1_1/SkeletonOnly/right_arm_link4.STL scale=1 1 1
- link right_arm_link5: geometry collision mesh filename=../../meshes/Bessica_D_v1_1/SkeletonOnly/right_arm_link5.STL scale=1 1 1; visual mesh filename=../../meshes/Bessica_D_v1_1/SkeletonOnly/right_arm_link5.STL scale=1 1 1
- link right_arm_link6: geometry collision mesh filename=../../meshes/Bessica_D_v1_1/SkeletonOnly/right_arm_link6.STL scale=1 1 1; visual mesh filename=../../meshes/Bessica_D_v1_1/SkeletonOnly/right_arm_link6.STL scale=1 1 1
- link right_arm_link7: geometry collision mesh filename=../../meshes/Bessica_D_v1_1/SkeletonOnly/right_arm_link7.STL scale=1 1 1; visual mesh filename=../../meshes/Bessica_D_v1_1/SkeletonOnly/right_arm_link7.STL scale=1 1 1
Joints:
- joint head: child head -> head_link
- joint left_arm_base_joint: parent head -> head_link
- joint right_arm_base_joint: parent head -> head_link

Commit message: Update the joint 4 direction

File: synriard/urdf/Bessica_D_v1_1/Bessica_D_v1_1_skeleton.urdf (robot description, URDF)
Before this commit: robot Bessica_D_v1_1_skeleton, 24 links, 23 joints
Joints:
- joint left_arm_joint4: axis 0 0 1 -> 0 0 -1; limit lower=-0.5236 upper=2.95 effort=5 velocity=12 -> lower=-2.95 upper=0.5236 effort=5 velocity=12
- joint right_arm_joint4: axis 0 0 1 -> 0 0 -1; limit lower=-0.5236 upper=2.95 effort=5 velocity=12 -> lower=-2.95 upper=0.5236 effort=5 velocity=12

Commit message: Update joint 4 direction of bessica

File: synriard/urdf/Bessica_D_v1_1/Bessica_D_v1_1_skeleton.urdf (robot description, URDF)
Before this commit: robot Bessica_D_v1_1_skeleton, 24 links, 23 joints
Joints:
- joint left_arm_joint4: axis 0 0 -1 -> 0 0 1; limit lower=-2.95 upper=0.5236 effort=5 velocity=12 -> lower=-0.5236 upper=2.95 effort=5 velocity=12
- joint right_arm_joint4: axis 0 0 -1 -> 0 0 1; limit lower=-2.95 upper=0.5236 effort=5 velocity=12 -> lower=-0.5236 upper=2.95 effort=5 velocity=12
