Commit message: Update AM v1.1

File: synriard/urdf/Alicia_M_v1_1/Alicia_M_v1_1_gripper_100mm.urdf (robot description, URDF)
Before this commit: robot alicia_m_v1_1_gripper_100mm, 10 links, 9 joints
Links:
- removed link grasp_base
- added link Grasp_base, mass 0.03877; collision mesh filename=../../meshes/Alicia_M_v1_1/grasp_base.STL; visual mesh filename=../../meshes/Alicia_M_v1_1/grasp_base.STL
- added link tool0; visual sphere radius=0.005
Joints:
- removed joint grasp_base_joint
- removed joint grasp_joint_left
- removed joint grasp_joint_right
- added joint Grasp2tool: type fixed, parent Grasp_base, child tool0, origin xyz=3.3333E-05 -0.000675 0.095 rpy=0 0 0, axis 0 0 0
- added joint Grasp_base_joint: type fixed, parent link6, child Grasp_base, origin xyz=-3.3333E-05 0 0.055 rpy=0 0 0, axis 0 0 0
- added joint left_finger: type prismatic, parent Grasp_base, child link7, origin xyz=3.3333E-05 -0.048175 0.096 rpy=1.5708 0.00034722 0, axis 0 0 1, limit lower=-0.05 upper=0.0 effort=5 velocity=10
- added joint right_finger: type prismatic, parent Grasp_base, child link8, origin xyz=3.3333E-05 0.046825 0.096 rpy=1.5708 0.00034722 0, axis 0 0 1, limit lower=0.0 upper=0.05 effort=5 velocity=10, mimic joint=grasp_joint_right multiplier=-1.0 offset=0
- joint joint1: axis 0 0 -1 -> 0 0 1
- joint joint2: axis 0 0 -1 -> 0 0 1; limit lower=0 upper=3.14 effort=5 velocity=10 -> lower=-3.14 upper=0 effort=5 velocity=10
- joint joint4: axis -0.00034722 0 -1 -> -0.00034722 0 1
- joint joint5: axis 0 0 -1 -> 0 0 1
- joint joint6: axis -0.00034722 0 -1 -> -0.00034722 0 1
