Commit message: update mimic joint name

File: synriard/urdf/Alicia_M_v1_1/Alicia_M_v1_1_follower.urdf (robot description, URDF)
Before this commit: robot alicia_m_v1_1_follower, 10 links, 9 joints
Joints:
- joint right_finger: mimic joint=grasp_joint_right multiplier=-1.0 offset=0 -> joint=left_finger multiplier=-1.0 offset=0

Commit message: Rename joints in Alicia_M_v1_1_follower.urdf from lowercase to CamelCase format

File: synriard/urdf/Alicia_M_v1_1/Alicia_M_v1_1_follower.urdf (robot description, URDF)
Before this commit: robot alicia_m_v1_1_follower, 10 links, 9 joints
Joints:
- removed joint joint1
- removed joint joint2
- removed joint joint3
- removed joint joint4
- removed joint joint5
- removed joint joint6
- added joint Joint1: type revolute, parent base_link, child link1, origin xyz=0 0 0.10705 rpy=0 0 0, axis 0 0 1, limit lower=-2.75 upper=2.75 effort=5 velocity=10
- added joint Joint2: type revolute, parent link1, child link2, origin xyz=0 0 0.046 rpy=1.5708 0 0, axis 0 0 1, limit lower=-3.14 upper=0 effort=5 velocity=10
- added joint Joint3: type revolute, parent link2, child link3, origin xyz=-0.28185 0.040324 0 rpy=0 0 1.5708, axis 0 0 -1, limit lower=-3.14 upper=0 effort=5 velocity=10
- added joint Joint4: type revolute, parent link3, child link4, origin xyz=0.028563 -0.091416 0 rpy=-1.5708 0 -3.1412, axis -0.00034722 0 1, limit lower=-1.57 upper=1.57 effort=5 velocity=10
- added joint Joint5: type revolute, parent link4, child link5, origin xyz=-8.0556E-05 0 0.151 rpy=1.5708 0.00034722 0, axis 0 0 1, limit lower=-1.57 upper=1.57 effort=5 velocity=10
- added joint Joint6: type revolute, parent link5, child link6, origin xyz=5.2431E-05 0.081 0 rpy=-1.5708 0 0.00034722, axis -0.00034722 0 1, limit lower=-2.75 upper=2.75 effort=5 velocity=10

Commit message: Update joint limitation of Alicia-M

File: synriard/urdf/Alicia_M_v1_1/Alicia_M_v1_1_follower.urdf (robot description, URDF)
Before this commit: robot alicia_m_v1_1_follower, 10 links, 9 joints
Links:
- link base_link: geometry collision mesh filename=base_link.STL; visual mesh filename=base_link.STL
- link link1: geometry collision mesh filename=link1.STL; visual mesh filename=link1.STL
- link link2: geometry collision mesh filename=link2.STL; visual mesh filename=link2.STL
- link link3: geometry collision mesh filename=link3.STL; visual mesh filename=link3.STL
- link link4: geometry collision mesh filename=link4.STL; visual mesh filename=link4.STL
- link link5: geometry collision mesh filename=link5.STL; visual mesh filename=link5.STL
- link link6: geometry collision mesh filename=link6.STL; visual mesh filename=link6.STL
- link link7: geometry collision mesh filename=link7.STL; visual mesh filename=link7.STL
- link link8: geometry collision mesh filename=link8.STL; visual mesh filename=link8.STL
Joints:
- joint Joint4: limit lower=-1.57 upper=1.57 effort=5 velocity=10 -> lower=-1.50 upper=1.50 effort=5 velocity=10
- joint Joint5: limit lower=-1.57 upper=1.57 effort=5 velocity=10 -> lower=-1.55 upper=1.55 effort=5 velocity=10

Commit message: [fix] bug of axis in AM v1.1

File: synriard/urdf/Alicia_M_v1_1/Alicia_M_v1_1_follower.urdf (robot description, URDF)
Before this commit: robot alicia_m_v1_1_follower, 10 links, 9 joints
Links:
- added link grasp_base, mass 0.0142808342625993; collision mesh filename=grasp_base.STL; visual mesh filename=grasp_base.STL
- link base_link: mass 2.5385 -> 1.75527696706568
- link link1: mass 0.54365 -> 0.237800297288607; geometry collision mesh filename=Link1.STL; visual mesh filename=Link1.STL
- link link2: mass 1.1153 -> 0.579389297908421; geometry collision mesh filename=Link2.STL; visual mesh filename=Link2.STL
- link link3: mass 0.4356 -> 0.523091405901433; geometry collision mesh filename=Link3.STL; visual mesh filename=Link3.STL
- link link4: mass 0.57265 -> 0.558638138215147; geometry collision mesh filename=Link4.STL; visual mesh filename=Link4.STL
- link link5: mass 0.38891 -> 0.345531194942532; geometry collision mesh filename=Link5.STL; visual mesh filename=Link5.STL
- link link6: mass 0.35658 -> 0.46822726567622; geometry collision mesh filename=Link6.STL; visual mesh filename=Link6.STL
- link link7: mass 0.048674 -> 0.0243852132391449; geometry collision mesh filename=Link7.STL; visual mesh filename=Link7.STL
- link link8: mass 0.048674 -> 0.0243852132391449; geometry collision mesh filename=Link8.STL; visual mesh filename=Link8.STL
Joints:
- added joint grasp_base_joint: type fixed, parent link6, child grasp_base, origin xyz=0.0852198249102375 0.00365621749159879 0.705182667183205 rpy=0 0 0, axis 0 0 0
- joint Joint1: limit lower=-2.75 upper=2.75 effort=5 velocity=10 -> lower=-2.7475 upper=2.7475 effort=5 velocity=10; origin xyz=0 0 0.10705 rpy=0 0 0 -> xyz=0 -0.0039812 0.09125 rpy=0 0 1.5708
- joint Joint2: origin xyz=0 0 0.046 rpy=1.5708 0 0 -> xyz=0.0039812 0 0.0425 rpy=1.5708 0 -1.5708
- joint Joint3: origin xyz=-0.28185 0.040324 0 rpy=0 0 1.5708 -> xyz=-0.28184 0.040424 0 rpy=0 0 0
- joint Joint4: axis -0.00034722 0 1 -> 0 0 1; limit lower=-1.50 upper=1.50 effort=5 velocity=10 -> lower=-1.57 upper=1.57 effort=5 velocity=10; origin xyz=0.028563 -0.091416 0 rpy=-1.5708 0 -3.1412 -> xyz=0.10092 0.028546 0.0036562 rpy=-1.5708 0 -1.5708
- joint Joint5: limit lower=-1.55 upper=1.55 effort=5 velocity=10 -> lower=-1.57 upper=1.57 effort=5 velocity=10; origin xyz=-8.0556E-05 0 0.151 rpy=1.5708 0.00034722 0 -> xyz=0 0.0036562 0.1365 rpy=1.5708 0 0
- joint Joint6: axis -0.00034722 0 1 -> 0 0 1; limit lower=-2.75 upper=2.75 effort=5 velocity=10 -> lower=-2.791 upper=2.791 effort=5 velocity=10; origin xyz=5.2431E-05 0.081 0 rpy=-1.5708 0 0.00034722 -> xyz=0 0.091 0.0036563 rpy=-1.5708 0 0
- joint left_finger: axis 0 0 1 -> 0 0 -1; limit lower=-0.05 upper=0.0 effort=5 velocity=10 -> lower=-0.05 upper=0 effort=5 velocity=10; origin xyz=0 -0.048175 0.151 rpy=1.5708 0.00034722 0 -> xyz=-0.0852198249102478 -0.0536572471053041 -0.563682569174653 rpy=-3.14159264689699 -1.57079450020183 1.57079632010208; parent link6 -> grasp_base
- joint right_finger: limit lower=0.0 upper=0.05 effort=5 velocity=10 -> lower=0 upper=0.05 effort=5 velocity=10; origin xyz=0 0.046825 0.151 rpy=1.5708 0.00034722 0 -> xyz=-0.0852198249102447 0.0463427528945291 -0.563682751833062 rpy=0 1.57079450020183 -1.57079633348771; parent link6 -> grasp_base

Commit message: Fix xml link name mismatch

File: synriard/urdf/Alicia_M_v1_1/Alicia_M_v1_1_follower.urdf (robot description, URDF)
Before this commit: robot alicia_m_v1_1_follower, 11 links, 10 joints
Joints:
- joint Joint4: limit lower=-1.57 upper=1.57 effort=5 velocity=10 -> lower=-2.79253 upper=2.79253 effort=5 velocity=10
