Commit message: Update the bessica m urdf

File: synriard/urdf/Bessica_M_v1_0/Bessica_M_v1_0.urdf (robot description, URDF)
Before this commit: robot Bessica_M_v1_0, 22 links, 21 joints
Links:
- link Left_arm_link1: mass 0.375516464391834 -> 0.375516464240854
- link Left_arm_link2: mass 0.0428315653175016 -> 0.0664892171532656
- link Left_arm_link3: mass 0.281936177906827 -> 0.276673991803197
- link Left_arm_link4: mass 0.147999944408839 -> 0.147999944374733
- link Left_arm_link5: mass 0.162665516517614 -> 0.162665516295154
- link Left_arm_link6: mass 0.148254477928819 -> 0.148254477929042
- link Left_arm_link7: mass 0.162887358777237 -> 0.162887358777534
- link Left_arm_link8: mass 0.0239390375083336 -> 0.0239390375083334
- link Right_arm_link1: mass 0.375516464240854 -> 0.375516464391834
- link Right_arm_link2: mass 0.0664892171532656 -> 0.0428315653175016
- link Right_arm_link3: mass 0.276673991803197 -> 0.281936177906827
- link Right_arm_link4: mass 0.147999944374733 -> 0.147999944408839
- link Right_arm_link5: mass 0.162665516295154 -> 0.162665516517614
- link Right_arm_link6: mass 0.148254477929042 -> 0.148254477928819
- link Right_arm_link7: mass 0.162887358777534 -> 0.162887358777237
- link Right_arm_link8: mass 0.0239390375083334 -> 0.0239390375083336
Joints:
- joint Left_arm_joint1: axis 0 1 0 -> 0 0 -1; origin xyz=-0.146389856983547 0.288056431115987 0 rpy=3.14159265358979 0 -1.91986217719376 -> xyz=0.14638985542209 0.288056431115988 0 rpy=1.5707963267949 0 1.91986217719376
- joint Left_arm_joint2: axis 0 0 -1 -> 0 0 1; limit lower=-0.13 upper=1.57 effort=5 velocity=10 -> lower=-1.57 upper=0.13 effort=5 velocity=10; origin xyz=9.9999999999878E-05 0.0649999999999999 0 rpy=-3.14159265358979 0 -1.5707963267949 -> xyz=9.99999999994339E-05 0.0301000000000004 0.0649999999999997 rpy=1.5707963267949 1.5707963267949 0
- joint Left_arm_joint3: origin xyz=0.00889252372646782 -0.0694320081404333 0 rpy=1.5707963267949 0 0.349065850398866 -> xyz=0.00889252372646632 -0.0694320081404338 0.0301000000000011 rpy=1.5707963267949 0 0.349065850398862
- joint Left_arm_joint4: limit lower=-1.35 upper=0.13 effort=5 velocity=10 -> lower=-0.13 upper=1.35 effort=5 velocity=10; origin xyz=0 0 0.15105 rpy=-1.5707963267949 0 0 -> xyz=0 -0.029675000000001 0.151050000000001 rpy=1.5707963267949 0 0
- joint Left_arm_joint5: axis 0 0 -1 -> 0 0 1; limit lower=-1.04 upper=0.52 effort=5 velocity=10 -> lower=-0.52 upper=1.04 effort=5 velocity=10; origin xyz=0 -0.0983000000000001 0.00117500000000332 rpy=1.5707963267949 0 0 -> xyz=0 0.098299999999999 -0.0284999999999962 rpy=1.5707963267949 0 0
- joint Left_arm_joint6: axis 0 0 1 -> 0 0 -1; origin xyz=0.000499999999999251 -0.00117500000000305 0.139500000000004 rpy=1.5707963267949 0 -1.5707963267949 -> xyz=0.000500000000001166 0 -0.139500000000004 rpy=1.5707963267949 0 -1.5707963267949
- joint Left_arm_joint7: origin xyz=0 0 0 rpy=1.5707963267949 1.53474992982451 -1.5707963267949 -> xyz=0 0 0 rpy=3.14159265358979 1.5707963267949 0
- joint Left_arm_joint8: origin xyz=-0.031434667830233 -0.177982756632216 0.00367500000001846 rpy=3.1055462566194 1.5707963267949 0 -> xyz=0.025 0.179 0.00249999999999894 rpy=0 1.5707963267949 0
- joint Left_arm_joint9: origin xyz=0.0185328521185251 -0.179784686200892 0.00367500000001854 rpy=0.0360463969703927 1.5707963267949 0 -> xyz=-0.0250000000000001 0.179 0.00249999999999898 rpy=3.14159265358979 1.5707963267949 0
- joint Right_arm_joint1: axis 0 0 -1 -> 0 1 0; origin xyz=0.14638985542209 0.288056431115988 0 rpy=1.5707963267949 0 1.91986217719376 -> xyz=-0.146389856983547 0.288056431115987 0 rpy=3.14159265358979 0 -1.91986217719376
- joint Right_arm_joint2: axis 0 0 1 -> 0 0 -1; limit lower=-1.57 upper=0.13 effort=5 velocity=10 -> lower=-0.13 upper=1.57 effort=5 velocity=10; origin xyz=9.99999999994339E-05 0.0301000000000004 0.0649999999999997 rpy=1.5707963267949 1.5707963267949 0 -> xyz=9.9999999999878E-05 0.0649999999999999 0 rpy=-3.14159265358979 0 -1.5707963267949
- joint Right_arm_joint3: origin xyz=0.00889252372646632 -0.0694320081404338 0.0301000000000011 rpy=1.5707963267949 0 0.349065850398862 -> xyz=0.00889252372646782 -0.0694320081404333 0 rpy=1.5707963267949 0 0.349065850398866
- joint Right_arm_joint4: limit lower=-0.13 upper=1.35 effort=5 velocity=10 -> lower=-1.35 upper=0.13 effort=5 velocity=10; origin xyz=0 -0.029675000000001 0.151050000000001 rpy=1.5707963267949 0 0 -> xyz=0 0 0.15105 rpy=-1.5707963267949 0 0
- joint Right_arm_joint5: axis 0 0 1 -> 0 0 -1; limit lower=-0.52 upper=1.04 effort=5 velocity=10 -> lower=-1.04 upper=0.52 effort=5 velocity=10; origin xyz=0 0.098299999999999 -0.0284999999999962 rpy=1.5707963267949 0 0 -> xyz=0 -0.0983000000000001 0.00117500000000332 rpy=1.5707963267949 0 0
- joint Right_arm_joint6: axis 0 0 -1 -> 0 0 1; origin xyz=0.000500000000001166 0 -0.139500000000004 rpy=1.5707963267949 0 -1.5707963267949 -> xyz=0.000499999999999251 -0.00117500000000305 0.139500000000004 rpy=1.5707963267949 0 -1.5707963267949
- joint Right_arm_joint7: origin xyz=0 0 0 rpy=3.14159265358979 1.5707963267949 0 -> xyz=0 0 0 rpy=1.5707963267949 1.53474992982451 -1.5707963267949
- joint Right_arm_joint8: origin xyz=0.025 0.179 0.00249999999999894 rpy=0 1.5707963267949 0 -> xyz=-0.031434667830233 -0.177982756632216 0.00367500000001846 rpy=3.1055462566194 1.5707963267949 0
- joint Right_arm_joint9: origin xyz=-0.0250000000000001 0.179 0.00249999999999898 rpy=3.14159265358979 1.5707963267949 0 -> xyz=0.0185328521185251 -0.179784686200892 0.00367500000001854 rpy=0.0360463969703927 1.5707963267949 0

Commit message: Update the bessica m urdf

File: synriard/urdf/Bessica_M_v1_0/Bessica_M_v1_0.urdf (robot description, URDF)
Before this commit: robot Bessica_M_v1_0, 22 links, 21 joints
Joints:
- removed joint Left_arm_joint1
- removed joint Left_arm_joint2
- removed joint Left_arm_joint3
- removed joint Left_arm_joint4
- removed joint Left_arm_joint5
- removed joint Left_arm_joint6
- removed joint Left_arm_joint7
- removed joint Left_arm_joint8
- removed joint Left_arm_joint9
- removed joint Right_arm_joint1
- removed joint Right_arm_joint2
- removed joint Right_arm_joint3
- removed joint Right_arm_joint4
- removed joint Right_arm_joint5
- removed joint Right_arm_joint6
- removed joint Right_arm_joint7
- removed joint Right_arm_joint8
- removed joint Right_arm_joint9
- added joint Left_gripper1: type prismatic, parent Left_arm_link7, child Left_arm_link8, origin xyz=0.025 0.179 0.00249999999999894 rpy=0 1.5707963267949 0, axis 0 0 1, limit lower=-0.025 upper=0.025 effort=5 velocity=10
- added joint Left_gripper2: type prismatic, parent Left_arm_link7, child Left_arm_link9, origin xyz=-0.0250000000000001 0.179 0.00249999999999898 rpy=3.14159265358979 1.5707963267949 0, axis 0 0 -1, limit lower=-0.025 upper=0.025 effort=5 velocity=10
- added joint Left_joint1: type revolute, parent Torso_link3, child Left_arm_link1, origin xyz=0.14638985542209 0.288056431115988 0 rpy=1.5707963267949 0 1.91986217719376, axis 0 0 -1, limit lower=-0.39 upper=1.83 effort=5 velocity=10
- added joint Left_joint2: type revolute, parent Left_arm_link1, child Left_arm_link2, origin xyz=9.99999999994339E-05 0.0301000000000004 0.0649999999999997 rpy=1.5707963267949 1.5707963267949 0, axis 0 0 -1, limit lower=-0.13 upper=1.57 effort=5 velocity=10
- added joint Left_joint3: type revolute, parent Left_arm_link2, child Left_arm_link3, origin xyz=0.00889252372646632 -0.0694320081404338 0.0301000000000011 rpy=1.5707963267949 0 0.349065850398862, axis 0 0 -1, limit lower=-0.78 upper=0.78 effort=5 velocity=10
- added joint Left_joint4: type revolute, parent Left_arm_link3, child Left_arm_link4, origin xyz=0 -0.029675000000001 0.151050000000001 rpy=1.5707963267949 0 0, axis 0 0 -1, limit lower=-0.13 upper=1.35 effort=5 velocity=10
- added joint Left_joint5: type revolute, parent Left_arm_link4, child Left_arm_link5, origin xyz=0 0.098299999999999 -0.0284999999999962 rpy=1.5707963267949 0 0, axis 0 0 1, limit lower=-0.52 upper=1.04 effort=5 velocity=10
- added joint Left_joint6: type revolute, parent Left_arm_link5, child Left_arm_link6, origin xyz=0.000500000000001166 0 -0.139500000000004 rpy=1.5707963267949 0 -1.5707963267949, axis 0 0 -1, limit lower=-0.52 upper=0.52 effort=5 velocity=10
- added joint Left_joint7: type revolute, parent Left_arm_link6, child Left_arm_link7, origin xyz=0 0 0 rpy=3.14159265358979 1.5707963267949 0, axis 0 0 1, limit lower=-0.78 upper=0.78 effort=5 velocity=10
- added joint Right_gripper1: type prismatic, parent Right_arm_link7, child Right_arm_link8, origin xyz=-0.031434667830233 -0.177982756632216 0.00367500000001846 rpy=3.1055462566194 1.5707963267949 0, axis 0 0 1, limit lower=-0.025 upper=0.025 effort=5 velocity=10
- added joint Right_gripper2: type prismatic, parent Right_arm_link7, child Right_arm_link9, origin xyz=0.0185328521185251 -0.179784686200892 0.00367500000001854 rpy=0.0360463969703927 1.5707963267949 0, axis 0 0 -1, limit lower=-0.025 upper=0.025 effort=5 velocity=10
- added joint Right_joint1: type revolute, parent Torso_link3, child Right_arm_link1, origin xyz=-0.146389856983547 0.288056431115987 0 rpy=3.14159265358979 0 -1.91986217719376, axis 0 1 0, limit lower=-0.39 upper=1.83 effort=5 velocity=10
- added joint Right_joint2: type revolute, parent Right_arm_link1, child Right_arm_link2, origin xyz=9.9999999999878E-05 0.0649999999999999 0 rpy=-3.14159265358979 0 -1.5707963267949, axis 0 0 -1, limit lower=-0.13 upper=1.57 effort=5 velocity=10
- added joint Right_joint3: type revolute, parent Right_arm_link2, child Right_arm_link3, origin xyz=0.00889252372646782 -0.0694320081404333 0 rpy=1.5707963267949 0 0.349065850398866, axis 0 0 1, limit lower=-0.78 upper=0.78 effort=5 velocity=10
- added joint Right_joint4: type revolute, parent Right_arm_link3, child Right_arm_link4, origin xyz=0 0 0.15105 rpy=-1.5707963267949 0 0, axis 0 0 -1, limit lower=-1.35 upper=0.13 effort=5 velocity=10
- added joint Right_joint5: type revolute, parent Right_arm_link4, child Right_arm_link5, origin xyz=0 -0.0983000000000001 0.00117500000000332 rpy=1.5707963267949 0 0, axis 0 0 1, limit lower=-0.52 upper=1.04 effort=5 velocity=10
- added joint Right_joint6: type revolute, parent Right_arm_link5, child Right_arm_link6, origin xyz=0.000499999999999251 -0.00117500000000305 0.139500000000004 rpy=1.5707963267949 0 -1.5707963267949, axis 0 0 1, limit lower=-0.52 upper=0.52 effort=5 velocity=10
- added joint Right_joint7: type revolute, parent Right_arm_link6, child Right_arm_link7, origin xyz=0 0 0 rpy=1.5707963267949 1.53474992982451 -1.5707963267949, axis 0 0 -1, limit lower=-0.78 upper=0.78 effort=5 velocity=10

Commit message: Add a head link and correct the joint limitation of bessica m

File: synriard/urdf/Bessica_M_v1_0/Bessica_M_v1_0.urdf (robot description, URDF)
Before this commit: robot Bessica_M_v1_0, 22 links, 21 joints
Links:
- added link head_link; visual sphere radius=0.005
Joints:
- added joint head_joint: type fixed, parent Torso_link1, child head_link, origin xyz=-0.018 -0.003 -0.5 rpy=-3.14159265358979 0 0, axis 0 0 0
- joint Left_joint1: limit lower=-0.39 upper=1.83 effort=5 velocity=10 -> lower=-3.14159265358979 upper=3.14159265358979 effort=5 velocity=10
- joint Left_joint2: limit lower=-0.13 upper=1.57 effort=5 velocity=10 -> lower=0 upper=3.14159265358979 effort=5 velocity=10
- joint Left_joint3: limit lower=-0.78 upper=0.78 effort=5 velocity=10 -> lower=-1.5707963267949 upper=1.5707963267949 effort=5 velocity=10
- joint Left_joint4: limit lower=-0.13 upper=1.35 effort=5 velocity=10 -> lower=-2.35619449019234 upper=0.261799387799149 effort=5 velocity=10
- joint Left_joint5: limit lower=-0.52 upper=1.04 effort=5 velocity=10 -> lower=-1.309 upper=1.309 effort=5 velocity=10
- joint Left_joint6: limit lower=-0.52 upper=0.52 effort=5 velocity=10 -> lower=-1.0472 upper=1.0472 effort=5 velocity=10
- joint Left_joint7: limit lower=-0.78 upper=0.78 effort=5 velocity=10 -> lower=-3.14159265358979 upper=3.14159265358979 effort=5 velocity=10
- joint Right_joint1: limit lower=-0.39 upper=1.83 effort=5 velocity=10 -> lower=-3.14159265358979 upper=3.14159265358979 effort=5 velocity=10
- joint Right_joint2: limit lower=-0.13 upper=1.57 effort=5 velocity=10 -> lower=0 upper=3.14159265358979 effort=5 velocity=10
- joint Right_joint3: limit lower=-0.78 upper=0.78 effort=5 velocity=10 -> lower=-1.5707963267949 upper=1.5707963267949 effort=5 velocity=10
- joint Right_joint4: axis 0 0 -1 -> 0 0 1; limit lower=-1.35 upper=0.13 effort=5 velocity=10 -> lower=-0.261799387799149 upper=2.35619449019234 effort=5 velocity=10
- joint Right_joint5: limit lower=-0.52 upper=1.04 effort=5 velocity=10 -> lower=-1.309 upper=1.309 effort=5 velocity=10
- joint Right_joint6: limit lower=-0.52 upper=0.52 effort=5 velocity=10 -> lower=-1.0472 upper=1.0472 effort=5 velocity=10
- joint Right_joint7: limit lower=-0.78 upper=0.78 effort=5 velocity=10 -> lower=-3.14159265358979 upper=3.14159265358979 effort=5 velocity=10

Commit message: Update the parent link of head link in bessica m urdf

File: synriard/urdf/Bessica_M_v1_0/Bessica_M_v1_0.urdf (robot description, URDF)
Before this commit: robot Bessica_M_v1_0, 23 links, 22 joints
Joints:
- joint head_joint: parent Torso_link1 -> Torso_link3
