Commit message: Update mesh names

File: synriard/urdf/Alicia_D_v5_5/Alicia_D_v5_5_gripper_100mm.urdf (robot description, URDF)
Before this commit: robot Alicia_D_v5_5_gripper_100mm, 11 links, 10 joints
Links:
- removed link Grasp_base
- removed link Link1
- removed link Link2
- removed link Link3
- removed link Link4
- removed link Link5
- removed link Link6
- removed link Link7
- removed link Link8
- added link grasp_base, mass 0.119820573147005; collision mesh filename=../../meshes/Alicia_D_v5_5/grasp_base.STL; visual mesh filename=../../meshes/Alicia_D_v5_5/grasp_base.STL
- added link link1, mass 0.193725361315237; collision mesh filename=../../meshes/Alicia_D_v5_5/link1.STL; visual mesh filename=../../meshes/Alicia_D_v5_5/link1.STL
- added link link2, mass 0.216765318032361; collision mesh filename=../../meshes/Alicia_D_v5_5/link2.STL; visual mesh filename=../../meshes/Alicia_D_v5_5/link2.STL
- added link link3, mass 0.0845575681430802; collision mesh filename=../../meshes/Alicia_D_v5_5/link3.STL; visual mesh filename=../../meshes/Alicia_D_v5_5/link3.STL
- added link link4, mass 0.0653695953286747; collision mesh filename=../../meshes/Alicia_D_v5_5/link4.STL; visual mesh filename=../../meshes/Alicia_D_v5_5/link4.STL
- added link link5, mass 0.0463941316397046; collision mesh filename=../../meshes/Alicia_D_v5_5/link5.STL; visual mesh filename=../../meshes/Alicia_D_v5_5/link5.STL
- added link link6, mass 0.000754053623586768; collision mesh filename=../../meshes/Alicia_D_v5_5/link6.STL; visual mesh filename=../../meshes/Alicia_D_v5_5/link6.STL
- added link link7, mass 0.0256461121677861; collision mesh filename=../../meshes/Alicia_D_v5_5/link7.STL; visual mesh filename=../../meshes/Alicia_D_v5_5/link7.STL
- added link link8, mass 0.025646112167786; collision mesh filename=../../meshes/Alicia_D_v5_5/link8.STL; visual mesh filename=../../meshes/Alicia_D_v5_5/link8.STL
Joints:
- joint Grasp2tool: parent Grasp_base -> grasp_base
- joint Joint1: child Link1 -> link1
- joint Joint2: child Link2 -> link2; parent Link1 -> link1
- joint Joint3: child Link3 -> link3; parent Link2 -> link2
- joint Joint4: child Link4 -> link4; parent Link3 -> link3
- joint Joint5: child Link5 -> link5; parent Link4 -> link4
- joint Joint6: child Link6 -> link6; parent Link5 -> link5
- joint Joint6_to_gripper_base: child Grasp_base -> grasp_base; parent Link6 -> link6
- joint left_finger: child Link7 -> link7; parent Grasp_base -> grasp_base
- joint right_finger: child Link8 -> link8; parent Grasp_base -> grasp_base

Commit message: A big refactor
compare mjcf with urdf in robocore 2.5dev, make sure they are the same

File: synriard/urdf/Alicia_D_v5_5/Alicia_D_v5_5_gripper_100mm.urdf (robot description, URDF)
Before this commit: robot Alicia_D_v5_5_gripper_100mm, 11 links, 10 joints
Links:
- removed link grasp_base
Joints:
- removed joint Grasp2tool
- removed joint Joint6_to_gripper_base
- added joint tool0_fixed_joint: type fixed, parent link6, child tool0, origin xyz=0 0 0.13 rpy=0 0 0, axis 0 0 0
- joint left_finger: parent grasp_base -> link6
- joint right_finger: parent grasp_base -> link6

File: synriard/urdf/Alicia_D_v5_6/Alicia_D_v5_6_gripper_50mm.urdf (robot description, URDF)
Before this commit: robot Alicia_D_v5_6_gripper_50mm, 10 links, 9 joints
Joints:
- removed joint finger
- added joint tool0_fixed_joint: type fixed, parent link6, child tool0, origin xyz=0 0 -0.13 rpy=0 0 0, axis 0 0 0

File: synriard/urdf/Alicia_D_v5_6/Alicia_D_v5_6_leader.urdf (robot description, URDF)
Before this commit: robot Alicia_D_v5_6_leader, 8 links, 7 joints
Joints:
- removed joint tool0_joint
- added joint tool0_fixed_joint: type fixed, parent link6, child tool0, origin xyz=0 0 0.05 rpy=0 0 0, axis 0 0 0

File: synriard/urdf/Alicia_D_v5_6/Alicia_D_v5_6_leader_ur.urdf (robot description, URDF)
Before this commit: robot Alicia_D_v5_6_leader_ur, 8 links, 7 joints
Joints:
- removed joint tool0_joint
- added joint tool0_fixed_joint: type fixed, parent link6, child tool0, origin xyz=0 0 0.05 rpy=0 0 0, axis 0 0 0

File: synriard/urdf/Alicia_D_v5_6/Alicia_D_v5_6_vertical_50mm.urdf (robot description, URDF)
Before this commit: robot Alicia_D_v5_6_vertical_50mm, 10 links, 9 joints
Joints:
- removed joint finger
- added joint tool0_fixed_joint: type fixed, parent link6, child tool0, origin xyz=0 0 0.13 rpy=0 0 0, axis 0 0 0

File: synriard/urdf/Alicia_M_v1_1/Alicia_M_v1_1_follower.urdf (robot description, URDF)
Before this commit: robot Alicia_D_v5_6_gripper_100mm, 10 links, 9 joints
Links:
- removed link left_gripper
- removed link right_gripper
- added link link7, mass 0.048674; collision mesh filename=../../meshes/Alicia_M_v1_1/follower/link7.STL; visual mesh filename=../../meshes/Alicia_M_v1_1/follower/link7.STL
- added link link8, mass 0.048674; collision mesh filename=../../meshes/Alicia_M_v1_1/follower/link8.STL; visual mesh filename=../../meshes/Alicia_M_v1_1/follower/link8.STL
- link base_link: mass 0.733961424954529 -> 2.5385; geometry collision mesh filename=../../meshes/Alicia_M_v1_1/follower/base_link.STL; visual mesh filename=../../meshes/Alicia_M_v1_1/follower/base_link.STL
- link link1: mass 0.195233495556057 -> 0.54365; geometry collision mesh filename=../../meshes/Alicia_M_v1_1/follower/link1.STL; visual mesh filename=../../meshes/Alicia_M_v1_1/follower/link1.STL
- link link2: mass 0.207033693066089 -> 1.1153; geometry collision mesh filename=../../meshes/Alicia_M_v1_1/follower/link2.STL; visual mesh filename=../../meshes/Alicia_M_v1_1/follower/link2.STL
- link link3: mass 0.0845575651613574 -> 0.4356; geometry collision mesh filename=../../meshes/Alicia_M_v1_1/follower/link3.STL; visual mesh filename=../../meshes/Alicia_M_v1_1/follower/link3.STL
- link link4: mass 0.0653695951425785 -> 0.57265; geometry collision mesh filename=../../meshes/Alicia_M_v1_1/follower/link4.STL; visual mesh filename=../../meshes/Alicia_M_v1_1/follower/link4.STL
- link link5: mass 0.050763902309721 -> 0.38891; geometry collision mesh filename=../../meshes/Alicia_M_v1_1/follower/link5.STL; visual mesh filename=../../meshes/Alicia_M_v1_1/follower/link5.STL
- link link6: mass 0.119820573151617 -> 0.35658; geometry collision mesh filename=../../meshes/Alicia_M_v1_1/follower/link6.STL; visual mesh filename=../../meshes/Alicia_M_v1_1/follower/link6.STL
Joints:
- removed joint Joint1
- removed joint Joint2
- removed joint Joint3
- removed joint Joint4
- removed joint Joint5
- removed joint Joint6
- added joint joint1: type revolute, parent base_link, child link1, origin xyz=0 0 0.10705 rpy=0 0 0, axis 0 0 1, limit lower=-2.75 upper=2.75 effort=5 velocity=10
- added joint joint2: type revolute, parent link1, child link2, origin xyz=0 0 0.046 rpy=1.5708 0 0, axis 0 0 1, limit lower=-3.14 upper=0 effort=5 velocity=10
- added joint joint3: type revolute, parent link2, child link3, origin xyz=-0.28185 0.040324 0 rpy=0 0 1.5708, axis 0 0 -1, limit lower=-3.14 upper=0 effort=5 velocity=10
- added joint joint4: type revolute, parent link3, child link4, origin xyz=0.028563 -0.091416 0 rpy=-1.5708 0 -3.1412, axis -0.00034722 0 1, limit lower=-1.57 upper=1.57 effort=5 velocity=10
- added joint joint5: type revolute, parent link4, child link5, origin xyz=-8.0556E-05 0 0.151 rpy=1.5708 0.00034722 0, axis 0 0 1, limit lower=-1.57 upper=1.57 effort=5 velocity=10
- added joint joint6: type revolute, parent link5, child link6, origin xyz=5.2431E-05 0.081 0 rpy=-1.5708 0 0.00034722, axis -0.00034722 0 1, limit lower=-2.75 upper=2.75 effort=5 velocity=10
- joint left_finger: child left_gripper -> link7; limit lower=0 upper=0.05 effort=5 velocity=12 -> lower=-0.05 upper=0.0 effort=5 velocity=10; origin xyz=-0.000200000000001088 -0.050497849845622 0.130979659620446 rpy=1.5707963267949 0 3.14159265358979 -> xyz=0 -0.048175 0.151 rpy=1.5708 0.00034722 0
- joint right_finger: axis 0 0 -1 -> 0 0 1; child right_gripper -> link8; limit lower=-0.05 upper=0 effort=5 velocity=12 -> lower=0.0 upper=0.05 effort=5 velocity=10; mimic (none) -> joint=grasp_joint_right multiplier=-1.0 offset=0; origin xyz=-0.000199999999998035 0.050502150154378 0.130979659620446 rpy=-1.5707963267949 0 3.14159265358978 -> xyz=0 0.046825 0.151 rpy=1.5708 0.00034722 0
- joint tool0_fixed_joint: origin xyz=0 0 0.13 rpy=0 0 0 -> xyz=0 0 0.15 rpy=0 0 0

File: synriard/urdf/Bessica_D_v1_1/Bessica_D_v1_1_covered.urdf (robot description, URDF)
Before this commit: robot bessica_d, 24 links, 23 joints
Links:
- removed link head
- removed link left_gripper_center
- removed link right_gripper_center
- added link head_link, mass 0.14240268640264; collision mesh filename=../../meshes/Bessica_D_v1_1/SkeletonOnly/head.STL scale=1 1 1; visual mesh filename=../../meshes/Bessica_D_v1_1/SkeletonOnly/head.STL scale=1 1 1
- added link left_tool0; visual sphere radius=0.005
- added link right_tool0; visual sphere radius=0.005
- link base_link: mass 2.26415289791904 -> 2.97915154863328; geometry collision mesh filename=../../meshes/Bessica_D_v1_1/SkeletonOnly/base_link.STL scale=1 1 1; visual mesh filename=../../meshes/Bessica_D_v1_1/SkeletonOnly/base_link.STL scale=1 1 1
- link left_arm_base_link: mass 0.760760214288355 -> 0.708886467098045; geometry collision mesh filename=../../meshes/Bessica_D_v1_1/SkeletonOnly/left_arm_base_link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 scale=1 1 1; visual mesh filename=../../meshes/Bessica_D_v1_1/SkeletonOnly/left_arm_base_link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 scale=1 1 1
- link left_arm_gripper_left_finger: mass 0.0256462689646809 -> 0.025646269010605; geometry collision mesh filename=../../meshes/Bessica_D_v1_1/SkeletonOnly/left_arm_gripper_l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 scale=1 1 1; visual mesh filename=../../meshes/Bessica_D_v1_1/SkeletonOnly/left_arm_gripper_l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 scale=1 1 1
- link left_arm_gripper_right_finger: mass 0.0256462690106051 -> 0.025646269010605; geometry collision mesh filename=../../meshes/Bessica_D_v1_1/SkeletonOnly/left_arm_gripper_r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 scale=1 1 1; visual mesh filename=../../meshes/Bessica_D_v1_1/SkeletonOnly/left_arm_gripper_r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 scale=1 1 1
- link left_arm_link1: mass 0.315733947117255 -> 0.197841071704829; geometry collision mesh filename=../../meshes/Bessica_D_v1_1/SkeletonOnly/left_arm_link1.STL scale=1 1 1; visual mesh filename=../../meshes/Bessica_D_v1_1/SkeletonOnly/left_arm_link1.STL scale=1 1 1
- link left_arm_link2: mass 0.0501482304995307 -> 0.047269050971783; geometry collision mesh filename=../../meshes/Bessica_D_v1_1/SkeletonOnly/left_arm_link2.STL scale=1 1 1; visual mesh filename=../../meshes/Bessica_D_v1_1/SkeletonOnly/left_arm_link2.STL scale=1 1 1
- link left_arm_link3: mass 0.373333387538863 -> 0.140451564579074; geometry collision mesh filename=../../meshes/Bessica_D_v1_1/SkeletonOnly/left_arm_link3.STL scale=1 1 1; visual mesh filename=../../meshes/Bessica_D_v1_1/SkeletonOnly/left_arm_link3.STL scale=1 1 1
- link left_arm_link4: mass 0.0480071391158089 -> 0.0427207248079551; geometry collision mesh filename=../../meshes/Bessica_D_v1_1/SkeletonOnly/left_arm_link4.STL scale=1 1 1; visual mesh filename=../../meshes/Bessica_D_v1_1/SkeletonOnly/left_arm_link4.STL scale=1 1 1
- link left_arm_link5: mass 0.207077276180107 -> 0.110396951419793; geometry collision mesh filename=../../meshes/Bessica_D_v1_1/SkeletonOnly/left_arm_link5.STL scale=1 1 1; visual mesh filename=../../meshes/Bessica_D_v1_1/SkeletonOnly/left_arm_link5.STL scale=1 1 1
- link left_arm_link6: mass 0.0325622574715583 -> 0.0345706786766011; geometry collision mesh filename=../../meshes/Bessica_D_v1_1/SkeletonOnly/left_arm_link6.STL scale=1 1 1; visual mesh filename=../../meshes/Bessica_D_v1_1/SkeletonOnly/left_arm_link6.STL scale=1 1 1
- link left_arm_link7: mass 0.134233364312826 -> 0.130827779886618; geometry collision mesh filename=../../meshes/Bessica_D_v1_1/SkeletonOnly/left_arm_link7.STL scale=1 1 1; visual mesh filename=../../meshes/Bessica_D_v1_1/SkeletonOnly/left_arm_link7.STL scale=1 1 1
- link right_arm_base_link: mass 0.760760214237615 -> 0.708886467477366; geometry collision mesh filename=../../meshes/Bessica_D_v1_1/SkeletonOnly/right_arm_base_lin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 scale=1 1 1; visual mesh filename=../../meshes/Bessica_D_v1_1/SkeletonOnly/right_arm_base_lin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 scale=1 1 1
- link right_arm_gripper_left_finger: mass 0.0256462690507917 -> 0.0256462690507918; geometry collision mesh filename=../../meshes/Bessica_D_v1_1/SkeletonOnly/right_arm_gripper_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 scale=1 1 1; visual mesh filename=../../meshes/Bessica_D_v1_1/SkeletonOnly/right_arm_gripper_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 scale=1 1 1
- link right_arm_gripper_right_finger: mass 0.025646269050792 -> 0.0256462690507921; geometry collision mesh filename=../../meshes/Bessica_D_v1_1/SkeletonOnly/right_arm_gripper_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 scale=1 1 1; visual mesh filename=../../meshes/Bessica_D_v1_1/SkeletonOnly/right_arm_gripper_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 scale=1 1 1
- link right_arm_link1: mass 0.3157339691478 -> 0.208265932443548; geometry collision mesh filename=../../meshes/Bessica_D_v1_1/SkeletonOnly/right_arm_link1.STL scale=1 1 1; visual mesh filename=../../meshes/Bessica_D_v1_1/SkeletonOnly/right_arm_link1.STL scale=1 1 1
- link right_arm_link2: mass 0.0501482304791555 -> 0.0472690682635543; geometry collision mesh filename=../../meshes/Bessica_D_v1_1/SkeletonOnly/right_arm_link2.STL scale=1 1 1; visual mesh filename=../../meshes/Bessica_D_v1_1/SkeletonOnly/right_arm_link2.STL scale=1 1 1
- link right_arm_link3: mass 0.368447313337917 -> 0.140451564761292; geometry collision mesh filename=../../meshes/Bessica_D_v1_1/SkeletonOnly/right_arm_link3.STL scale=1 1 1; visual mesh filename=../../meshes/Bessica_D_v1_1/SkeletonOnly/right_arm_link3.STL scale=1 1 1
- link right_arm_link4: mass 0.048007139134458 -> 0.0427207248079551; geometry collision mesh filename=../../meshes/Bessica_D_v1_1/SkeletonOnly/right_arm_link4.STL scale=1 1 1; visual mesh filename=../../meshes/Bessica_D_v1_1/SkeletonOnly/right_arm_link4.STL scale=1 1 1
- link right_arm_link5: mass 0.207077281082729 -> 0.110396949965053; geometry collision mesh filename=../../meshes/Bessica_D_v1_1/SkeletonOnly/right_arm_link5.STL scale=1 1 1; visual mesh filename=../../meshes/Bessica_D_v1_1/SkeletonOnly/right_arm_link5.STL scale=1 1 1
- link right_arm_link6: mass 0.0325622574715594 -> 0.0345706786766012; geometry collision mesh filename=../../meshes/Bessica_D_v1_1/SkeletonOnly/right_arm_link6.STL scale=1 1 1; visual mesh filename=../../meshes/Bessica_D_v1_1/SkeletonOnly/right_arm_link6.STL scale=1 1 1
- link right_arm_link7: mass 0.130617660751133 -> 0.134443483448265; geometry collision mesh filename=../../meshes/Bessica_D_v1_1/SkeletonOnly/right_arm_link7.STL scale=1 1 1; visual mesh filename=../../meshes/Bessica_D_v1_1/SkeletonOnly/right_arm_link7.STL scale=1 1 1
Joints:
- removed joint left_gripper_joint
- removed joint right_gripper_joint
- added joint left_tool0_fixed_joint: type fixed, parent left_arm_link7, child left_tool0, origin xyz=0.15 0 0 rpy=0 0 0, axis 0 0 0
- added joint right_tool0_fixed_joint: type fixed, parent right_arm_link7, child right_tool0, origin xyz=0.15 0 0 rpy=0 0 0, axis 0 0 0
- joint head: child head -> head_link; origin xyz=-0.058269 -0.0021593 1.1945 rpy=0 0 0 -> xyz=0.0608244989821353 0.00175926213288549 0.700041453535696 rpy=0 0 0
- joint left_arm_base_joint: origin xyz=0 -0.100000000333333 1.01500000133333 rpy=1.5707963267949 0 0 -> xyz=-0.0608244908152262 0.0882407378671147 -0.185541452202364 rpy=1.5707963267949 0 -3.14159265358979; parent base_link -> head_link
- joint left_arm_gripper_joint1: axis 0 0 0 -> 0 0 1; child left_arm_gripper_left_finger -> left_arm_gripper_right_finger; limit lower=0.05 upper=0 effort=5 velocity=12 -> lower=-0.05 upper=0 effort=5 velocity=12; origin xyz=0.141279659620444 -0.0505000000000146 -0.000149999999993239 rpy=-1.57079632679466 0 0 -> xyz=0.14058 0.046348 0.00015 rpy=1.5708 0 0; type fixed -> prismatic
- joint left_arm_gripper_joint2: axis 0 0 0 -> 0 0 -1; child left_arm_gripper_right_finger -> left_arm_gripper_left_finger; limit (none) -> lower=0 upper=0.05 effort=5 velocity=12; origin xyz=0.141279659620445 0.0504999999999851 -0.000149999999972228 rpy=1.57079632679513 0 0 -> xyz=0.14058 -0.054652 0.00015 rpy=-1.5708 0 0; type fixed -> prismatic
- joint left_arm_joint1: limit lower=-2.14 upper=2.14 effort=5 velocity=12 -> lower=-2.749 upper=2.749 effort=5 velocity=12; origin xyz=0 0 0.1145 rpy=0 0 0 -> xyz=4.99975002436759E-05 0 0.1146 rpy=3.14159265358979 0 0
- joint left_arm_joint2: axis 0 0 -1 -> 0 0 0.999999999999908; limit lower=-2.14 upper=2.14 effort=5 velocity=12 -> lower=-0.1 upper=3.14159 effort=5 velocity=12; origin xyz=0 0 0.04287 rpy=1.57079632679489 0 1.5707963267949 -> xyz=0 0 -0.04286 rpy=1.5707963267949 0 -1.5707963267949
- joint left_arm_joint3: axis 0 0 1 -> 0 0 -0.999999999999908; limit lower=-2.14 upper=2.14 effort=5 velocity=12 -> lower=-2.79 upper=2.79 effort=5 velocity=12; origin xyz=-0.0657500000000001 -9.99999999995171E-05 -0.000400000003120824 rpy=1.5707963267949 0 -1.5707963267949 -> xyz=-0.0645499982324007 0 -0.000299995732645275 rpy=0 -1.5707963267949 0
- joint left_arm_joint4: limit lower=-2.14 upper=2.14 effort=5 velocity=12 -> lower=-0.5236 upper=2.95 effort=5 velocity=12; origin xyz=0.00383999999999432 0 0.20080999933334 rpy=-1.5707963267949 0 0 -> xyz=-1.89941608896571E-05 -4.99999999989398E-05 0.1816 rpy=1.57079632191723 -1.57079611188729 0
- joint left_arm_joint5: limit lower=-2.14 upper=2.14 effort=5 velocity=12 -> lower=-2.79 upper=2.79 effort=5 velocity=12; origin xyz=0 -0.0657500006666611 0.000199999999990721 rpy=-1.5707963267949 0 0 -> xyz=0 -0.0488000000000013 9.99999999971857E-05 rpy=1.5707963267949 1.5707963267949 0
- joint left_arm_joint6: limit lower=-2.14 upper=2.14 effort=5 velocity=12 -> lower=-1.675 upper=1.675 effort=5 velocity=12; origin xyz=0.00379000000002061 5.00000000002069E-05 -0.17879999933334 rpy=1.5707963267949 0 0 -> xyz=0.00289000000000006 -0.00207606624709478 0.108009995732641 rpy=-1.5707963267949 0 0
- joint left_arm_joint7: limit lower=-2.14 upper=2.14 effort=5 velocity=12 -> lower=-1.448 upper=1.448 effort=5 velocity=12; origin xyz=9.99999999615753E-05 -0.0556000006666605 -9.99999999948057E-05 rpy=-1.57079632679513 0 -1.5707963267949 -> xyz=-0.00149999999999997 -0.0563100878103864 0.00415239451449378 rpy=1.5707963267949 0 -1.5707963267949
- joint right_arm_base_joint: origin xyz=0 0.0999999996666618 1.01500000066667 rpy=0 0 0 -> xyz=-0.060825 -0.091759 -0.18554 rpy=3.1416 0 -3.1416; parent base_link -> head_link
- joint right_arm_gripper_joint1: axis 0 0 0 -> 0 0 -1; limit lower=0 upper=-0.05 effort=5 velocity=12 -> lower=-0.05 upper=0 effort=5 velocity=12; origin xyz=0.141279659620446 -0.0505000000000126 -0.000150000000035122 rpy=-1.57079632679466 0 0 -> xyz=0.14128 -0.0505 0.00015 rpy=-1.5708 0 0; type fixed -> prismatic
- joint right_arm_gripper_joint2: axis 0 0 0 -> 0 0 1; limit lower=0.05 upper=0 effort=5 velocity=12 -> lower=0 upper=0.05 effort=5 velocity=12; origin xyz=0.141279659620446 0.050499999999987 -0.00015000000001425 rpy=1.57079632679513 0 0 -> xyz=0.14128 0.0505 0.00015 rpy=1.5708 0 0; type fixed -> prismatic
- joint right_arm_joint1: limit lower=-2.14 upper=2.14 effort=5 velocity=12 -> lower=-2.749 upper=2.749 effort=5 velocity=12; origin xyz=0 0.114500000000005 0 rpy=3.14159265358979 0 0 -> xyz=-4.9995E-05 -0.1146 0 rpy=0 0 0
- joint right_arm_joint2: axis 0 0 -1 -> 0 0 1; limit lower=-2.14 upper=2.14 effort=5 velocity=12 -> lower=-0.1 upper=3.1416 effort=5 velocity=12; origin xyz=0 -0.0428699999999995 0 rpy=-3.14159264133724 1.57079625690226 0 -> xyz=0 -0.04286 0 rpy=0 1.5708 0
- joint right_arm_joint3: limit lower=-2.14 upper=2.14 effort=5 velocity=12 -> lower=-2.79 upper=2.79 effort=5 velocity=12; origin xyz=-0.0639500000000018 -0.000100000000001099 -0.000399999996885698 rpy=1.57079632679464 0 -1.5707963267949 -> xyz=-0.06455 0 -0.0003 rpy=3.1416 1.5708 0
- joint right_arm_joint4: axis 0 0 -1 -> 0 0 1; limit lower=-2.14 upper=2.14 effort=5 velocity=12 -> lower=-0.5236 upper=2.95 effort=5 velocity=12; origin xyz=0.00384000000000018 0 0.20261 rpy=-1.57079632679465 0 0 -> xyz=-1.8989E-05 -4.9997E-05 0.1816 rpy=1.5708 1.5708 0
- joint right_arm_joint5: axis 0 0 -1 -> 0 0 1; limit lower=-2.14 upper=2.14 effort=5 velocity=12 -> lower=-2.79 upper=2.79 effort=5 velocity=12; origin xyz=0 -0.0639500000000002 0.000199999999992483 rpy=-1.57079632679515 0 0 -> xyz=0 0.0487999946213909 0.000100002721817094 rpy=1.5707963267948 -1.5707963267949 3.14159265358979
- joint right_arm_joint6: axis 0 0 1 -> 0 0 -1; limit lower=-2.14 upper=2.14 effort=5 velocity=12 -> lower=-1.675 upper=1.675 effort=5 velocity=12; origin xyz=0.00378999999999963 5.00000000468472E-05 -0.1806 rpy=1.57079632679515 0 0 -> xyz=0.00289 -0.0020761 0.10801 rpy=-1.5708 0 0
- joint right_arm_joint7: limit lower=-2.14 upper=2.14 effort=5 velocity=12 -> lower=-1.448 upper=1.448 effort=5 velocity=12; origin xyz=0.000100000000024303 -0.0556000006666655 -9.99999999954217E-05 rpy=-1.57079632679513 0 -1.5707963267949 -> xyz=-0.0015 -0.05561 0 rpy=1.5708 0 -1.5708
