Commit message: A big refactor
compare mjcf with urdf in robocore 2.5dev, make sure they are the same

File: synriard/urdf/Bessica_M_v1_0/Bessica_M_v1_0.urdf (robot description, URDF)
Before this commit: robot Bessica_M_v1_0, 23 links, 22 joints
Links:
- removed link Left_arm_link1
- removed link Left_arm_link2
- removed link Left_arm_link3
- removed link Left_arm_link4
- removed link Left_arm_link5
- removed link Left_arm_link6
- removed link Left_arm_link7
- removed link Left_arm_link8
- removed link Left_arm_link9
- removed link Right_arm_link1
- removed link Right_arm_link2
- removed link Right_arm_link3
- removed link Right_arm_link4
- removed link Right_arm_link5
- removed link Right_arm_link6
- removed link Right_arm_link7
- removed link Right_arm_link8
- removed link Right_arm_link9
- removed link Torso_link1
- removed link Torso_link2
- removed link Torso_link3
- removed link head_link
- added link head; visual sphere radius=0.005
- added link left_arm_link1, mass 0.375516464240854; collision mesh filename=../../meshes/Bessica_M_v1_0/left_arm_link1.STL; visual mesh filename=../../meshes/Bessica_M_v1_0/left_arm_link1.STL
- added link left_arm_link2, mass 0.0664892171532656; collision mesh filename=../../meshes/Bessica_M_v1_0/left_arm_link2.STL; visual mesh filename=../../meshes/Bessica_M_v1_0/left_arm_link2.STL
- added link left_arm_link3, mass 0.276673991803197; collision mesh filename=../../meshes/Bessica_M_v1_0/left_arm_link3.STL; visual mesh filename=../../meshes/Bessica_M_v1_0/left_arm_link3.STL
- added link left_arm_link4, mass 0.147999944374733; collision mesh filename=../../meshes/Bessica_M_v1_0/left_arm_link4.STL; visual mesh filename=../../meshes/Bessica_M_v1_0/left_arm_link4.STL
- added link left_arm_link5, mass 0.162665516295154; collision mesh filename=../../meshes/Bessica_M_v1_0/left_arm_link5.STL; visual mesh filename=../../meshes/Bessica_M_v1_0/left_arm_link5.STL
- added link left_arm_link6, mass 0.148254477929042; collision mesh filename=../../meshes/Bessica_M_v1_0/left_arm_link6.STL; visual mesh filename=../../meshes/Bessica_M_v1_0/left_arm_link6.STL
- added link left_arm_link7, mass 0.162887358777534; collision mesh filename=../../meshes/Bessica_M_v1_0/left_arm_link7.STL; visual mesh filename=../../meshes/Bessica_M_v1_0/left_arm_link7.STL
- added link left_arm_link8, mass 0.0239390375083334; collision mesh filename=../../meshes/Bessica_M_v1_0/left_arm_link8.STL; visual mesh filename=../../meshes/Bessica_M_v1_0/left_arm_link8.STL
- added link left_arm_link9, mass 0.0239390375083335; collision mesh filename=../../meshes/Bessica_M_v1_0/left_arm_link9.STL; visual mesh filename=../../meshes/Bessica_M_v1_0/left_arm_link9.STL
- added link left_tool0; visual sphere radius=0.005
- added link right_arm_link1, mass 0.375516464391834; collision mesh filename=../../meshes/Bessica_M_v1_0/right_arm_link1.STL; visual mesh filename=../../meshes/Bessica_M_v1_0/right_arm_link1.STL
- added link right_arm_link2, mass 0.0428315653175016; collision mesh filename=../../meshes/Bessica_M_v1_0/right_arm_link2.STL; visual mesh filename=../../meshes/Bessica_M_v1_0/right_arm_link2.STL
- added link right_arm_link3, mass 0.281936177906827; collision mesh filename=../../meshes/Bessica_M_v1_0/right_arm_link3.STL; visual mesh filename=../../meshes/Bessica_M_v1_0/right_arm_link3.STL
- added link right_arm_link4, mass 0.147999944408839; collision mesh filename=../../meshes/Bessica_M_v1_0/right_arm_link4.STL; visual mesh filename=../../meshes/Bessica_M_v1_0/right_arm_link4.STL
- added link right_arm_link5, mass 0.162665516517614; collision mesh filename=../../meshes/Bessica_M_v1_0/right_arm_link5.STL; visual mesh filename=../../meshes/Bessica_M_v1_0/right_arm_link5.STL
- added link right_arm_link6, mass 0.148254477928819; collision mesh filename=../../meshes/Bessica_M_v1_0/right_arm_link6.STL; visual mesh filename=../../meshes/Bessica_M_v1_0/right_arm_link6.STL
- added link right_arm_link7, mass 0.162887358777237; collision mesh filename=../../meshes/Bessica_M_v1_0/right_arm_link7.STL; visual mesh filename=../../meshes/Bessica_M_v1_0/right_arm_link7.STL
- added link right_arm_link8, mass 0.0239390375083336; collision mesh filename=../../meshes/Bessica_M_v1_0/right_arm_link8.STL; visual mesh filename=../../meshes/Bessica_M_v1_0/right_arm_link8.STL
- added link right_arm_link9, mass 0.0239390375083335; collision mesh filename=../../meshes/Bessica_M_v1_0/right_arm_link9.STL; visual mesh filename=../../meshes/Bessica_M_v1_0/right_arm_link9.STL
- added link right_tool0; visual sphere radius=0.005
- added link torso_link1, mass 0.102875531767425; collision mesh filename=../../meshes/Bessica_M_v1_0/torso_link1.STL; visual mesh filename=../../meshes/Bessica_M_v1_0/torso_link1.STL
- added link torso_link2, mass 0.0301213530387122; collision mesh filename=../../meshes/Bessica_M_v1_0/torso_link2.STL; visual mesh filename=../../meshes/Bessica_M_v1_0/torso_link2.STL
- added link torso_link3, mass 2.00367952776906; collision mesh filename=../../meshes/Bessica_M_v1_0/torso_link3.STL; visual mesh filename=../../meshes/Bessica_M_v1_0/torso_link3.STL
Joints:
- removed joint Left_gripper1
- removed joint Left_gripper2
- removed joint Left_joint1
- removed joint Left_joint2
- removed joint Left_joint3
- removed joint Left_joint4
- removed joint Left_joint5
- removed joint Left_joint6
- removed joint Left_joint7
- removed joint Right_gripper1
- removed joint Right_gripper2
- removed joint Right_joint1
- removed joint Right_joint2
- removed joint Right_joint3
- removed joint Right_joint4
- removed joint Right_joint5
- removed joint Right_joint6
- removed joint Right_joint7
- removed joint Torso_joint1
- removed joint Torso_joint2
- removed joint Torso_joint3
- removed joint head_joint
- added joint head_fixed_joint: type fixed, parent torso_link3, child head, origin xyz=0 0.4 0 rpy=0 0 0, axis 0 0 0
- added joint left_gripper1: type prismatic, parent left_arm_link7, child left_arm_link8, origin xyz=0.025 0.179 0.00249999999999894 rpy=0 1.5707963267949 0, axis 0 0 1, limit lower=-0.025 upper=0.025 effort=5 velocity=10
- added joint left_gripper2: type prismatic, parent left_arm_link7, child left_arm_link9, origin xyz=-0.0250000000000001 0.179 0.00249999999999898 rpy=3.14159265358979 1.5707963267949 0, axis 0 0 -1, limit lower=-0.025 upper=0.025 effort=5 velocity=10
- added joint left_joint1: type revolute, parent torso_link3, child left_arm_link1, origin xyz=0.14638985542209 0.288056431115988 0 rpy=1.5707963267949 0 1.91986217719376, axis 0 0 -1, limit lower=-3.14159265358979 upper=3.14159265358979 effort=5 velocity=10
- added joint left_joint2: type revolute, parent left_arm_link1, child left_arm_link2, origin xyz=9.99999999994339E-05 0.0301000000000004 0.0649999999999997 rpy=1.5707963267949 1.5707963267949 0, axis 0 0 -1, limit lower=0 upper=3.14159265358979 effort=5 velocity=10
- added joint left_joint3: type revolute, parent left_arm_link2, child left_arm_link3, origin xyz=0.00889252372646632 -0.0694320081404338 0.0301000000000011 rpy=1.5707963267949 0 0.349065850398862, axis 0 0 -1, limit lower=-1.5707963267949 upper=1.5707963267949 effort=5 velocity=10
- added joint left_joint4: type revolute, parent left_arm_link3, child left_arm_link4, origin xyz=0 -0.029675000000001 0.151050000000001 rpy=1.5707963267949 0 0, axis 0 0 -1, limit lower=-2.35619449019234 upper=0.261799387799149 effort=5 velocity=10
- added joint left_joint5: type revolute, parent left_arm_link4, child left_arm_link5, origin xyz=0 0.098299999999999 -0.0284999999999962 rpy=1.5707963267949 0 0, axis 0 0 1, limit lower=-1.309 upper=1.309 effort=5 velocity=10
- added joint left_joint6: type revolute, parent left_arm_link5, child left_arm_link6, origin xyz=0.000500000000001166 0 -0.139500000000004 rpy=1.5707963267949 0 -1.5707963267949, axis 0 0 -1, limit lower=-1.0472 upper=1.0472 effort=5 velocity=10
- added joint left_joint7: type revolute, parent left_arm_link6, child left_arm_link7, origin xyz=0 0 0 rpy=3.14159265358979 1.5707963267949 0, axis 0 0 1, limit lower=-3.14159265358979 upper=3.14159265358979 effort=5 velocity=10
- added joint left_tool0_fixed_joint: type fixed, parent left_arm_link7, child left_tool0, origin xyz=0 0.17 0 rpy=0 0 0, axis 0 0 0
- added joint right_gripper1: type prismatic, parent right_arm_link7, child right_arm_link8, origin xyz=-0.031434667830233 -0.177982756632216 0.00367500000001846 rpy=3.1055462566194 1.5707963267949 0, axis 0 0 1, limit lower=-0.025 upper=0.025 effort=5 velocity=10
- added joint right_gripper2: type prismatic, parent right_arm_link7, child right_arm_link9, origin xyz=0.0185328521185251 -0.179784686200892 0.00367500000001854 rpy=0.0360463969703927 1.5707963267949 0, axis 0 0 -1, limit lower=-0.025 upper=0.025 effort=5 velocity=10
- added joint right_joint1: type revolute, parent torso_link3, child right_arm_link1, origin xyz=-0.146389856983547 0.288056431115987 0 rpy=3.14159265358979 0 -1.91986217719376, axis 0 1 0, limit lower=-3.14159265358979 upper=3.14159265358979 effort=5 velocity=10
- added joint right_joint2: type revolute, parent right_arm_link1, child right_arm_link2, origin xyz=9.9999999999878E-05 0.0649999999999999 0 rpy=-3.14159265358979 0 -1.5707963267949, axis 0 0 -1, limit lower=0 upper=3.14159265358979 effort=5 velocity=10
- added joint right_joint3: type revolute, parent right_arm_link2, child right_arm_link3, origin xyz=0.00889252372646782 -0.0694320081404333 0 rpy=1.5707963267949 0 0.349065850398866, axis 0 0 1, limit lower=-1.5707963267949 upper=1.5707963267949 effort=5 velocity=10
- added joint right_joint4: type revolute, parent right_arm_link3, child right_arm_link4, origin xyz=0 0 0.15105 rpy=-1.5707963267949 0 0, axis 0 0 1, limit lower=-0.261799387799149 upper=2.35619449019234 effort=5 velocity=10
- added joint right_joint5: type revolute, parent right_arm_link4, child right_arm_link5, origin xyz=0 -0.0983000000000001 0.00117500000000332 rpy=1.5707963267949 0 0, axis 0 0 1, limit lower=-1.309 upper=1.309 effort=5 velocity=10
- added joint right_joint6: type revolute, parent right_arm_link5, child right_arm_link6, origin xyz=0.000499999999999251 -0.00117500000000305 0.139500000000004 rpy=1.5707963267949 0 -1.5707963267949, axis 0 0 1, limit lower=-1.0472 upper=1.0472 effort=5 velocity=10
- added joint right_joint7: type revolute, parent right_arm_link6, child right_arm_link7, origin xyz=0 0 0 rpy=1.5707963267949 1.53474992982451 -1.5707963267949, axis 0 0 -1, limit lower=-3.14159265358979 upper=3.14159265358979 effort=5 velocity=10
- added joint right_tool0_fixed_joint: type fixed, parent right_arm_link7, child right_tool0, origin xyz=0 -0.17 0 rpy=0 0 0, axis 0 0 0
- added joint torso_joint1: type revolute, parent base_link, child torso_link1, origin xyz=0.0148249165957707 -0.00771286978644379 -0.004 rpy=3.14159265358979 0 0, axis 0 0 -1, limit lower=-1.57 upper=1.57 effort=5 velocity=10
- added joint torso_joint2: type revolute, parent torso_link1, child torso_link2, origin xyz=-0.0138252880602436 -0.00771287056717217 -0.036549137497876 rpy=-1.5707963267949 0 0, axis -1 0 0, limit lower=-0.52 upper=0.52 effort=5 velocity=10
- added joint torso_joint3: type revolute, parent torso_link2, child torso_link3, origin xyz=0 0 0 rpy=0 1.5707963267949 0, axis 1 0 0, limit lower=-0.52 upper=0.52 effort=5 velocity=10
