Commit message: Update ARX base link

File: synriard/urdf/Alicia_M_v1_2/Alicia_M_v1_2_follower.urdf (robot description, URDF)
Before this commit: robot alicia_m_v1_2_follower, 11 links, 10 joints
Joints:
- removed joint Joint1
- removed joint Joint2
- removed joint Joint3
- removed joint Joint4
- removed joint Joint5
- removed joint Joint6
- added joint joint1: type revolute, parent base_link, child link1, origin xyz=0 -0.0039812 0.09125 rpy=0 0 1.5708, axis 0 0 1, limit lower=-2.7475 upper=2.7475 effort=5 velocity=10
- added joint joint2: type revolute, parent link1, child link2, origin xyz=0.0039812 0 0.0425 rpy=1.5708 0 -1.5708, axis 0 0 1, limit lower=-3.14 upper=0 effort=5 velocity=10
- added joint joint3: type revolute, parent link2, child link3, origin xyz=-0.28184 0.040424 0 rpy=0 0 0, axis 0 0 -1, limit lower=-3.14 upper=0 effort=5 velocity=10
- added joint joint4: type revolute, parent link3, child link4, origin xyz=0.10092 0.028546 0.0036562 rpy=-1.5708 0 -1.5708, axis 0 0 1, limit lower=-2.79 upper=2.79 effort=5 velocity=10
- added joint joint5: type revolute, parent link4, child link5, origin xyz=0 0.0036562 0.1365 rpy=1.5708 0 0, axis 0 0 1, limit lower=-1.57 upper=1.57 effort=5 velocity=10
- added joint joint6: type revolute, parent link5, child link6, origin xyz=0 0.091 0.0036563 rpy=-1.5708 0 0, axis 0 0 1, limit lower=-2.791 upper=2.791 effort=5 velocity=10

File: synriard/urdf/Alicia_M_v1_2/Alicia_M_v1_2_follower_ARX.urdf (robot description, URDF)
Before this commit: robot alicia_m_v1_2_follower_arx, 10 links, 9 joints
Links:
- link link3: mass 0.684309098992517 -> 0.684506224399253
- link link4: mass 0.317091443783321 -> 0.315728889586979
- link link5: mass 0.394074042340231 -> 0.392709523715002
- link link6: mass 0.460840762126963 -> 0.460840761441095
- link link7: mass 0.0249330594865369 -> 0.0249330633936771
- link link8: mass 0.0249330594865369 -> 0.0249330541832031
Joints:
- joint joint1: origin xyz=-0.00398121749160003 0.273740741564725 0.0728140344645214 rpy=0 0 0 -> xyz=0.0086095 0 0.09725 rpy=0 0 1.5708
- joint joint2: origin xyz=0.0039812174916006 0 0.0425000000000036 rpy=1.57079632679489 0 -1.57079632679491 -> xyz=0.0039812 0 0.0425 rpy=1.5708 0 -1.5708
- joint joint3: origin xyz=-0.281841109234439 0.0404241161390766 0 rpy=0 0 0 -> xyz=-0.28184 0.040424 0 rpy=0 0 0
- joint joint4: origin xyz=0.178415999231107 0.0285459415460252 0 rpy=-3.14159265358979 0 3.14159265358978 -> xyz=0.17842 0.028546 0 rpy=-3.1416 0 3.1416
- joint joint5: origin xyz=-0.0629999999999848 0.0340000000000015 -0.00365621749161699 rpy=1.57079632679492 -1.5707963267949 0 -> xyz=-0.063 0.034 -0.0036562 rpy=1.5708 -1.5708 0
- joint joint6: origin xyz=0 0.0290000000000179 0.0403039405042308 rpy=-1.5708 0 -0.013549 -> xyz=8.4179E-05 0.029 0.040304 rpy=-1.5708 0 -0.0029027
- joint left_finger: child link7 -> link8; origin xyz=-0.0500000000000199 0 0.141500000000001 rpy=-3.14159265358979 0 3.14159265358979 -> xyz=0.049964 -0.0018931 0.1415 rpy=3.1416 0.010646 0
- joint right_finger: axis -1 0 0 -> 1 0 0; child link8 -> link7; limit lower=0 upper=0.05 effort=5 velocity=10 -> lower=-0.05 upper=0 effort=5 velocity=10; origin xyz=0.0499999999999802 0 0.1415 rpy=3.14159265358977 0.0135488130341979 0 -> xyz=-0.049964 0.0018931 0.1415 rpy=-3.1416 -0.010646 3.1416
- joint tool0_fixed_joint: origin xyz=0 0 0.14 rpy=0 0 0 -> xyz=0 0 0.15 rpy=0 0 0

Commit message: Update alicia m parameters

File: synriard/urdf/Alicia_M_v1_2/Alicia_M_v1_2_follower.urdf (robot description, URDF)
Before this commit: robot alicia_m_v1_2_follower, 11 links, 10 joints
Joints:
- joint tool0_fixed_joint: origin xyz=0 0 0.15 rpy=0 0 0 -> xyz=0 0 0.1295 rpy=0 0 0

File: synriard/urdf/Alicia_M_v1_2/Alicia_M_v1_2_follower_ARX.urdf (robot description, URDF)
Before this commit: robot alicia_m_v1_2_follower_arx, 10 links, 9 joints
Joints:
- joint joint4: limit lower=-1.57 upper=1.57 effort=5 velocity=10 -> lower=-1.57 upper=0.785 effort=5 velocity=10
- joint tool0_fixed_joint: origin xyz=0 0 0.15 rpy=0 0 0 -> xyz=0 0 0.1295 rpy=0 0 0

File: synriard/urdf/Corina_v1_2/Corina_v1_2.urdf (robot description, URDF)
Before this commit: robot Corina_v1_2, 21 links, 20 joints
Joints:
- removed joint right__hand_joint2
- added joint right_hand_joint2: type revolute, parent right_hand_link, child right_hand_link2, origin xyz=0 0 0.0422 rpy=0 -1.5708 0, axis 0 0 1, limit lower=-1.57 upper=1.57 effort=5 velocity=10
- joint left_leg_joint: limit lower=-1.57 upper=1.57 effort=5 velocity=10 -> lower=-1.57 upper=1.57 effort=27 velocity=36
- joint left_leg_joint2: limit lower=-3.14 upper=0 effort=5 velocity=10 -> lower=-3.14 upper=0 effort=27 velocity=36
- joint left_leg_joint3: limit lower=-1.57 upper=1.57 effort=5 velocity=10 -> lower=-1.57 upper=1.57 effort=11 velocity=120
- joint left_leg_joint4: limit lower=-1.57 upper=1.57 effort=5 velocity=10 -> lower=-1.57 upper=1.57 effort=27 velocity=36
- joint left_leg_joint5: limit lower=-0.26 upper=0.26 effort=5 velocity=10 -> lower=-0.26 upper=0.26 effort=11 velocity=120
- joint left_leg_joint6: limit lower=-0.26 upper=0.26 effort=5 velocity=10 -> lower=-0.26 upper=0.26 effort=11 velocity=120
- joint right_leg_joint1: limit lower=-1.57 upper=1.57 effort=5 velocity=10 -> lower=-1.57 upper=1.57 effort=27 velocity=36
- joint right_leg_joint2: limit lower=0 upper=3.14 effort=5 velocity=10 -> lower=0 upper=3.14 effort=27 velocity=36
- joint right_leg_joint3: limit lower=-1.57 upper=1.57 effort=5 velocity=10 -> lower=-1.57 upper=1.57 effort=11 velocity=120
- joint right_leg_joint4: limit lower=-1.57 upper=1.57 effort=5 velocity=10 -> lower=-1.57 upper=1.57 effort=27 velocity=36
- joint right_leg_joint5: limit lower=-0.26 upper=0.26 effort=5 velocity=10 -> lower=-0.26 upper=0.26 effort=11 velocity=120
- joint right_leg_joint6: limit lower=-0.26 upper=0.26 effort=5 velocity=10 -> lower=-0.26 upper=0.26 effort=11 velocity=120
