Commit message: Update ARX joint direction

File: synriard/urdf/Alicia_M_v1_2/Alicia_M_v1_2_follower_ARX.urdf (robot description, URDF)
Before this commit: robot alicia_m_v1_2_follower_arx, 10 links, 9 joints
Joints:
- joint joint2: axis 0 0 1 -> 0 0 -1; limit lower=-3.14 upper=0 effort=5 velocity=10 -> lower=0 upper=3.14 effort=5 velocity=10
- joint joint4: axis 0 0 -1 -> 0 0 1
- joint joint5: axis 0 0 1 -> 0 0 -1
- joint joint6: axis 0 0 1 -> 0 0 -1

Commit message: Update the tool0 axis direction

File: synriard/urdf/Alicia_M_v1_2/Alicia_M_v1_2_follower_ARX.urdf (robot description, URDF)
Before this commit: robot alicia_m_v1_2_follower_arx, 10 links, 9 joints
Joints:
- joint joint2: axis 0 0 -1 -> 0 0 1; limit lower=0 upper=3.14 effort=5 velocity=10 -> lower=-3.14 upper=0 effort=5 velocity=10
- joint joint4: axis 0 0 1 -> 0 0 -1; limit lower=-1.57 upper=0.785 effort=5 velocity=10 -> lower=-1.884 upper=1.57 effort=5 velocity=10
- joint joint5: axis 0 0 -1 -> 0 0 1
- joint joint6: axis 0 0 -1 -> 0 0 1
- joint tool0_fixed_joint: origin xyz=0 0 0.1295 rpy=0 0 0 -> xyz=0 0 0.1295 rpy=0 0 -1.5707963
