Commit message: Add arx with paxini sensor

File: synriard/urdf/Alicia_M_v1_2/Alicia_M_v1_2_follower_ARX_PX6D.urdf (robot description, URDF)
Before this commit: robot alicia_m_v1_2_follower, 11 links, 10 joints
Links:
- removed link grasp_base
- link base_link: mass 1.75527696706568 -> 1.30948144128201; geometry collision mesh filename=base_link.stl; visual mesh filename=base_link.stl
- link link1: mass 0.237800297288607 -> 0.243059270540488; geometry collision mesh filename=link1.stl; visual mesh filename=link1.stl
- link link2: mass 0.579389297908421 -> 0.579389297158098; geometry collision mesh filename=link2.stl; visual mesh filename=link2.stl
- link link3: mass 0.523091405901433 -> 0.706595565443392; geometry collision mesh filename=link3.stl; visual mesh filename=link3.stl
- link link4: mass 0.558638138215147 -> 0.365110913723452; geometry collision mesh filename=link4.stl; visual mesh filename=link4.stl
- link link5: mass 0.345531194942532 -> 0.351145554712444; geometry collision mesh filename=link5.stl; visual mesh filename=link5.stl
- link link6: mass 0.46822726567622 -> 0.504336757553032; geometry collision mesh filename=link6.stl; visual mesh filename=link6.stl
- link link7: mass 0.0243852132391449 -> 0.0249330594865369; geometry collision mesh filename=link7.stl; visual mesh filename=link7.stl
- link link8: mass 0.0243852132391449 -> 0.0249330594865369; geometry collision mesh filename=link8.stl; visual mesh filename=link8.stl
Joints:
- removed joint grasp_base_joint
- removed joint left_finger
- removed joint right_finger
- added joint joint7: type prismatic, parent link6, child link7, origin xyz=0 0.05 0.17531 rpy=1.5708 -1.5708 0, axis 0 0 -1, limit lower=-0.05 upper=0 effort=5 velocity=10
- added joint joint8: type prismatic, parent link6, child link8, origin xyz=0 -0.05 0.17531 rpy=0 1.5708 1.5708, axis 0 0 1, limit lower=0 upper=0.05 effort=5 velocity=10
- joint joint1: origin xyz=0 -0.0039812 0.09125 rpy=0 0 1.5708 -> xyz=0.0086095 0 0.09725 rpy=0 0 0
- joint joint2: axis 0 0 1 -> 0 0 -1; origin xyz=0.0039812 0 0.0425 rpy=1.5708 0 -1.5708 -> xyz=0 -0.0004 0.0425 rpy=-1.5708 0 0
- joint joint3: origin xyz=-0.28184 0.040424 0 rpy=0 0 0 -> xyz=-0.28185 -0.040324 0 rpy=3.1416 0 0
- joint joint4: limit lower=-2.79 upper=2.79 effort=5 velocity=10 -> lower=-1.57 upper=1.57 effort=5 velocity=10; origin xyz=0.10092 0.028546 0.0036562 rpy=-1.5708 0 -1.5708 -> xyz=0.21842 0.028546 0 rpy=0 0 0
- joint joint5: origin xyz=0 0.0036562 0.1365 rpy=1.5708 0 0 -> xyz=0.063 0.034 -0.000675 rpy=1.5708 0 0
- joint joint6: origin xyz=0 0.091 0.0036563 rpy=-1.5708 0 0 -> xyz=0.0300000000000271 0 0.0403039405042227 rpy=0 1.5707963267949 0
- joint tool0_fixed_joint: origin xyz=0 0 0.1375 rpy=0 0 0 -> xyz=0 0 0.1735 rpy=0 0 0

File: synriard/urdf/Alicia_M_v1_2/Alicia_M_v1_2_follower_ARX_deprecated.urdf (robot description, URDF)
Before this commit: robot alicia_m_v1_2_follower_arx, 10 links, 9 joints
Links:
- link base_link: geometry collision mesh filename=base_link.STL; visual mesh filename=base_link.STL
- link link1: mass 0.243059270540488 -> 0.243059269381487; geometry collision mesh filename=link1.STL; visual mesh filename=link1.STL
- link link2: mass 0.37082554681883 -> 0.370825547442299; geometry collision mesh filename=link2.STL; visual mesh filename=link2.STL
- link link3: mass 0.706595565442677 -> 0.684506224399253; geometry collision mesh filename=link3.STL; visual mesh filename=link3.STL
- link link4: mass 0.31793009090046 -> 0.315728889586979; geometry collision mesh filename=link4.STL; visual mesh filename=link4.STL
- link link5: mass 0.351145554017841 -> 0.392709523715002; geometry collision mesh filename=link5.STL; visual mesh filename=link5.STL
- link link6: mass 0.460840762126697 -> 0.460840761441095; geometry collision mesh filename=link6.STL; visual mesh filename=link6.STL
- link link7: mass 0.0249330594865369 -> 0.0249330633936771; geometry collision mesh filename=link7.STL; visual mesh filename=link7.STL
- link link8: mass 0.0249330594865369 -> 0.0249330541832031; geometry collision mesh filename=link8.STL; visual mesh filename=link8.STL
Joints:
- removed joint joint7
- removed joint joint8
- added joint left_finger: type prismatic, parent link6, child link8, origin xyz=0.049964 -0.0018931 0.1415 rpy=3.1416 0.010646 0, axis 1 0 0, limit lower=-0.05 upper=0 effort=5 velocity=10
- added joint right_finger: type prismatic, parent link6, child link7, origin xyz=-0.049964 0.0018931 0.1415 rpy=-3.1416 -0.010646 3.1416, axis 1 0 0, limit lower=-0.05 upper=0 effort=5 velocity=10
- joint joint1: origin xyz=0.0086095 0 0.09725 rpy=0 0 0 -> xyz=0.0086095 0 0.09725 rpy=0 0 1.5708
- joint joint2: axis 0 -1 0 -> 0 0 1; origin xyz=0 -0.0004 0.0425 rpy=0 0 0 -> xyz=0.0039812 0 0.0425 rpy=1.5708 0 -1.5708
- joint joint3: axis 0 1 0 -> 0 0 -1; origin xyz=-0.28185 0 0.040324 rpy=0 0 0 -> xyz=-0.28184 0.040424 0 rpy=0 0 0
- joint joint4: axis 0 -1 0 -> 0 0 -1; limit lower=-1.57 upper=1.57 effort=5 velocity=10 -> lower=-1.884 upper=1.57 effort=5 velocity=10; origin xyz=0.21842 0 0.028546 rpy=0 0 0 -> xyz=0.17842 0.028546 0 rpy=-3.1416 0 3.1416
- joint joint5: axis 0 0 -1 -> 0 0 1; origin xyz=0.063 0.000675 0.034 rpy=0 0 0 -> xyz=-0.063 0.034 -0.0036562 rpy=1.5708 -1.5708 0
- joint joint6: axis 1 0 0 -> 0 0 1; origin xyz=0.03 0 -0.040304 rpy=0 0 0 -> xyz=8.4179E-05 0.029 0.040304 rpy=-1.5708 0 -0.0029027
- joint tool0_fixed_joint: origin xyz=0.1375 0 0 rpy=0 1.5707963 0 -> xyz=0 0 0.1375 rpy=0 0 -1.5707963
