Commit message: Correct the corina link name

File: synriard/urdf/Corina_v1_2/Corina_v1_2.urdf (robot description, URDF)
Before this commit: robot Corina_v1_2, 21 links, 20 joints
Links:
- link left_hand_link: mass 0.0514916625984502 -> 0.0414870697899481; geometry collision mesh filename=../../meshes/Corina/left_hand_link1.STL; visual mesh filename=../../meshes/Corina/left_hand_link1.STL
- link left_hand_link2: mass 0.095580268868723 -> 0.0945218936792809
- link left_hand_link3: mass 0.0549751310205965 -> 0.0549751310206084
- link left_hand_link4: mass 0.0708003399992638 -> 0.0708003399992637
- link right_hand_link: mass 0.0414870697899481 -> 0.0514916625984502; geometry collision mesh filename=../../meshes/Corina/right_hand_link1.STL; visual mesh filename=../../meshes/Corina/right_hand_link1.STL
- link right_hand_link2: mass 0.0945218936792809 -> 0.095580268868723
- link right_hand_link3: mass 0.0549751310206084 -> 0.0549751310205965
- link right_hand_link4: mass 0.0708003399992637 -> 0.0708003399992638
Joints:
- joint left_hand_joint: origin xyz=0 -0.107 0.195 rpy=-1.5707963267949 0 -3.14159265358979 -> xyz=0 0.107 0.195 rpy=1.5708 0 3.1416
- joint left_hand_joint2: axis 0 0 -1 -> 0 0 1; origin xyz=0 0 0.042199999999999 rpy=0 -1.5707963267949 0 -> xyz=0 0 0.0422 rpy=0 -1.5708 0
- joint left_hand_joint3: origin xyz=0.0791000000000001 0 0 rpy=0 1.5707963267949 0 -> xyz=0.0791 0 0 rpy=0 1.5708 0
- joint left_hand_joint4: origin xyz=0 0 0.0412 rpy=1.5708 1.5708 0 -> xyz=0 0 0.0412 rpy=-1.5708 0 3.1416
- joint right_hand_joint: origin xyz=0 0.107 0.195 rpy=1.5708 0 3.1416 -> xyz=0 -0.107 0.195 rpy=-1.5707963267949 0 -3.14159265358979
- joint right_hand_joint2: axis 0 0 1 -> 0 0 -1; origin xyz=0 0 0.0422 rpy=0 -1.5708 0 -> xyz=0 0 0.042199999999999 rpy=0 -1.5707963267949 0
- joint right_hand_joint3: origin xyz=0.0791 0 0 rpy=0 1.5708 0 -> xyz=0.0791000000000001 0 0 rpy=0 1.5707963267949 0
- joint right_hand_joint4: origin xyz=0 0 0.0412 rpy=-1.5708 0 3.1416 -> xyz=0 0 0.0412 rpy=1.5708 1.5708 0
